Commit message: Add support wheels on the forks

File: hr_recycler_common/hr_recycler_description/urdf/elevator/elevator.urdf.xacro (robot description, xacro)
@@ -59,4 +59,28 @@
 		</inertial>
 	</link>
+	<joint name="${prefix}_support_wheel_joint" type="fixed">
+			<origin xyz="0 0 -${wheel_radius/2.0+fork_height/2.0}" rpy="0 0 0"/>
+			<parent link="${prefix}_platform_link"/>
+			<child link="${prefix}_support_wheel_link" />
+	</joint>
+	<link name="${prefix}_support_wheel_link">
+		<visual>
+				<origin xyz="-0.2 0 0" rpy="${M_PI/2} 0 0" />
+				<geometry>
+					<cylinder radius="${wheel_radius/2.0}" length="${wheel_height}"/>
+				</geometry>
+		</visual>
+		<collision>
+			<origin xyz="0 0 0" rpy="${M_PI/2} 0 0" />
+			<geometry>
+				<cylinder radius="${wheel_radius/2.0}" length="${wheel_height}"/>
+			</geometry>
+		</collision>
+		<inertial>
+			<mass value="${wheel_mass}" />
+			<origin xyz="0 0 0" />
+			<cylinder_inertia m="${wheel_mass}" r="${wheel_radius}" h="${wheel_height}" />
+		</inertial>
+	</link>
 	<!--xacro:elevator_transmission prefix="${prefix}" /-->
 	<!--xacro:elevator_gazebo prefix="${prefix}" /-->

Commit message: corrected support_wheel radius

File: hr_recycler_common/hr_recycler_description/urdf/elevator/elevator.urdf.xacro (robot description, xacro)
@@ -74,5 +74,5 @@
 			<origin xyz="0 0 0" rpy="${M_PI/2} 0 0" />
 			<geometry>
-				<cylinder radius="${wheel_radius/2.0}" length="${wheel_height}"/>
+				<cylinder radius="${wheel_radius/2.0-fork_height/2.0}" length="${wheel_height}"/>
 			</geometry>
 		</collision>

Commit message: repare fork's collision

File: hr_recycler_common/hr_recycler_description/urdf/elevator/elevator.urdf.xacro (robot description, xacro)
@@ -45,7 +45,7 @@
 		</visual>
 		<collision>
-			<origin xyz="0 0 -0.0" rpy="0 0 0 " />
+			<origin xyz="-${fork_length/2} 0 0" rpy="0 0 0" />
 			<geometry>
-				<box size="0.65 0.5 0.025" />
+				<box size="${fork_length} ${fork_width} ${fork_height}"/>
 			</geometry>
 			<!--geometry>
@@ -72,5 +72,5 @@
 		</visual>
 		<collision>
-			<origin xyz="0 0 0" rpy="${M_PI/2} 0 0" />
+			<origin xyz="-0.2 0 0" rpy="${M_PI/2} 0 0" />
 			<geometry>
 				<cylinder radius="${wheel_radius/2.0-fork_height/2.0}" length="${wheel_height}"/>

Commit message: repare support_wheel radius

File: hr_recycler_common/hr_recycler_description/urdf/elevator/elevator.urdf.xacro (robot description, xacro)
@@ -68,5 +68,5 @@
 				<origin xyz="-0.2 0 0" rpy="${M_PI/2} 0 0" />
 				<geometry>
-					<cylinder radius="${wheel_radius/2.0}" length="${wheel_height}"/>
+					<cylinder radius="${wheel_radius/2.0-fork_height/2.0}" length="${wheel_height}"/>
 				</geometry>
 		</visual>

Commit message: added transmissions

File: hr_recycler_common/hr_recycler_description/urdf/elevator/elevator.urdf.xacro (robot description, xacro)
@@ -59,6 +59,6 @@
 		</inertial>
 	</link>
-	<joint name="${prefix}_support_wheel_joint" type="fixed">
-			<origin xyz="0 0 -${wheel_radius/2.0+fork_height/2.0}" rpy="0 0 0"/>
+	<joint name="${prefix}_support_wheel_joint" type="continuous">
+			<origin xyz="-0.2 0 -${wheel_radius/2.0+fork_height/2.0}" rpy="0 0 0"/>
 			<parent link="${prefix}_platform_link"/>
 			<child link="${prefix}_support_wheel_link" />
@@ -66,5 +66,5 @@
 	<link name="${prefix}_support_wheel_link">
 		<visual>
-				<origin xyz="-0.2 0 0" rpy="${M_PI/2} 0 0" />
+				<origin xyz="0 0 0" rpy="${M_PI/2} 0 0" />
 				<geometry>
 					<cylinder radius="${wheel_radius/2.0-fork_height/2.0}" length="${wheel_height}"/>
@@ -72,5 +72,5 @@
 		</visual>
 		<collision>
-			<origin xyz="-0.2 0 0" rpy="${M_PI/2} 0 0" />
+			<origin xyz="0 0 0" rpy="${M_PI/2} 0 0" />
 			<geometry>
 				<cylinder radius="${wheel_radius/2.0-fork_height/2.0}" length="${wheel_height}"/>
@@ -83,4 +83,14 @@
 		</inertial>
 	</link>
+        <transmission name="${prefix}_support_wheel_transmission">
+      <type>transmission_interface/SimpleTransmission</type>
+      <joint name="${prefix}_support_wheel_joint">
+        <hardwareInterface>hardware_interface/EffortJointInterface</hardwareInterface>
+      </joint>
+      <actuator name="${prefix}_support_wheel_motor">
+        <hardwareInterface>hardware_interface/EffortActuatorInterface</hardwareInterface>
+        <mechanicalReduction>${traction_mechanical_reduction}</mechanicalReduction>
+      </actuator>
+    </transmission>
 	<!--xacro:elevator_transmission prefix="${prefix}" /-->
 	<!--xacro:elevator_gazebo prefix="${prefix}" /-->

File: hr_recycler_common/hr_recycler_description/urdf/wheels/motor_wheel.urdf.xacro (robot description, xacro)
@@ -15,5 +15,5 @@
   <xacro:property name="traction_joint_damping" value="1000.0" />
   <xacro:property name="traction_joint_friction" value="1000.0" />
-  <xacro:property name="traction_joint_effort_limit" value="1000.0" />
+  <xacro:property name="traction_joint_effort_limit" value="100000.0" />
   <xacro:property name="traction_joint_velocity_limit" value="6.28" />
   <xacro:property name="traction_mechanical_reduction" value="1.0" />
@@ -33,5 +33,5 @@
       <dynamics damping="${steer_joint_damping}" friction="${steer_joint_friction}"/>
     </joint>
-    <!--transmission name="${prefix}wheel_steer_trans">
+    <transmission name="${prefix}wheel_steer_trans">
       <type>transmission_interface/SimpleTransmission</type>
       <joint name="${prefix}wheel_steer_joint">
@@ -42,5 +42,5 @@
         <mechanicalReduction>${steer_mechanical_reduction}</mechanicalReduction>
       </actuator>
-    </transmission-->
+    </transmission>
     <link name="${prefix}wheel_steer_link">
       <!--visual>
@@ -79,5 +79,5 @@
       <dynamics damping="${traction_joint_damping}" friction="${traction_joint_friction}"/>
     </joint>
-    <!--transmission name="${prefix}wheel_traction">
+    <transmission name="${prefix}wheel_traction">
       <type>transmission_interface/SimpleTransmission</type>
       <joint name="${prefix}wheel_traction_joint">
@@ -88,5 +88,5 @@
         <mechanicalReduction>${traction_mechanical_reduction}</mechanicalReduction>
       </actuator>
-    </transmission-->
+    </transmission>
     <link name="${prefix}wheel_traction_link">
       <visual>

Commit message: working only traction with velocity controller

File: hr_recycler_common/hr_recycler_description/urdf/elevator/elevator.urdf.xacro (robot description, xacro)
@@ -59,5 +59,5 @@
 		</inertial>
 	</link>
-	<joint name="${prefix}_support_wheel_joint" type="continuous">
+	<joint name="${prefix}_support_wheel_joint" type="fixed">
 			<origin xyz="-0.2 0 -${wheel_radius/2.0+fork_height/2.0}" rpy="0 0 0"/>
 			<parent link="${prefix}_platform_link"/>
@@ -83,5 +83,5 @@
 		</inertial>
 	</link>
-        <transmission name="${prefix}_support_wheel_transmission">
+        <!--transmission name="${prefix}_support_wheel_transmission">
       <type>transmission_interface/SimpleTransmission</type>
       <joint name="${prefix}_support_wheel_joint">
@@ -92,5 +92,5 @@
         <mechanicalReduction>${traction_mechanical_reduction}</mechanicalReduction>
       </actuator>
-    </transmission>
+    </transmission-->
 	<!--xacro:elevator_transmission prefix="${prefix}" /-->
 	<!--xacro:elevator_gazebo prefix="${prefix}" /-->

File: hr_recycler_common/hr_recycler_description/urdf/wheels/motor_wheel.urdf.xacro (robot description, xacro)
@@ -25,5 +25,5 @@
   <xacro:macro name="motor_wheel" params="prefix parent *origin hq">
     <!--MOTOR WHEEL -->
-    <joint name="${prefix}wheel_steer_joint" type="revolute">
+    <joint name="${prefix}wheel_steer_joint" type="fixed">
       <parent link="${parent}"/>
       <child link="${prefix}wheel_steer_link"/>
@@ -33,14 +33,14 @@
       <dynamics damping="${steer_joint_damping}" friction="${steer_joint_friction}"/>
     </joint>
-    <transmission name="${prefix}wheel_steer_trans">
+    <!--transmission name="${prefix}wheel_steer_trans">
       <type>transmission_interface/SimpleTransmission</type>
       <joint name="${prefix}wheel_steer_joint">
-        <hardwareInterface>hardware_interface/PositionJointInterface</hardwareInterface>
+        <hardwareInterface>hardware_interface/EffortJointInterface</hardwareInterface>
       </joint>
       <actuator name="${prefix}wheel_steer_motor">
-        <hardwareInterface>hardware_interface/PositionActuatorInterface</hardwareInterface>
+        <hardwareInterface>hardware_interface/EffortActuatorInterface</hardwareInterface>
         <mechanicalReduction>${steer_mechanical_reduction}</mechanicalReduction>
       </actuator>
-    </transmission>
+    </transmission-->
     <link name="${prefix}wheel_steer_link">
       <!--visual>

Commit message: changed support_wheel_radius, steer works

File: hr_recycler_common/hr_recycler_description/urdf/elevator/elevator.urdf.xacro (robot description, xacro)
@@ -8,4 +8,6 @@
 	<xacro:property name="fork_height" value="0.05" />
 	<xacro:property name="fork_separation" value="0.116" />
+	<xacro:property name="support_wheel_radius" value="${wheel_radius/2.0-fork_height/2.0}" />
+	<xacro:property name="support_wheel_height" value="${wheel_height/2.0}" />
 	<!-- PARAMS: -->
 	<!-- name : name of the link: -->
@@ -68,5 +70,5 @@
 				<origin xyz="0 0 0" rpy="${M_PI/2} 0 0" />
 				<geometry>
-					<cylinder radius="${wheel_radius/2.0-fork_height/2.0}" length="${wheel_height}"/>
+					<cylinder radius="${support_wheel_radius}" length="${wheel_height}"/>
 				</geometry>
 		</visual>
@@ -74,5 +76,5 @@
 			<origin xyz="0 0 0" rpy="${M_PI/2} 0 0" />
 			<geometry>
-				<cylinder radius="${wheel_radius/2.0-fork_height/2.0}" length="${wheel_height}"/>
+				<cylinder radius="${support_wheel_radius}" length="${wheel_height}"/>
 			</geometry>
 		</collision>

Commit message: Changed support_wheels position.

File: hr_recycler_common/hr_recycler_description/urdf/elevator/elevator.urdf.xacro (robot description, xacro)
@@ -12,5 +12,5 @@
   <xacro:property name="fork_z" value="0.0" />
   <!-- Support wheel position -->
-  <xacro:property name="support_wheel_origin" value="-1.5 0.0 ${wheel_radius/4.0}" />
+  <xacro:property name="support_wheel_origin" value="-1.3175 0.0 ${wheel_radius/4.0-0.005}" />
   <!-- Limit elevator -->
   <xacro:property name="upper_limit_elevator" value="0.07" />

Commit message: added true base_link to elevator

File: hr_recycler_common/hr_recycler_description/urdf/elevator/elevator.urdf.xacro (robot description, xacro)
@@ -44,13 +44,24 @@
   <!-- ************** -->
   <xacro:macro name="elevator" params="prefix parent hq *origin" >
-    <joint name="${prefix}base_elevator_joint" type="prismatic">
+    <joint name="${prefix}elevator_base_joint" type="fixed">
         <xacro:insert_block name="origin" />
         <parent link="${parent}"/>
-        <child link="${prefix}base_elevator_link" />
+        <child link="${prefix}elevator_base_link" />
+    </joint>
+    <link name="${prefix}elevator_base_link" >
+      <inertial>
+        <mass value="1" />
+        <origin xyz="0 0 0" />
+        <box_inertia  m="0.001" x="0.001" y="0.001" z="0.001"/>
+      </inertial>
+    </link>
+    <joint name="${prefix}elevator_joint" type="prismatic">
+        <parent link="${prefix}elevator_base_link"/>
+        <child link="${prefix}elevator_link" />
         <axis xyz="0 0 1"/>
         <limit effort="1000.0" lower="0.0" upper="${upper_limit_elevator}" velocity="1"/>
     </joint>
     <!-- This piece supports the two lower forks -->
-    <link name="${prefix}base_elevator_link">
+    <link name="${prefix}elevator_link">
       <visual>
         <origin xyz="0 0 0.410" rpy="0 0 0" />
@@ -74,11 +85,11 @@
       </collision>
     </link>
-    <joint name="${prefix}elevator_joint" type="fixed">
+    <joint name="${prefix}forks_joint" type="fixed">
        <xacro:insert_block name="origin" />
-       <parent link="${prefix}base_elevator_link"/>
-       <child link="${prefix}elevator_link" />
+       <parent link="${prefix}elevator_link"/>
+       <child link="${prefix}forks_link" />
      </joint>
      <!-- This piece holds the forks that are going to be elevated -->
-     <link name="${prefix}elevator_link">
+     <link name="${prefix}forks_link">
        <inertial>
          <mass value="1" />
@@ -100,4 +111,12 @@
            <mesh filename="package://hr_recycler_description/meshes/elevator/hr_recycler_forks.stl" scale="-1 1 1"/>
          </geometry>
+         <surface>
+           <friction>
+             <ode>
+               <mu>100000</mu>
+               <mu2>50000</mu2>
+             </ode>
+           </friction>
+         </surface>
        </collision>
      </link>
@@ -112,10 +131,10 @@
     <!-- TRANSMISSIONS -->
     <!-- ************* -->
-     <transmission name="${prefix}base_elevator_joint_transmission">
+     <transmission name="${prefix}elevator_joint_transmission">
        <type>transmission_interface/SimpleTransmission</type>
-       <joint name="${prefix}base_elevator_joint">
+       <joint name="${prefix}elevator_joint">
          <hardwareInterface>hardware_interface/PositionJointInterface</hardwareInterface>
        </joint>
-       <actuator name="${prefix}base_elevator_joint_motor">
+       <actuator name="${prefix}elevator_joint_motor">
          <hardwareInterface>hardware_interface/PositionActuatorInterface</hardwareInterface>
          <mechanicalReduction>${traction_mechanical_reduction}</mechanicalReduction>

Commit message: added single fork model, needs to correct pose

File: hr_recycler_common/hr_recycler_description/urdf/elevator/elevator.urdf.xacro (robot description, xacro)
@@ -69,7 +69,7 @@
           <mesh filename="package://hr_recycler_description/meshes/bases/base.stl" scale="-1 1 1"/>
         </geometry>
-         <material name="darkgrey">
-           <color rgba="0.1 0.1 0.1 1"/>
-         </material>
+        <material name="darkgrey">
+          <color rgba="0.1 0.1 0.1 1"/>
+        </material>
       </visual>
       <inertial>
@@ -86,5 +86,5 @@
     </link>
     <joint name="${prefix}forks_joint" type="fixed">
-       <xacro:insert_block name="origin" />
+       <origin xyz="-0.363 0.195 0.080" rpy="0 0 3.1415" />
        <parent link="${prefix}elevator_link"/>
        <child link="${prefix}forks_link" />
@@ -94,20 +94,24 @@
        <inertial>
          <mass value="1" />
-         <origin xyz="-0.2 0 0" />
+         <origin xyz="0 0 0" />
          <solid_cuboid_inertia m="${fork_mass}" h="${fork_height}" d="${fork_length}" w="${fork_width}"/>
        </inertial>
        <visual>
-         <origin xyz="-1.3725 0 0.080" rpy="0 0 0" />
+         <!--<origin xyz="${fork_length} 0 0" rpy="0 0 0" />-->
+         <!--<geometry>-->
+           <!--<mesh filename="package://hr_recycler_description/meshes/elevator/single_fork.stl"/>-->
+         <!--</geometry>-->
+         <origin xyz="${fork_length/2.0} 0.0 0.0" rpy="0 0 0" />
          <geometry>
-           <mesh filename="package://hr_recycler_description/meshes/elevator/hr_recycler_forks.stl" scale="-1 1 1"/>
+            <box size="${fork_length} ${fork_width} ${fork_height}" />
          </geometry>
-          <material name="darkgrey">
-            <color rgba="0.1 0.1 0.1 1"/>
-          </material>
+         <material name="darkgrey">
+           <color rgba="0.1 0.1 0.1 1.0"/>
+         </material>
        </visual>
        <collision>
-         <origin xyz="-1.3725 0 0.080" rpy="0 0 0" />
+         <origin xyz="${fork_length/2.0} 0.0 0.0" rpy="0 0 0" />
          <geometry>
-           <mesh filename="package://hr_recycler_description/meshes/elevator/hr_recycler_forks.stl" scale="-1 1 1"/>
+            <box size="${fork_length} ${fork_width} ${fork_height}" />
          </geometry>
          <surface>

Commit message: added individual forks

File: hr_recycler_common/hr_recycler_description/urdf/elevator/elevator.urdf.xacro (robot description, xacro)
@@ -39,4 +39,46 @@
   			<origin xyz="${support_wheel_origin}" rpy="0 0 0"/>
   	</xacro:omni_wheel>
+  </xacro:macro>
+  <xacro:macro name="fork" params="prefix parent hq *origin">
+    <joint name="${prefix}forks_joint" type="fixed">
+  	   <xacro:insert_block name="origin" />
+       <parent link="${parent}"/>
+       <child link="${prefix}fork_link" />
+     </joint>
+     <!-- This piece holds the forks that are going to be elevated -->
+     <link name="${prefix}fork_link">
+       <inertial>
+         <mass value="1" />
+         <origin xyz="0 0 0" />
+         <solid_cuboid_inertia m="${fork_mass}" h="${fork_height}" d="${fork_length}" w="${fork_width}"/>
+       </inertial>
+       <visual>
+         <!--<origin xyz="${fork_length} 0 0" rpy="0 0 0" />-->
+         <!--<geometry>-->
+           <!--<mesh filename="package://hr_recycler_description/meshes/elevator/single_fork.stl"/>-->
+         <!--</geometry>-->
+         <origin xyz="${fork_length/2.0} 0.0 0.0" rpy="0 0 0" />
+         <geometry>
+            <box size="${fork_length} ${fork_width} ${fork_height}" />
+         </geometry>
+         <material name="darkgrey">
+           <color rgba="0.1 0.1 0.1 1.0"/>
+         </material>
+       </visual>
+       <collision>
+         <origin xyz="${fork_length/2.0} 0.0 0.0" rpy="0 0 0" />
+         <geometry>
+            <box size="${fork_length} ${fork_width} ${fork_height}" />
+         </geometry>
+         <surface>
+           <friction>
+             <ode>
+               <mu>100000</mu>
+               <mu2>50000</mu2>
+             </ode>
+           </friction>
+         </surface>
+       </collision>
+     </link>
   </xacro:macro>
   <!-- ************** -->
@@ -85,44 +127,10 @@
       </collision>
     </link>
-    <joint name="${prefix}forks_joint" type="fixed">
+    <xacro:fork prefix="${prefix}left_" parent="${prefix}elevator_link" hq="${hq}">
+       <origin xyz="-0.363 -0.195 0.080" rpy="0 0 3.1415" />
+    </xacro:fork>
+    <xacro:fork prefix="${prefix}right_" parent="${prefix}elevator_link" hq="${hq}">
        <origin xyz="-0.363 0.195 0.080" rpy="0 0 3.1415" />
-       <parent link="${prefix}elevator_link"/>
-       <child link="${prefix}forks_link" />
-     </joint>
-     <!-- This piece holds the forks that are going to be elevated -->
-     <link name="${prefix}forks_link">
-       <inertial>
-         <mass value="1" />
-         <origin xyz="0 0 0" />
-         <solid_cuboid_inertia m="${fork_mass}" h="${fork_height}" d="${fork_length}" w="${fork_width}"/>
-       </inertial>
-       <visual>
-         <!--<origin xyz="${fork_length} 0 0" rpy="0 0 0" />-->
-         <!--<geometry>-->
-           <!--<mesh filename="package://hr_recycler_description/meshes/elevator/single_fork.stl"/>-->
-         <!--</geometry>-->
-         <origin xyz="${fork_length/2.0} 0.0 0.0" rpy="0 0 0" />
-         <geometry>
-            <box size="${fork_length} ${fork_width} ${fork_height}" />
-         </geometry>
-         <material name="darkgrey">
-           <color rgba="0.1 0.1 0.1 1.0"/>
-         </material>
-       </visual>
-       <collision>
-         <origin xyz="${fork_length/2.0} 0.0 0.0" rpy="0 0 0" />
-         <geometry>
-            <box size="${fork_length} ${fork_width} ${fork_height}" />
-         </geometry>
-         <surface>
-           <friction>
-             <ode>
-               <mu>100000</mu>
-               <mu2>50000</mu2>
-             </ode>
-           </friction>
-         </surface>
-       </collision>
-     </link>
+    </xacro:fork>
     <!-- Called two lower forks -->
     <xacro:elevator_platform prefix="${prefix}left_" parent="${prefix}base_footprint" hq="${hq}">
