Commit message: steering works, but forks are skidding

File: hr_recycler_common/hr_recycler_description/urdf/bases/hr_recycler.urdf.xacro (robot description, xacro)
@@ -9,5 +9,5 @@
   <xacro:property name="base_width" value="0.754" />
   <xacro:property name="base_height" value="0.533" />
-  <xacro:property name="base_mass" value="1.0"/>
+  <xacro:property name="base_mass" value="100.0"/>
   <xacro:property name="fork_length" value="1.176" />
   <xacro:property name="fork_width" value="0.11" />
@@ -44,21 +44,18 @@
     </inertial>
     <visual>
-       <origin xyz="0 0 ${wheel_radius+base_height/2.0+separation_wheel_box}" rpy="0 0 0" />
-       <xacro:if value="${hq}">
-         <geometry>
-		   <!--<mesh filename="package://hr_recycler_description/meshes/bases/hr_recycler_base.stl"/>-->
+      <origin xyz="0 0 ${wheel_radius+base_height/2.0+separation_wheel_box}" rpy="0 0 0" />
+      <geometry>
 	       <box size="${base_length} ${base_width} ${base_height}"/>
-         </geometry>
-       </xacro:if>
-       <xacro:unless value="${hq}">
-         <geometry>
-           <!--<mesh filename="package://hr_recycler_description/meshes/bases/hr_recycler.stl"/>-->
-	       <box size="0.679 0.754 0.533"/>
-         </geometry>
-       </xacro:unless>
+      </geometry>
        <material name="darkgrey">
          <color rgba="0.1 0.1 0.1 1"/>
        </material>
     </visual>
+    <collision>
+      <origin xyz="0 0 ${wheel_radius+base_height/2.0+separation_wheel_box}" rpy="0 0 0" />
+      <geometry>
+	       <box size="${base_length} ${base_width} ${base_height}"/>
+      </geometry>
+    </collision>
   </link>
   </xacro:macro>

File: hr_recycler_common/hr_recycler_description/urdf/elevator/elevator.urdf.xacro (robot description, xacro)
@@ -54,7 +54,7 @@
 		</collision>
 		<inertial>
-			<mass value="0.005" />
+			<mass value="1" />
 			<origin xyz="0 0 -0.27" />
-			<solid_cuboid_inertia m="0.005" h="0.05" d="0.05" w="0.05"/>
+			<solid_cuboid_inertia m="1" h="0.05" d="0.05" w="0.05"/>
 		</inertial>
 	</link>
@@ -78,7 +78,7 @@
 		</collision>
 		<inertial>
-			<mass value="${wheel_mass}" />
+			<mass value="0.1" />
 			<origin xyz="0 0 0" />
-			<cylinder_inertia m="${wheel_mass}" r="${wheel_radius}" h="${wheel_height}" />
+			<cylinder_inertia m="0.1" r="${wheel_radius}" h="${wheel_height}" />
 		</inertial>
 	</link>

File: hr_recycler_common/hr_recycler_description/urdf/wheels/motor_wheel.urdf.xacro (robot description, xacro)
@@ -25,5 +25,5 @@
   <xacro:macro name="motor_wheel" params="prefix parent *origin hq">
     <!--MOTOR WHEEL -->
-    <joint name="${prefix}wheel_steer_joint" type="fixed">
+    <joint name="${prefix}wheel_steer_joint" type="revolute">
       <parent link="${parent}"/>
       <child link="${prefix}wheel_steer_link"/>
@@ -33,14 +33,14 @@
       <dynamics damping="${steer_joint_damping}" friction="${steer_joint_friction}"/>
     </joint>
-    <!--transmission name="${prefix}wheel_steer_trans">
+    <transmission name="${prefix}wheel_steer_trans">
       <type>transmission_interface/SimpleTransmission</type>
       <joint name="${prefix}wheel_steer_joint">
-        <hardwareInterface>hardware_interface/EffortJointInterface</hardwareInterface>
+        <hardwareInterface>hardware_interface/VelocityJointInterface</hardwareInterface>
       </joint>
       <actuator name="${prefix}wheel_steer_motor">
-        <hardwareInterface>hardware_interface/EffortActuatorInterface</hardwareInterface>
+        <hardwareInterface>hardware_interface/VelocityActuatorInterface</hardwareInterface>
         <mechanicalReduction>${steer_mechanical_reduction}</mechanicalReduction>
       </actuator>
-    </transmission-->
+    </transmission>
     <link name="${prefix}wheel_steer_link">
       <!--visual>

Commit message: Created two small supports for solving issues with the elevator. Now, it can lift objects without falling forward.

File: hr_recycler_common/hr_recycler_description/urdf/bases/hr_recycler.urdf.xacro (robot description, xacro)
@@ -9,5 +9,5 @@
   <xacro:property name="base_width" value="0.754" />
   <xacro:property name="base_height" value="0.533" />
-  <xacro:property name="base_mass" value="100.0"/>
+  <xacro:property name="base_mass" value="25.0"/>
   <xacro:property name="visual_base_link_z" value="${wheel_radius+base_height/2.0+separation_wheel_box}" />
   <xacro:property name="fork_length" value="1.176" />
@@ -60,4 +60,50 @@
     </collision>
   </link>
+  <!-- BASE HELPER! -->
+  <!-- Two small boxes that help the to not tip over -->
+  <joint name="${prefix}base_helper_joint" type="continuous">
+    <origin xyz="-${base_length/2.0+0.3} ${base_width/2.0-wheel_radius/2.0} -${wheel_radius/2.0}" rpy="0 0 0" />
+    <parent link="${prefix}base_link"/>
+    <child link="${prefix}base_helper_link" />
+  </joint>
+  <link name="${prefix}base_helper_link">
+    <!--visual>
+      <origin xyz="0 0 0" rpy="0 0 0" />
+      <geometry>
+         <sphere radius="${wheel_radius/2.0}"/>
+      </geometry>
+       <material name="darkgrey">
+         <color rgba="0.1 0.1 0.1 1"/>
+       </material>
+    </visual-->
+    <collision>
+      <origin xyz="0 0 0" rpy="0 0 0" />
+      <geometry>
+        <sphere radius="${wheel_radius/2.0}"/>
+      </geometry>
+    </collision>
+    </link>
+    <joint name="${prefix}base_helper_2_joint" type="continuous">
+      <origin xyz="-${base_length/2.0+0.3} -${base_width/2.0-wheel_radius/2.0} -${wheel_radius/2.0}" rpy="0 0 0" />
+      <parent link="${prefix}base_link"/>
+      <child link="${prefix}base_helper_2_link" />
+    </joint>
+    <link name="${prefix}base_helper_2_link">
+      <!--visual>
+        <origin xyz="0 0 0" rpy="0 0 0" />
+        <geometry>
+           <box size="${wheel_radius} ${wheel_radius} ${wheel_radius}"/>
+        </geometry>
+         <material name="darkgrey">
+           <color rgba="0.1 0.1 0.1 1"/>
+         </material>
+      </visual-->
+      <collision>
+        <origin xyz="0 0 0" rpy="0 0 0" />
+        <geometry>
+          <sphere radius="${wheel_radius/2.0}"/>
+        </geometry>
+      </collision>
+      </link>
   </xacro:macro>
 </robot>

File: hr_recycler_common/hr_recycler_description/urdf/elevator/both_elevator.urdf.xacro (robot description, xacro)
@@ -9,8 +9,5 @@
   	<xacro:property name="fork_width" value="0.11" />
   	<xacro:property name="fork_height" value="0.05" />
-  	<xacro:property name="fork_mass" value="1.0" />
-    <!--xacro:macro name="cylinder_inertia" params="m r h">
-      <inertia ixx="${m*(3*r*r+h*h)/12}" ixy = "0" ixz = "0" iyy="${m*(3*r*r+h*h)/12}" iyz = "0" izz="${m*r*r/2}" />
-    </xacro:macro-->
+  	<xacro:property name="fork_mass" value="10.0" />
     <joint name="${prefix}_both_elevator_joint" type="prismatic">
         <xacro:insert_block name="origin" />
@@ -18,13 +15,13 @@
         <child link="${prefix}_platform_link" />
         <axis xyz="0 0 1"/>
-        <limit effort="1000.0" lower="0.0" upper="0.25" velocity="0.01"/>
+        <limit effort="1000.0" lower="0.0" upper="0.25" velocity="1.0"/>
     </joint>
     <transmission name="${prefix}both_elevator_transmission">
       <type>transmission_interface/SimpleTransmission</type>
       <joint name="${prefix}_both_elevator_joint">
-        <hardwareInterface>hardware_interface/VelocityJointInterface</hardwareInterface>
+        <hardwareInterface>hardware_interface/PositionJointInterface</hardwareInterface>
       </joint>
       <actuator name="${prefix}_both_elevator_motor">
-        <hardwareInterface>hardware_interface/VelocityActuatorInterface</hardwareInterface>
+        <hardwareInterface>hardware_interface/PositionActuatorInterface</hardwareInterface>
         <mechanicalReduction>${traction_mechanical_reduction}</mechanicalReduction>
       </actuator>
@@ -38,8 +35,8 @@
     </link>
     <xacro:elevator_platform prefix="$(arg prefix)left_fork" parent="${prefix}_platform_link" hq="${hq}">
-        <origin xyz="0 ${elevator_y} 0" rpy="0 0 0"/>
+        <origin xyz="0 ${elevator_y} -0.02" rpy="0 0 0"/>
     </xacro:elevator_platform>
     <xacro:elevator_platform prefix="$(arg prefix)right_fork" parent="${prefix}_platform_link" hq="${hq}">
-        <origin xyz="0 -${elevator_y} 0" rpy="0 0 0"/>
+        <origin xyz="0 -${elevator_y} -0.02" rpy="0 0 0"/>
     </xacro:elevator_platform>
   </xacro:macro>

File: hr_recycler_common/hr_recycler_description/urdf/elevator/elevator.urdf.xacro (robot description, xacro)
@@ -6,10 +6,10 @@
 	<xacro:property name="fork_length" value="1.176" />
 	<xacro:property name="fork_width" value="0.11" />
-	<xacro:property name="fork_height" value="0.05" />
-	<xacro:property name="fork_mass" value="1.0" />
+	<xacro:property name="fork_height" value="0.03" />
+	<xacro:property name="fork_mass" value="25.0" />
 	<xacro:property name="fork_separation" value="0.116" />
-	<xacro:property name="support_wheel_radius" value="${wheel_radius/2.0-fork_height/4.0}" />
+	<xacro:property name="support_wheel_radius" value="${wheel_radius/2.0-fork_height/2.0}" />
 	<xacro:property name="support_wheel_length" value="${fork_width}" />
-  <xacro:property name="support_wheel_mass" value="1.0" />
+  <xacro:property name="support_wheel_mass" value="5.0" />
 	<xacro:property name="support_wheel_joint_x" value="${0.16-fork_length}" />
 	<xacro:property name="support_wheel_joint_y" value="0.0" />
@@ -30,5 +30,5 @@
 			<child link="${prefix}_platform_link" />
 			<axis xyz="0 0 1"/>
-			<limit effort="1000.0" lower="0.0" upper="1.0" velocity="0.01"/>
+			<limit effort="1000.0" lower="0.0" upper="1.0" velocity="1"/>
 	</joint>
 	<link name="${prefix}_platform_link">
@@ -70,19 +70,18 @@
 			<parent link="${prefix}_platform_link"/>
 			<child link="${prefix}_support_wheel_link" />
+			<limit effort="1000.0" velocity="1.0"/>
 			<axis xyz="0 1 0" rpy="0 0 0" />
 	</joint>
 	<link name="${prefix}_support_wheel_link">
 		<visual>
-				<origin xyz="0 0 0" rpy="${M_PI/2} 0 0" />
+				<origin xyz="0 0 0.01" rpy="${M_PI/2} 0 0" />
 				<geometry>
 					<cylinder radius="${support_wheel_radius}" length="${support_wheel_length}"/>
-					<!--sphere radius="${support_wheel_radius}"/-->
 				</geometry>
 		</visual>
 		<collision>
-			<origin xyz="0 0 0" rpy="${M_PI/2} 0 0" />
+			<origin xyz="0 0 +0.01" rpy="${M_PI/2} 0 0" />
 			<geometry>
 				<cylinder radius="${support_wheel_radius}" length="${support_wheel_length}"/>
-				<!--sphere radius="${support_wheel_radius}" /-->
 			</geometry>
 		</collision>
@@ -93,14 +92,4 @@
 		</inertial>
 	</link>
-        <!--transmission name="${prefix}_support_wheel_transmission">
-      <type>transmission_interface/SimpleTransmission</type>
-      <joint name="${prefix}_support_wheel_joint">
-        <hardwareInterface>hardware_interface/EffortJointInterface</hardwareInterface>
-      </joint>
-      <actuator name="${prefix}_support_wheel_motor">
-        <hardwareInterface>hardware_interface/EffortActuatorInterface</hardwareInterface>
-        <mechanicalReduction>${traction_mechanical_reduction}</mechanicalReduction>
-      </actuator>
-    </transmission-->
 	<!--xacro:elevator_transmission prefix="${prefix}" /-->
 	<!--xacro:elevator_gazebo prefix="${prefix}" /-->

Commit message: Physics seems to work :)!!

File: hr_recycler_common/hr_recycler_description/urdf/bases/hr_recycler.urdf.xacro (robot description, xacro)
@@ -8,6 +8,6 @@
   <xacro:property name="base_length" value="0.679" />
   <xacro:property name="base_width" value="0.754" />
-  <xacro:property name="base_height" value="0.533" />
-  <xacro:property name="base_mass" value="2"/>
+  <xacro:property name="base_height" value="0.2" />
+  <xacro:property name="base_mass" value="50"/>
   <xacro:property name="visual_base_link_z" value="${wheel_radius+base_height/2.0+separation_wheel_box}" />
   <xacro:property name="fork_length" value="1.176" />
@@ -42,6 +42,5 @@
       <mass value="${base_mass}" />
       <origin xyz="0 0 -${wheel_radius}" />
-      <!--box_inertia  m="${base_mass}" x="${base_length}" y="${base_width}" z="${base_height}"/-->
-      <box_inertia  m="${base_mass}" x="0.005" y="0.005" z="0.005"/>
+      <box_inertia  m="${base_mass}" x="${base_length}" y="${base_width}" z="${base_height}"/>
     </inertial>
     <visual>

File: hr_recycler_common/hr_recycler_description/urdf/wheels/motor_wheel.urdf.xacro (robot description, xacro)
@@ -4,8 +4,9 @@
   <!-- Wheels -->
   <xacro:property name="wheel_radius" value="0.1" />
-  <xacro:property name="wheel_height" value="0.14" />
+  <xacro:property name="wheel_height" value="0.1" />
+  <!--xacro:property name="wheel_height" value="0.14" /-->
   <xacro:property name="wheel_mass" value="4.0" />
   <!-- in kg-->
-  <xacro:property name="steer_joint_damping" value="2000.0" />
+  <xacro:property name="steer_joint_damping" value="1000" />
   <xacro:property name="steer_joint_friction" value="1000.0" />
   <xacro:property name="steer_joint_effort_limit" value="9999.0" />
@@ -13,5 +14,5 @@
   <xacro:property name="steer_mechanical_reduction" value="1.0" />
   <xacro:property name="steer_joint_position_limit" value="1.56" />
-  <xacro:property name="traction_joint_damping" value="1000.0" />
+  <xacro:property name="traction_joint_damping" value="5" />
   <xacro:property name="traction_joint_friction" value="1000.0" />
   <xacro:property name="traction_joint_effort_limit" value="100000.0" />

Commit message: now use inertia macros from inertia.urdf.xacro wherever is possible

File: hr_recycler_common/hr_recycler_description/urdf/bases/hr_recycler.urdf.xacro (robot description, xacro)
@@ -1,4 +1,5 @@
 <?xml version="1.0"?>
 <robot name="hr_recycler" xmlns:xacro="http://www.ros.org/wiki/xacro">
+  <xacro:include filename="$(find hr_recycler_description)/urdf/inertia.urdf.xacro" />
   <xacro:macro name="hr_recycler" params="prefix publish_bf hq">
   <!-- Robot mechanical and motor parameters -->
@@ -9,10 +10,4 @@
   <xacro:property name="base_mass" value="1"/>
   <xacro:property name="base_link_origin" value="0 0 0.46" />
-  <!-- Inertial equation -->
-  <xacro:macro name="box_inertia" params="m x y z">
-    <inertia  ixx="${m*(y*y+z*z)/12}" ixy = "0" ixz = "0"
-              iyy="${m*(x*x+z*z)/12}" iyz = "0"
-              izz="${m*(x*x+z*z)/12}" />
-  </xacro:macro>
   <!-- BASE FOOTPRINT -->
   <link name="${prefix}base_footprint">
@@ -28,5 +23,7 @@
       <mass value="${base_mass}" />
       <origin xyz="${base_link_origin}" /><!-- Base_link's inertia origin ->  base_footprint -->
-      <box_inertia  m="${base_mass}" x="${base_length}" y="${base_width}" z="${base_height}"/>
+      <!-- yes, axis in solid_cuboid_inertia are changed, w relates to X axis, d to Z axis, and h to Y axis -->
+      <!-- Keep this comment -->
+      <solid_cuboid_inertia  m="${base_mass}" d="${base_height}" w="${base_length}" h="${base_width}"/>
     </inertial>
     <visual>

File: hr_recycler_common/hr_recycler_description/urdf/elevator/elevator.urdf.xacro (robot description, xacro)
@@ -15,11 +15,4 @@
   <!-- Limit elevator -->
   <xacro:property name="upper_limit_elevator" value="0.07" />
-  <!-- Inertial equation depending of forms -->
-  <xacro:macro name="solid_cuboid_inertia" params="m h d w">
-   <inertia  ixx="${(m*(h*h+d*d))/12}" ixy = "0" ixz = "0"
-             iyy="${(m*(w*w+d*d))/12}" iyz = "0"
-             izz="${(m*(w*w+h*h))/12}"
-    />
-  </xacro:macro>
   <!-- Platform is divided into two parts: TOP PLATFORM with a prismatic
    joint, BELOW PLATFORM which has the two support wheels.-->
@@ -51,5 +44,7 @@
          <mass value="1" />
          <origin xyz="0 0 0" />
-         <solid_cuboid_inertia m="${fork_mass}" h="${fork_height}" d="${fork_length}" w="${fork_width}"/>
+         <!-- yes, axis in solid_cuboid_inertia are changed, w relates to X axis, d to Z axis, and h to Y axis -->
+         <!-- Keep this comment -->
+         <solid_cuboid_inertia m="${fork_mass}" h="${fork_width}" d="${fork_height}" w="${fork_length}"/>
        </inertial>
        <visual>
@@ -95,5 +90,7 @@
         <mass value="1" />
         <origin xyz="0 0 0" />
-        <box_inertia  m="0.001" x="0.001" y="0.001" z="0.001"/>
+         <!-- yes, axis in solid_cuboid_inertia are changed, w relates to X axis, d to Z axis, and h to Y axis -->
+         <!-- Keep this comment -->
+         <solid_cuboid_inertia m="0.001" h="0.001" d="0.001" w="0.001"/>
       </inertial>
     </link>
@@ -118,5 +115,7 @@
         <mass value="1" />
         <origin xyz="-0.8 0 0" />
-        <box_inertia  m="1" x="1.67" y="0.1" z="0.03"/>
+         <!-- yes, axis in solid_cuboid_inertia are changed, w relates to X axis, d to Z axis, and h to Y axis -->
+         <!-- Keep this comment -->
+         <solid_cuboid_inertia m="0.001" h="0.1" d="0.03" w="1.67"/>
       </inertial>
       <collision>

File: hr_recycler_common/hr_recycler_description/urdf/inertia.urdf.xacro (robot description, xacro)
@@ -31,4 +31,6 @@
   </xacro:macro>
   <!-- TODO Solid cuboid of width w, height h, depth d, and mass m -->
+  <!-- yes, axis in solid_cuboid_inertia are changed, w relates to X axis, d to Z axis, and h to Y axis -->
+  <!-- Keep this comment -->
   <xacro:macro name="solid_cuboid_inertia" params="m h d w">
     <inertia  ixx="${(m*(h*h+d*d))/12}" ixy = "0" ixz = "0"
