Commit message: First version of model

File: hr_recycler_common/hr_recycler_description/robots/hr_recycler_std.urdf.xacro (robot description, xacro)
@@ -6,12 +6,15 @@
 	<!-- First we import all posible elements defined in the urdf.xacro files. All these elements are defined as macro:xacros -->
 	<!-- Import HR-RECYCLER base elements -->
-    <xacro:include filename="$(find hr_recycler_description)/urdf/bases/hr_recycler.urdf.xacro" />
+  <xacro:include filename="$(find hr_recycler_description)/urdf/bases/hr_recycler.urdf.xacro" />
 	<!-- Import HR-RECYCLER wheels -->
 	<xacro:include filename="$(find hr_recycler_description)/urdf/wheels/rubber_wheel.urdf.xacro" />
 	<xacro:include filename="$(find hr_recycler_description)/urdf/wheels/omni_wheel.urdf.xacro" />
+	<xacro:include filename="$(find hr_recycler_description)/urdf/wheels/motor_wheel.urdf.xacro" />
+  <!-- Import HR-RECYCLER elevator -->
+	<xacro:include filename="$(find hr_recycler_description)/urdf/elevator/elevator.urdf.xacro" />
 	<!-- Import all available sensors -->
 	<xacro:include filename="$(find robotnik_sensors)/urdf/all_sensors.urdf.xacro" />
     <!-- Import Gazebo Stuff -->
-    <xacro:include filename="$(find hr_recycler_description)/urdf/common.gazebo.xacro" />
+  <xacro:include filename="$(find hr_recycler_description)/urdf/common.gazebo.xacro" />
 	<!-- ***************** -->
 	<!-- Global parameters -->
@@ -19,7 +22,7 @@
 	<xacro:property name="PI" value="3.1415926535897931"/>
 	<!-- Wheel parameters -->
-	<xacro:property name="wheel_offset_x" value="0.0"/>    <!-- x,y,z in translation from base_link to the center of the wheel -->
-	<xacro:property name="wheel_offset_y" value="0.26"/>
-	<xacro:property name="wheel_offset_z" value="0.025"/>
+	<xacro:property name="wheel_offset_x" value="0.5"/>    <!-- x,y,z in translation from base_link to the center of the wheel -->
+	<xacro:property name="wheel_offset_y" value="0.0"/>
+	<xacro:property name="wheel_offset_z" value="0.0"/>
 	<!-- Castor paramters -->
 	<xacro:property name="omni_x" value="0.296"/>
@@ -31,7 +34,7 @@
 	<!-- ELEVATOR PARAMETERS -->
 	<!-- ******************* -->
-	<xacro:property name="elevator_x" value="0.0" />
-	<xacro:property name="elevator_y" value="0.0" />
-	<xacro:property name="elevator_z" value="0.285" />
+	<xacro:property name="elevator_x" value="1.4" />
+	<xacro:property name="elevator_y" value="0.195" />
+	<xacro:property name="elevator_z" value="0.0" />
 	<!-- *************** -->
 	<!-- Robots Elements -->
@@ -39,6 +42,15 @@
 	<!-- Here we create the robot elements using the xacro:macros imported at the beggining of this file -->
 	<!-- HR-RECYCLER base -->
+	<xacro:arg name="prefix" default="hr_recycler_"/>
 	<xacro:hr_recycler prefix="$(arg prefix)" publish_bf="true" hq="${hq}" />
-	<xacro:arg name="prefix" default="hr_recycler_"/>
+	<xacro:motor_wheel prefix="$(arg prefix)back" parent="$(arg prefix)base_link" hq="${hq}">
+			<origin xyz="0 0 ${wheel_radius}" rpy="0 0 0"/>
+	</xacro:motor_wheel>
+	<xacro:elevator_platform prefix="$(arg prefix)left_fork" parent="$(arg prefix)base_link" hq="${hq}">
+			<origin xyz="${elevator_x} ${elevator_y} ${elevator_z}" rpy="0 0 0"/>
+	</xacro:elevator_platform>
+  <xacro:elevator_platform prefix="$(arg prefix)right_fork" parent="$(arg prefix)base_link" hq="${hq}">
+			<origin xyz="${elevator_x} -${elevator_y} ${elevator_z}" rpy="0 0 0"/>
+	</xacro:elevator_platform>
 	<!-- Gazebo ros control pluggins -->
 	<xacro:ros_control/>

File: hr_recycler_common/hr_recycler_description/urdf/bases/hr_recycler.urdf.xacro (robot description, xacro)
@@ -14,4 +14,5 @@
   <xacro:property name="fork_height" value="0.05" />
   <xacro:property name="fork_separation" value="0.116" />
+  <xacro:property name="separation_wheel_box" value="0.08" />
   <xacro:macro name="box_inertia" params="m x y z">
     <inertia  ixx="${m*(y*y+z*z)/12}" ixy = "0" ixz = "0"
@@ -43,5 +44,5 @@
     </inertial>
     <visual>
-       <origin xyz="0 0 ${base_height/2.0}" rpy="0 0 0" />
+       <origin xyz="0 0 ${wheel_radius+base_height/2.0+separation_wheel_box}" rpy="0 0 0" />
        <xacro:if value="${hq}">
          <geometry>

File: hr_recycler_common/hr_recycler_description/urdf/elevator/elevator.urdf.xacro (robot description, xacro)
@@ -4,4 +4,8 @@
 	<xacro:include filename="$(find hr_recycler_description)/urdf/elevator/elevator.gazebo.xacro"/>
 	<xacro:macro name="elevator_platform" params="prefix parent hq *origin">
+	<xacro:property name="fork_length" value="1.176" />
+	<xacro:property name="fork_width" value="0.11" />
+	<xacro:property name="fork_height" value="0.05" />
+	<xacro:property name="fork_separation" value="0.116" />
 	<!-- PARAMS: -->
 	<!-- name : name of the link: -->
@@ -14,6 +18,6 @@
   </xacro:macro>
 	<!-- ELEVATOR PLATFORM -->
-	<joint name="${prefix}_platform_joint" type="prismatic">
-			<origin xyz="0.0 0.0 0.285" rpy="0 0 0 " />
+	<joint name="${prefix}_platform_joint" type="fixed">
+			<xacro:insert_block name="origin" />
 			<parent link="${parent}"/>
 			<child link="${prefix}_platform_link" />
@@ -23,13 +27,15 @@
 	<link name="${prefix}_platform_link">
 		<visual>
-			<origin xyz="0 0 0" rpy="0 0 0" />
+			<origin xyz="-${fork_length/2} 0 0" rpy="0 0 0" />
 			<xacro:if value="${hq}">
 				<geometry>
-					<mesh filename="package://hr_recycler_description/meshes/elevator/hr_recycler_elevator.dae"/>
+					<!--mesh filename="package://hr_recycler_description/meshes/elevator/hr_recycler_elevator.dae"/-->
+					<box size="${fork_length} ${fork_width} ${fork_height}"/>
 				</geometry>
 			</xacro:if>
 			<xacro:unless value="${hq}">
 				<geometry>
-					<mesh filename="package://hr_recycler_description/meshes/elevator/hr_recycler_elevator.stl"/>
+					<!--mesh filename="package://hr_recycler_description/meshes/elevator/hr_recycler_elevator.stl"/-->
+					<box size="${fork_length} ${fork_width} ${fork_height}"/>
 				</geometry>
 			</xacro:unless>
@@ -53,6 +59,6 @@
 		</inertial>
 	</link>
-	<xacro:elevator_transmission prefix="${prefix}" />
-	<xacro:elevator_gazebo prefix="${prefix}" />
+	<!--xacro:elevator_transmission prefix="${prefix}" /-->
+	<!--xacro:elevator_gazebo prefix="${prefix}" /-->
 	</xacro:macro>
 </robot>

Commit message: Changed the support wheel length and fixed fork to prismatic

File: hr_recycler_common/hr_recycler_description/robots/hr_recycler_std.urdf.xacro (robot description, xacro)
@@ -22,19 +22,38 @@
 	<xacro:property name="PI" value="3.1415926535897931"/>
 	<!-- Wheel parameters -->
-	<xacro:property name="wheel_offset_x" value="0.5"/>    <!-- x,y,z in translation from base_link to the center of the wheel -->
+	<xacro:property name="wheel_offset_x" value="0.0"/>    <!-- x,y,z in translation from base_link to the center of the wheel -->
 	<xacro:property name="wheel_offset_y" value="0.0"/>
-	<xacro:property name="wheel_offset_z" value="0.0"/>
+	<xacro:property name="wheel_offset_z" value="${wheel_radius}"/>
+  <xacro:property name="separation_wheel_box" value="0.08" />
+  <!-- Base parameters -->
+  <xacro:property name="base_length" value="0.679" />
+  <xacro:property name="base_height" value="0.533" />
+  <xacro:property name="base_width" value="0.754" />
 	<!-- Castor paramters -->
-	<xacro:property name="omni_x" value="0.296"/>
+	<!--xacro:property name="omni_x" value="0.296"/>
 	<xacro:property name="omni_y" value="0.249"/>
-	<xacro:property name="omni_z" value="0.010"/>
+	<xacro:property name="omni_z" value="0.010"/-->
 	<!-- Flag to select the high or low quality model -->
 	<xacro:property name="hq" value="true" />
+  <!-- ******************* -->
+	<!--  SENSOR PARAMETERS  -->
+	<!-- ******************* -->
+  <xacro:property name="sensor_x" value="${base_length/2.0+sensor_length}" />
+  <xacro:property name="sensor_y" value="0.0" />
+  <xacro:property name="sensor_z" value="${wheel_radius+separation_wheel_box}" />
+  <xacro:property name="sensor_length" value="0.055" />
+  <!-- ******************* -->
+	<!--  CAMERA PARAMETERS  -->
+	<!-- ******************* -->
+  <xacro:property name="camera_x" value="-${fork_length}" />
+  <xacro:property name="camera_y" value="0" />
+  <xacro:property name="camera_z" value="0" />
 	<!-- ******************* -->
 	<!-- ELEVATOR PARAMETERS -->
 	<!-- ******************* -->
-	<xacro:property name="elevator_x" value="1.4" />
+	<xacro:property name="elevator_x" value="-${base_length/2.0}" />
 	<xacro:property name="elevator_y" value="0.195" />
 	<xacro:property name="elevator_z" value="0.0" />
+  <xacro:property name="fork_length" value="1.176" />
 	<!-- *************** -->
 	<!-- Robots Elements -->
@@ -45,5 +64,5 @@
 	<xacro:hr_recycler prefix="$(arg prefix)" publish_bf="true" hq="${hq}" />
 	<xacro:motor_wheel prefix="$(arg prefix)back" parent="$(arg prefix)base_link" hq="${hq}">
-			<origin xyz="0 0 ${wheel_radius}" rpy="0 0 0"/>
+			<origin xyz="${wheel_offset_x} ${wheel_offset_y} ${wheel_offset_z}" rpy="0 0 0"/>
 	</xacro:motor_wheel>
 	<xacro:elevator_platform prefix="$(arg prefix)left_fork" parent="$(arg prefix)base_link" hq="${hq}">
@@ -53,4 +72,13 @@
 			<origin xyz="${elevator_x} -${elevator_y} ${elevator_z}" rpy="0 0 0"/>
 	</xacro:elevator_platform>
+  <xacro:sensor_sick_s300 prefix="$(arg prefix)front_laser" parent="$(arg prefix)base_link">
+      <origin xyz="${sensor_x} ${sensor_y} ${sensor_z}" rpy="0 0 0"/>
+  </xacro:sensor_sick_s300>
+  <xacro:sensor_r430 prefix="$(arg prefix)right_fork_camera" parent="$(arg prefix)right_fork_platform_link">
+      <origin xyz="${camera_x} ${camera_y} ${camera_z}" rpy="0 0 0"/>
+  </xacro:sensor_r430>
+  <xacro:sensor_r430 prefix="$(arg prefix)left_fork_camera" parent="$(arg prefix)left_fork_platform_link">
+      <origin xyz="${camera_x} ${camera_y} ${camera_z}" rpy="0 0 0"/>
+  </xacro:sensor_r430>
 	<!-- Gazebo ros control pluggins -->
 	<xacro:ros_control/>

File: hr_recycler_common/hr_recycler_description/urdf/bases/hr_recycler.urdf.xacro (robot description, xacro)
@@ -10,4 +10,5 @@
   <xacro:property name="base_height" value="0.533" />
   <xacro:property name="base_mass" value="100.0"/>
+  <xacro:property name="visual_base_link_z" value="${wheel_radius+base_height/2.0+separation_wheel_box}" />
   <xacro:property name="fork_length" value="1.176" />
   <xacro:property name="fork_width" value="0.11" />
@@ -44,5 +45,5 @@
     </inertial>
     <visual>
-      <origin xyz="0 0 ${wheel_radius+base_height/2.0+separation_wheel_box}" rpy="0 0 0" />
+      <origin xyz="0 0 ${visual_base_link_z}" rpy="0 0 0" />
       <geometry>
 	       <box size="${base_length} ${base_width} ${base_height}"/>
@@ -53,5 +54,5 @@
     </visual>
     <collision>
-      <origin xyz="0 0 ${wheel_radius+base_height/2.0+separation_wheel_box}" rpy="0 0 0" />
+      <origin xyz="0 0 ${visual_base_link_z}" rpy="0 0 0" />
       <geometry>
 	       <box size="${base_length} ${base_width} ${base_height}"/>

File: hr_recycler_common/hr_recycler_description/urdf/elevator/elevator.urdf.xacro (robot description, xacro)
@@ -7,7 +7,12 @@
 	<xacro:property name="fork_width" value="0.11" />
 	<xacro:property name="fork_height" value="0.05" />
+	<xacro:property name="fork_mass" value="25.0" />
 	<xacro:property name="fork_separation" value="0.116" />
-	<xacro:property name="support_wheel_radius" value="${wheel_radius/2.0-fork_height/2.0}" />
-	<xacro:property name="support_wheel_height" value="${wheel_height/2.0}" />
+	<xacro:property name="support_wheel_radius" value="${wheel_radius/2.0-fork_height/4.0}" />
+	<xacro:property name="support_wheel_length" value="${fork_width}" />
+  <xacro:property name="support_wheel_mass" value="5.0" />
+	<xacro:property name="support_wheel_joint_x" value="${0.16-fork_length}" />
+	<xacro:property name="support_wheel_joint_y" value="0.0" />
+	<xacro:property name="support_wheel_joint_z" value="-${wheel_radius/2.0+fork_height/4.0}" />
 	<!-- PARAMS: -->
 	<!-- name : name of the link: -->
@@ -20,10 +25,10 @@
   </xacro:macro>
 	<!-- ELEVATOR PLATFORM -->
-	<joint name="${prefix}_platform_joint" type="fixed">
+	<joint name="${prefix}_platform_joint" type="prismatic">
 			<xacro:insert_block name="origin" />
 			<parent link="${parent}"/>
 			<child link="${prefix}_platform_link" />
 			<axis xyz="0 0 1"/>
-			<limit effort="1000.0" lower="0.0" upper="0.05" velocity="0.01"/>
+			<limit effort="1000.0" lower="0.0" upper="1.0" velocity="0.01"/>
 	</joint>
 	<link name="${prefix}_platform_link">
@@ -56,13 +61,14 @@
 		</collision>
 		<inertial>
-			<mass value="1" />
+			<mass value="${fork_mass}" />
 			<origin xyz="0 0 -0.27" />
-			<solid_cuboid_inertia m="1" h="0.05" d="0.05" w="0.05"/>
+			<solid_cuboid_inertia m="${fork_mass}" h="${fork_height}" d="${fork_length}" w="${fork_width}"/>
 		</inertial>
 	</link>
-	<joint name="${prefix}_support_wheel_joint" type="fixed">
-			<origin xyz="-0.2 0 -${wheel_radius/2.0+fork_height/2.0}" rpy="0 0 0"/>
+	<joint name="${prefix}_support_wheel_joint" type="continuous">
+			<origin xyz="${support_wheel_joint_x} ${support_wheel_joint_y} ${support_wheel_joint_z}" rpy="0 0 0"/>
 			<parent link="${prefix}_platform_link"/>
 			<child link="${prefix}_support_wheel_link" />
+			<axis xyz="0 1 0" rpy="0 0 0" />
 	</joint>
 	<link name="${prefix}_support_wheel_link">
@@ -70,5 +76,6 @@
 				<origin xyz="0 0 0" rpy="${M_PI/2} 0 0" />
 				<geometry>
-					<cylinder radius="${support_wheel_radius}" length="${wheel_height}"/>
+					<cylinder radius="${support_wheel_radius}" length="${support_wheel_length}"/>
+					<!--sphere radius="${support_wheel_radius}"/-->
 				</geometry>
 		</visual>
@@ -76,11 +83,12 @@
 			<origin xyz="0 0 0" rpy="${M_PI/2} 0 0" />
 			<geometry>
-				<cylinder radius="${support_wheel_radius}" length="${wheel_height}"/>
+				<cylinder radius="${support_wheel_radius}" length="${support_wheel_length}"/>
+				<!--sphere radius="${support_wheel_radius}" /-->
 			</geometry>
 		</collision>
 		<inertial>
-			<mass value="0.1" />
+			<mass value="${support_wheel_mass}" />
 			<origin xyz="0 0 0" />
-			<cylinder_inertia m="0.1" r="${wheel_radius}" h="${wheel_height}" />
+			<cylinder_inertia m="${support_wheel_mass}" r="${support_wheel_length}" h="${support_wheel_length}" />
 		</inertial>
 	</link>

File: hr_recycler_common/hr_recycler_description/urdf/wheels/motor_wheel.urdf.xacro (robot description, xacro)
@@ -48,5 +48,4 @@
           <origin xyz="0 0 0" rpy="0 0 ${M_PI}" />
           <geometry>
-            <cylinder radius="1" length="1"/>
           </geometry>
         </xacro:if>
@@ -61,5 +60,4 @@
         <origin xyz="0 0 0" rpy="0 0 0" />
         <geometry>
-             <mesh filename="package://vulcano_base_description/meshes/wheels/steer_wheel.stl" />
         </geometry>
       </collision-->

Commit message: Added prismatic move, the sim works but the base tilts by weight

File: hr_recycler_common/hr_recycler_description/robots/hr_recycler_std.urdf.xacro (robot description, xacro)
@@ -13,4 +13,5 @@
   <!-- Import HR-RECYCLER elevator -->
 	<xacro:include filename="$(find hr_recycler_description)/urdf/elevator/elevator.urdf.xacro" />
+  <xacro:include filename="$(find hr_recycler_description)/urdf/elevator/both_elevator.urdf.xacro" />
 	<!-- Import all available sensors -->
 	<xacro:include filename="$(find robotnik_sensors)/urdf/all_sensors.urdf.xacro" />
@@ -66,10 +67,13 @@
 			<origin xyz="${wheel_offset_x} ${wheel_offset_y} ${wheel_offset_z}" rpy="0 0 0"/>
 	</xacro:motor_wheel>
-	<xacro:elevator_platform prefix="$(arg prefix)left_fork" parent="$(arg prefix)base_link" hq="${hq}">
+  <xacro:both_elevator prefix="$(arg prefix)both_forks" parent="$(arg prefix)base_link" hq="${hq}">
+      <origin xyz="${elevator_x} 0 ${elevator_z}" rpy="0 0 0"/>
+  </xacro:both_elevator>
+	<!--xacro:elevator_platform prefix="$(arg prefix)left_fork" parent="$(arg prefix)base_link" hq="${hq}">
 			<origin xyz="${elevator_x} ${elevator_y} ${elevator_z}" rpy="0 0 0"/>
-	</xacro:elevator_platform>
-  <xacro:elevator_platform prefix="$(arg prefix)right_fork" parent="$(arg prefix)base_link" hq="${hq}">
+	</xacro:elevator_platform-->
+  <!--xacro:elevator_platform prefix="$(arg prefix)right_fork" parent="$(arg prefix)base_link" hq="${hq}">
 			<origin xyz="${elevator_x} -${elevator_y} ${elevator_z}" rpy="0 0 0"/>
-	</xacro:elevator_platform>
+	</xacro:elevator_platform-->
   <xacro:sensor_sick_s300 prefix="$(arg prefix)front_laser" parent="$(arg prefix)base_link">
       <origin xyz="${sensor_x} ${sensor_y} ${sensor_z}" rpy="0 0 0"/>

File: hr_recycler_common/hr_recycler_description/urdf/elevator/elevator.gazebo.xacro (robot description, xacro)
@@ -2,5 +2,5 @@
 <robot xmlns:xacro="http://www.ros.org/wiki/xacro">
 	<xacro:macro name="elevator_gazebo" params="prefix">
-		<gazebo reference="${prefix}_platform_link">
+		<gazebo reference="${prefix}platform_link">
 			<mu1 value="5.0"/>
 			<mu2 value="0.5"/>

File: hr_recycler_common/hr_recycler_description/urdf/elevator/elevator.urdf.xacro (robot description, xacro)
@@ -7,9 +7,9 @@
 	<xacro:property name="fork_width" value="0.11" />
 	<xacro:property name="fork_height" value="0.05" />
-	<xacro:property name="fork_mass" value="25.0" />
+	<xacro:property name="fork_mass" value="1.0" />
 	<xacro:property name="fork_separation" value="0.116" />
 	<xacro:property name="support_wheel_radius" value="${wheel_radius/2.0-fork_height/4.0}" />
 	<xacro:property name="support_wheel_length" value="${fork_width}" />
-  <xacro:property name="support_wheel_mass" value="5.0" />
+  <xacro:property name="support_wheel_mass" value="1.0" />
 	<xacro:property name="support_wheel_joint_x" value="${0.16-fork_length}" />
 	<xacro:property name="support_wheel_joint_y" value="0.0" />
@@ -25,5 +25,5 @@
   </xacro:macro>
 	<!-- ELEVATOR PLATFORM -->
-	<joint name="${prefix}_platform_joint" type="prismatic">
+	<joint name="${prefix}_platform_joint" type="fixed">
 			<xacro:insert_block name="origin" />
 			<parent link="${parent}"/>

Commit message: Repare some issues with sensor and cameras.

File: hr_recycler_common/hr_recycler_description/robots/hr_recycler_std.urdf.xacro (robot description, xacro)
@@ -42,5 +42,5 @@
   <xacro:property name="sensor_x" value="${base_length/2.0+sensor_length}" />
   <xacro:property name="sensor_y" value="0.0" />
-  <xacro:property name="sensor_z" value="${wheel_radius+separation_wheel_box}" />
+  <xacro:property name="sensor_z" value="${wheel_radius+separation_wheel_box+0.087}" />
   <xacro:property name="sensor_length" value="0.055" />
   <!-- ******************* -->
@@ -77,11 +77,11 @@
 	</xacro:elevator_platform-->
   <xacro:sensor_sick_s300 prefix="$(arg prefix)front_laser" parent="$(arg prefix)base_link">
-      <origin xyz="${sensor_x} ${sensor_y} ${sensor_z}" rpy="0 0 0"/>
+      <origin xyz="${sensor_x} ${sensor_y} ${sensor_z}" rpy="${PI} 0 0"/>
   </xacro:sensor_sick_s300>
-  <xacro:sensor_r430 prefix="$(arg prefix)right_fork_camera" parent="$(arg prefix)right_fork_platform_link">
-      <origin xyz="${camera_x} ${camera_y} ${camera_z}" rpy="0 0 0"/>
+  <xacro:sensor_r430 prefix="$(arg prefix)right_fork_camera" parent="$(arg prefix)right_fork_platform_link" prefix_topic="front_right_rgbd_camera">
+      <origin xyz="${camera_x} ${camera_y} ${camera_z}" rpy="0 0 ${PI}"/>
   </xacro:sensor_r430>
-  <xacro:sensor_r430 prefix="$(arg prefix)left_fork_camera" parent="$(arg prefix)left_fork_platform_link">
-      <origin xyz="${camera_x} ${camera_y} ${camera_z}" rpy="0 0 0"/>
+  <xacro:sensor_r430 prefix="$(arg prefix)left_fork_camera" parent="$(arg prefix)left_fork_platform_link" prefix_topic="front_left_rgbd_camera">
+      <origin xyz="${camera_x} ${camera_y} ${camera_z}" rpy="0 0 ${PI}"/>
   </xacro:sensor_r430>
 	<!-- Gazebo ros control pluggins -->
