Commit message: Changed steer and elevator controller from Velocity to Position

File: hr_recycler_common/hr_recycler_description/robots/hr_recycler_std.urdf.xacro (robot description, xacro)
@@ -47,5 +47,5 @@
 	<!--  CAMERA PARAMETERS  -->
 	<!-- ******************* -->
-  <xacro:property name="camera_x" value="-${fork_length}" />
+  <xacro:property name="camera_x" value="-${fork_length+0.025}" />
   <xacro:property name="camera_y" value="0" />
   <xacro:property name="camera_z" value="0" />
@@ -54,5 +54,5 @@
 	<!-- ******************* -->
 	<xacro:property name="elevator_x" value="-${base_length/2.0}" />
-	<xacro:property name="elevator_y" value="0.195" />
+	<xacro:property name="elevator_y" value="0.0" />
 	<xacro:property name="elevator_z" value="0.0" />
   <xacro:property name="fork_length" value="1.176" />
@@ -68,12 +68,6 @@
 	</xacro:motor_wheel>
   <xacro:both_elevator prefix="$(arg prefix)both_forks" parent="$(arg prefix)base_link" hq="${hq}">
-      <origin xyz="${elevator_x} 0 ${elevator_z}" rpy="0 0 0"/>
+      <origin xyz="${elevator_x} ${elevator_y} ${elevator_z}" rpy="0 0 0"/>
   </xacro:both_elevator>
-	<!--xacro:elevator_platform prefix="$(arg prefix)left_fork" parent="$(arg prefix)base_link" hq="${hq}">
-			<origin xyz="${elevator_x} ${elevator_y} ${elevator_z}" rpy="0 0 0"/>
-	</xacro:elevator_platform-->
-  <!--xacro:elevator_platform prefix="$(arg prefix)right_fork" parent="$(arg prefix)base_link" hq="${hq}">
-			<origin xyz="${elevator_x} -${elevator_y} ${elevator_z}" rpy="0 0 0"/>
-	</xacro:elevator_platform-->
   <xacro:sensor_sick_s300 prefix="$(arg prefix)front_laser" parent="$(arg prefix)base_link">
       <origin xyz="${sensor_x} ${sensor_y} ${sensor_z}" rpy="${PI} 0 0"/>
@@ -85,4 +79,9 @@
       <origin xyz="${camera_x} ${camera_y} ${camera_z}" rpy="0 0 ${PI}"/>
   </xacro:sensor_r430>
+  <!--gazebo>
+    <plugin name="gazebo_ros_control" filename="libgazebo_ros_control.so">
+      <robotSimType>steer_bot_hardware_gazebo/SteerBotHardwareGazebo</robotSimType>
+    </plugin>
+  </gazebo-->
 	<!-- Gazebo ros control pluggins -->
 	<xacro:ros_control/>

File: hr_recycler_common/hr_recycler_description/urdf/wheels/motor_wheel.urdf.xacro (robot description, xacro)
@@ -36,30 +36,12 @@
       <type>transmission_interface/SimpleTransmission</type>
       <joint name="${prefix}wheel_steer_joint">
-        <hardwareInterface>hardware_interface/VelocityJointInterface</hardwareInterface>
+        <hardwareInterface>hardware_interface/PositionJointInterface</hardwareInterface>
       </joint>
       <actuator name="${prefix}wheel_steer_motor">
-        <hardwareInterface>hardware_interface/VelocityActuatorInterface</hardwareInterface>
+        <hardwareInterface>hardware_interface/PositionActuatorInterface</hardwareInterface>
         <mechanicalReduction>${steer_mechanical_reduction}</mechanicalReduction>
       </actuator>
     </transmission>
     <link name="${prefix}wheel_steer_link">
-      <!--visual>
-        <xacro:if value="${hq}">
-          <origin xyz="0 0 0" rpy="0 0 ${M_PI}" />
-          <geometry>
-          </geometry>
-        </xacro:if>
-        <xacro:unless value="${hq}">
-          <origin xyz="0 0 0" rpy="0 0 ${M_PI}" />
-          <geometry>
-            <cylinder radius="1" length="1"/>
-          </geometry>
-        </xacro:unless>
-      </visual-->
-      <!--collision>
-        <origin xyz="0 0 0" rpy="0 0 0" />
-        <geometry>
-        </geometry>
-      </collision-->
       <inertial>
         <mass value="${wheel_mass}" />
@@ -114,20 +96,4 @@
       </inertial>
     </link>
-    <!--<gazebo reference="${prefix}wheel_tracion_link">-->
-    <!--<mu1 value="1.0"/>-->
-    <!--<mu2 value="1.0"/>-->
-    <!--[><kp value="10000000.0" /><]-->
-    <!--[><kd value="1.0" /><]-->
-    <!--[><fdir1 value="1 0 0"/><]-->
-    <!--[><turnGravityOff>false</turnGravityOff><]-->
-    <!--</gazebo>-->
-    <!-- gazebo reference="${prefix}motor_wheel_link">
-        <mu1 value="1.0"/>
-        <mu2 value="1.0"/>
-        <kp value="10000000.0" />
-        <kd value="1.0" />
-        <fdir1 value="1 0 0"/>
-        <turnGravityOff>false</turnGravityOff>
-   </gazebo -->
   </xacro:macro>
 </robot>

Commit message: Added Ackermann, pid_yaml but it's as a comment, removed base helper, added fork, added gazebo motor wheel references.

File: hr_recycler_common/hr_recycler_description/robots/hr_recycler_std.urdf.xacro (robot description, xacro)
@@ -55,6 +55,7 @@
 	<xacro:property name="elevator_x" value="-${base_length/2.0}" />
 	<xacro:property name="elevator_y" value="0.0" />
-	<xacro:property name="elevator_z" value="0.0" />
+	<xacro:property name="elevator_z" value="${-wheel_radius/2.0+fork_height/2.0}" />
   <xacro:property name="fork_length" value="1.176" />
+  <xacro:property name="fork_height" value="0.015" />
 	<!-- *************** -->
 	<!-- Robots Elements -->
@@ -68,5 +69,5 @@
 	</xacro:motor_wheel>
   <xacro:both_elevator prefix="$(arg prefix)both_forks" parent="$(arg prefix)base_link" hq="${hq}">
-      <origin xyz="${elevator_x} ${elevator_y} ${elevator_z}" rpy="0 0 0"/>
+      <origin xyz="${elevator_x} ${elevator_y} ${elevator_z+0.05}" rpy="0 0 0"/>
   </xacro:both_elevator>
   <xacro:sensor_sick_s300 prefix="$(arg prefix)front_laser" parent="$(arg prefix)base_link">
@@ -79,9 +80,4 @@
       <origin xyz="${camera_x} ${camera_y} ${camera_z}" rpy="0 0 ${PI}"/>
   </xacro:sensor_r430>
-  <!--gazebo>
-    <plugin name="gazebo_ros_control" filename="libgazebo_ros_control.so">
-      <robotSimType>steer_bot_hardware_gazebo/SteerBotHardwareGazebo</robotSimType>
-    </plugin>
-  </gazebo-->
 	<!-- Gazebo ros control pluggins -->
 	<xacro:ros_control/>

File: hr_recycler_common/hr_recycler_description/urdf/bases/hr_recycler.urdf.xacro (robot description, xacro)
@@ -42,5 +42,5 @@
       <mass value="${base_mass}" />
       <origin xyz="0 0 0" />
-      <box_inertia  m="${base_mass}" x="${base_length}" y="${base_width}" z="${base_height}"/>
+      <box_inertia  m="${base_mass/6.0}" x="${base_length}" y="${base_width}" z="${base_height}"/>
     </inertial>
     <visual>
@@ -60,50 +60,4 @@
     </collision>
   </link>
-  <!-- BASE HELPER! -->
-  <!-- Two small boxes that help the to not tip over -->
-  <joint name="${prefix}base_helper_joint" type="continuous">
-    <origin xyz="-${base_length/2.0+0.3} ${base_width/2.0-wheel_radius/2.0} -${wheel_radius/2.0}" rpy="0 0 0" />
-    <parent link="${prefix}base_link"/>
-    <child link="${prefix}base_helper_link" />
-  </joint>
-  <link name="${prefix}base_helper_link">
-    <!--visual>
-      <origin xyz="0 0 0" rpy="0 0 0" />
-      <geometry>
-         <sphere radius="${wheel_radius/2.0}"/>
-      </geometry>
-       <material name="darkgrey">
-         <color rgba="0.1 0.1 0.1 1"/>
-       </material>
-    </visual-->
-    <collision>
-      <origin xyz="0 0 0" rpy="0 0 0" />
-      <geometry>
-        <sphere radius="${wheel_radius/2.0}"/>
-      </geometry>
-    </collision>
-    </link>
-    <joint name="${prefix}base_helper_2_joint" type="continuous">
-      <origin xyz="-${base_length/2.0+0.3} -${base_width/2.0-wheel_radius/2.0} -${wheel_radius/2.0}" rpy="0 0 0" />
-      <parent link="${prefix}base_link"/>
-      <child link="${prefix}base_helper_2_link" />
-    </joint>
-    <link name="${prefix}base_helper_2_link">
-      <!--visual>
-        <origin xyz="0 0 0" rpy="0 0 0" />
-        <geometry>
-           <box size="${wheel_radius} ${wheel_radius} ${wheel_radius}"/>
-        </geometry>
-         <material name="darkgrey">
-           <color rgba="0.1 0.1 0.1 1"/>
-         </material>
-      </visual-->
-      <collision>
-        <origin xyz="0 0 0" rpy="0 0 0" />
-        <geometry>
-          <sphere radius="${wheel_radius/2.0}"/>
-        </geometry>
-      </collision>
-      </link>
   </xacro:macro>
 </robot>

File: hr_recycler_common/hr_recycler_description/urdf/elevator/both_elevator.urdf.xacro (robot description, xacro)
@@ -4,27 +4,19 @@
   <xacro:macro name="both_elevator" params="prefix parent hq *origin" >
     <xacro:property name="fork_length" value="1.176" />
-    <xacro:property name="elevator_x" value="-${base_length/2.0}" />
+    <xacro:property name="elevator_x" value="0.0" />
   	<xacro:property name="elevator_y" value="0.195" />
-  	<xacro:property name="elevator_z" value="0.0" />
+  	<xacro:property name="elevator_z" value="${fork_height}" />
   	<xacro:property name="fork_width" value="0.11" />
-  	<xacro:property name="fork_height" value="0.05" />
+  	<xacro:property name="fork_height" value="0.015" />
   	<xacro:property name="fork_mass" value="10.0" />
-    <joint name="${prefix}_both_elevator_joint" type="prismatic">
+    <xacro:property name="fork_separation" value="0.116" />
+    <xacro:property name="fork_x" value="0.0" />
+    <xacro:property name="fork_y" value="0.195" />
+    <xacro:property name="fork_z" value="0.0" />
+    <joint name="${prefix}_both_elevator_joint" type="fixed">
         <xacro:insert_block name="origin" />
         <parent link="${parent}"/>
         <child link="${prefix}_platform_link" />
-        <axis xyz="0 0 1"/>
-        <limit effort="1000.0" lower="0.0" upper="0.25" velocity="1.0"/>
     </joint>
-    <transmission name="${prefix}both_elevator_transmission">
-      <type>transmission_interface/SimpleTransmission</type>
-      <joint name="${prefix}_both_elevator_joint">
-        <hardwareInterface>hardware_interface/PositionJointInterface</hardwareInterface>
-      </joint>
-      <actuator name="${prefix}_both_elevator_motor">
-        <hardwareInterface>hardware_interface/PositionActuatorInterface</hardwareInterface>
-        <mechanicalReduction>${traction_mechanical_reduction}</mechanicalReduction>
-      </actuator>
-    </transmission>
     <link name="${prefix}_platform_link">
       <inertial>
@@ -35,9 +27,105 @@
     </link>
     <xacro:elevator_platform prefix="$(arg prefix)left_fork" parent="${prefix}_platform_link" hq="${hq}">
-        <origin xyz="0 ${elevator_y} -0.02" rpy="0 0 0"/>
+        <origin xyz="${fork_x} ${fork_y} ${fork_z}" rpy="0 0 0"/>
     </xacro:elevator_platform>
     <xacro:elevator_platform prefix="$(arg prefix)right_fork" parent="${prefix}_platform_link" hq="${hq}">
-        <origin xyz="0 -${elevator_y} -0.02" rpy="0 0 0"/>
+        <origin xyz="${fork_x} -${fork_y} ${fork_z}" rpy="0 0 0"/>
     </xacro:elevator_platform>
+    <joint name="${prefix}_prismatic_both_forks_joint" type="prismatic">
+         <origin xyz="0 0 0" rpy="0 0 0"/>
+         <parent link="${prefix}_platform_link"/>
+         <child link="${prefix}_prismatic_forks_link" />
+         <axis xyz="0 0 1"/>
+         <limit effort="1000.0" lower="0.0" upper="0.25" velocity="1"/>
+     </joint>
+     <transmission name="${prefix}_prismatic_both_forks_joint_transmission">
+       <type>transmission_interface/SimpleTransmission</type>
+       <joint name="${prefix}_prismatic_both_forks_joint">
+         <hardwareInterface>hardware_interface/PositionJointInterface</hardwareInterface>
+       </joint>
+       <actuator name="${prefix}_prismatic_both_forks_joint_motor">
+         <hardwareInterface>hardware_interface/PositionActuatorInterface</hardwareInterface>
+         <mechanicalReduction>${traction_mechanical_reduction}</mechanicalReduction>
+       </actuator>
+     </transmission>
+     <link name="${prefix}_prismatic_forks_link">
+       <inertial>
+         <mass value="${fork_mass}" />
+         <origin xyz="0 0 1" />
+         <solid_cuboid_inertia m="${fork_mass/2.0}" h="${fork_height}" d="${fork_length}" w="${fork_width}"/>
+       </inertial>
+     </link>
+     <joint name="${prefix}_prismatic_left_fork_joint" type="fixed">
+         <origin xyz="${elevator_x} ${elevator_y} ${elevator_z}" rpy="0 0 0"/>
+         <parent link="${prefix}_prismatic_forks_link"/>
+         <child link="${prefix}_prismatic_left_fork" />
+     </joint>
+     <link name="${prefix}_prismatic_left_fork">
+       <visual>
+         <origin xyz="-${fork_length/2} 0 0" rpy="0 0 0" />
+         <xacro:if value="${hq}">
+           <geometry>
+             <!--mesh filename="package://hr_recycler_description/meshes/elevator/hr_recycler_elevator.dae"/-->
+             <box size="${fork_length} ${fork_width} ${fork_height}"/>
+           </geometry>
+         </xacro:if>
+         <xacro:unless value="${hq}">
+           <geometry>
+             <!--mesh filename="package://hr_recycler_description/meshes/elevator/hr_recycler_elevator.stl"/-->
+             <box size="${fork_length} ${fork_width} ${fork_height}"/>
+           </geometry>
+         </xacro:unless>
+         <material name="black">
+           <color rgba="0.0 0.0 0.0 1"/>
+         </material>
+       </visual>
+       <collision>
+         <origin xyz="-${fork_length/2} 0 0" rpy="0 0 0" />
+         <geometry>
+           <box size="${fork_length} ${fork_width} ${fork_height}"/>
+         </geometry>
+       </collision>
+       <inertial>
+         <mass value="${fork_mass}" />
+         <origin xyz="-1 0 0" />
+         <solid_cuboid_inertia m="${fork_mass}" h="${fork_height}" d="${fork_length}" w="${fork_width}"/>
+       </inertial>
+     </link>
+     <joint name="${prefix}_prismatic_right_fork_joint" type="fixed">
+         <origin xyz="${elevator_x} -${elevator_y} ${elevator_z}" rpy="0 0 0"/>
+         <parent link="${prefix}_prismatic_forks_link"/>
+         <child link="${prefix}_prismatic_right_fork" />
+     </joint>
+     <link name="${prefix}_prismatic_right_fork">
+       <visual>
+         <origin xyz="-${fork_length/2} 0 0" rpy="0 0 0" />
+         <xacro:if value="${hq}">
+           <geometry>
+             <!--mesh filename="package://hr_recycler_description/meshes/elevator/hr_recycler_elevator.dae"/-->
+             <box size="${fork_length} ${fork_width} ${fork_height}"/>
+           </geometry>
+         </xacro:if>
+         <xacro:unless value="${hq}">
+           <geometry>
+             <!--mesh filename="package://hr_recycler_description/meshes/elevator/hr_recycler_elevator.stl"/-->
+             <box size="${fork_length} ${fork_width} ${fork_height}"/>
+           </geometry>
+         </xacro:unless>
+         <material name="black">
+           <color rgba="0.0 0.0 0.0 1"/>
+         </material>
+       </visual>
+       <collision>
+         <origin xyz="-${fork_length/2} 0 0" rpy="0 0 0" />
+         <geometry>
+           <box size="${fork_length} ${fork_width} ${fork_height}"/>
+         </geometry>
+       </collision>
+       <inertial>
+         <mass value="${fork_mass}" />
+         <origin xyz="-1 0 0" />
+         <solid_cuboid_inertia m="${fork_mass}" h="${fork_height}" d="${fork_length}" w="${fork_width}"/>
+       </inertial>
+     </link>
   </xacro:macro>
 </robot>

File: hr_recycler_common/hr_recycler_description/urdf/elevator/elevator.urdf.xacro (robot description, xacro)
@@ -1,18 +1,16 @@
 <?xml version="1.0"?>
 <robot xmlns:xacro="http://www.ros.org/wiki/xacro">
-	<xacro:include filename="$(find hr_recycler_description)/urdf/elevator/elevator.transmission.xacro"/>
-	<xacro:include filename="$(find hr_recycler_description)/urdf/elevator/elevator.gazebo.xacro"/>
 	<xacro:macro name="elevator_platform" params="prefix parent hq *origin">
 	<xacro:property name="fork_length" value="1.176" />
 	<xacro:property name="fork_width" value="0.11" />
-	<xacro:property name="fork_height" value="0.03" />
-	<xacro:property name="fork_mass" value="25.0" />
+	<xacro:property name="fork_height" value="0.015" />
+	<xacro:property name="fork_mass" value="10.0" />
 	<xacro:property name="fork_separation" value="0.116" />
-	<xacro:property name="support_wheel_radius" value="${wheel_radius/2.0-fork_height/2.0}" />
+	<xacro:property name="support_wheel_radius" value="${wheel_radius/4.0}" />
 	<xacro:property name="support_wheel_length" value="${fork_width}" />
-  <xacro:property name="support_wheel_mass" value="5.0" />
+  <xacro:property name="support_wheel_mass" value="10.0" />
 	<xacro:property name="support_wheel_joint_x" value="${0.16-fork_length}" />
 	<xacro:property name="support_wheel_joint_y" value="0.0" />
-	<xacro:property name="support_wheel_joint_z" value="-${wheel_radius/2.0+fork_height/4.0}" />
+	<xacro:property name="support_wheel_joint_z" value="-${fork_height/2.0+support_wheel_radius}" />
 	<!-- PARAMS: -->
 	<!-- name : name of the link: -->
@@ -56,21 +54,28 @@
 				<box size="${fork_length} ${fork_width} ${fork_height}"/>
 			</geometry>
-			<!--geometry>
-					<mesh filename="package://hr_recycler_description/meshes/elevator/hr_recycler_elevator.dae"/>
-				</geometry-->
 		</collision>
 		<inertial>
 			<mass value="${fork_mass}" />
-			<origin xyz="0 0 -0.27" />
+			<origin xyz="-${fork_length} 0 0" />
 			<solid_cuboid_inertia m="${fork_mass}" h="${fork_height}" d="${fork_length}" w="${fork_width}"/>
 		</inertial>
 	</link>
 	<joint name="${prefix}_support_wheel_joint" type="continuous">
-			<origin xyz="${support_wheel_joint_x} ${support_wheel_joint_y} ${support_wheel_joint_z}" rpy="0 0 0"/>
+ 			<origin xyz="${support_wheel_joint_x} ${support_wheel_joint_y} ${support_wheel_joint_z-0.05}" rpy="0 0 0"/>
 			<parent link="${prefix}_platform_link"/>
 			<child link="${prefix}_support_wheel_link" />
-			<limit effort="1000.0" velocity="1.0"/>
+			<limit effort="1000.0" velocity="100.0"/>
 			<axis xyz="0 1 0" rpy="0 0 0" />
 	</joint>
+	<!--transmission name="${prefix}_support_wheel_joint_transmission">
+		<type>transmission_interface/SimpleTransmission</type>
+		<joint name="${prefix}_support_wheel_joint">
+			<hardwareInterface>hardware_interface/VelocityJointInterface</hardwareInterface>
+		</joint>
+		<actuator name="${prefix}_both_elevator_motor">
+			<hardwareInterface>hardware_interface/VelocityActuatorInterface</hardwareInterface>
+			<mechanicalReduction>$1</mechanicalReduction>
+		</actuator>
+	</transmission-->
 	<link name="${prefix}_support_wheel_link">
 		<visual>

File: hr_recycler_common/hr_recycler_description/urdf/wheels/motor_wheel.urdf.xacro (robot description, xacro)
@@ -10,5 +10,5 @@
   <xacro:property name="steer_joint_friction" value="1000.0" />
   <xacro:property name="steer_joint_effort_limit" value="9999.0" />
-  <xacro:property name="steer_joint_velocity_limit" value="2" />
+  <xacro:property name="steer_joint_velocity_limit" value="20" />
   <xacro:property name="steer_mechanical_reduction" value="1.0" />
   <xacro:property name="steer_joint_position_limit" value="1.56" />
@@ -96,4 +96,9 @@
       </inertial>
     </link>
+    <gazebo reference="${prefix}wheel_traction_link">
+      <mu1>2</mu1>
+      <mu2>2</mu2>
+      <material>Gazebo/Black</material>
+    </gazebo>
   </xacro:macro>
 </robot>
