Commit message: Changed some inertia's parameters. Added scaled omni-wheels. Added euro-pallet world.

File: hr_recycler_common/hr_recycler_description/robots/hr_recycler_std.urdf.xacro (robot description, xacro)
@@ -23,5 +23,5 @@
 	<xacro:property name="PI" value="3.1415926535897931"/>
 	<!-- Wheel parameters -->
-	<xacro:property name="wheel_offset_x" value="0.0"/>    <!-- x,y,z in translation from base_link to the center of the wheel -->
+	<xacro:property name="wheel_offset_x" value="0.1"/>    <!-- x,y,z in translation from base_link to the center of the wheel -->
 	<xacro:property name="wheel_offset_y" value="0.0"/>
 	<xacro:property name="wheel_offset_z" value="${wheel_radius}"/>
@@ -69,5 +69,5 @@
 	</xacro:motor_wheel>
   <xacro:both_elevator prefix="$(arg prefix)both_forks" parent="$(arg prefix)base_link" hq="${hq}">
-      <origin xyz="${elevator_x} ${elevator_y} ${elevator_z+0.05}" rpy="0 0 0"/>
+      <origin xyz="${elevator_x} ${elevator_y} ${elevator_z+0.01}" rpy="0 0 0"/>
   </xacro:both_elevator>
   <xacro:sensor_sick_s300 prefix="$(arg prefix)front_laser" parent="$(arg prefix)base_link">

File: hr_recycler_common/hr_recycler_description/urdf/bases/hr_recycler.urdf.xacro (robot description, xacro)
@@ -9,5 +9,5 @@
   <xacro:property name="base_width" value="0.754" />
   <xacro:property name="base_height" value="0.533" />
-  <xacro:property name="base_mass" value="25.0"/>
+  <xacro:property name="base_mass" value="2"/>
   <xacro:property name="visual_base_link_z" value="${wheel_radius+base_height/2.0+separation_wheel_box}" />
   <xacro:property name="fork_length" value="1.176" />
@@ -41,6 +41,7 @@
     <inertial>
       <mass value="${base_mass}" />
-      <origin xyz="0 0 0" />
-      <box_inertia  m="${base_mass/6.0}" x="${base_length}" y="${base_width}" z="${base_height}"/>
+      <origin xyz="0 0 -${wheel_radius}" />
+      <!--box_inertia  m="${base_mass}" x="${base_length}" y="${base_width}" z="${base_height}"/-->
+      <box_inertia  m="${base_mass}" x="0.005" y="0.005" z="0.005"/>
     </inertial>
     <visual>

File: hr_recycler_common/hr_recycler_description/urdf/common.gazebo.xacro (robot description, xacro)
@@ -9,4 +9,5 @@
         <controlPeriod>0.001</controlPeriod>
 	    <robotSimType>gazebo_ros_control/DefaultRobotHWSim</robotSimType>
+			<legacyModeNS>true</legacyModeNS>
       </plugin>
    </gazebo>

File: hr_recycler_common/hr_recycler_description/urdf/elevator/both_elevator.urdf.xacro (robot description, xacro)
@@ -9,5 +9,5 @@
   	<xacro:property name="fork_width" value="0.11" />
   	<xacro:property name="fork_height" value="0.015" />
-  	<xacro:property name="fork_mass" value="10.0" />
+  	<xacro:property name="fork_mass" value="1.0" />
     <xacro:property name="fork_separation" value="0.116" />
     <xacro:property name="fork_x" value="0.0" />
@@ -23,5 +23,5 @@
         <mass value="1" />
         <origin xyz="0 0 0" />
-        <cylinder_inertia m="1" r="1" h="1" />
+        <cylinder_inertia m="7" r="1" h="1" />
       </inertial>
     </link>

File: hr_recycler_common/hr_recycler_description/urdf/elevator/elevator.urdf.xacro (robot description, xacro)
@@ -1,13 +1,14 @@
 <?xml version="1.0"?>
 <robot xmlns:xacro="http://www.ros.org/wiki/xacro">
+	<xacro:include filename="$(find hr_recycler_description)/urdf/wheels/omni_wheel.urdf.xacro" />
 	<xacro:macro name="elevator_platform" params="prefix parent hq *origin">
 	<xacro:property name="fork_length" value="1.176" />
 	<xacro:property name="fork_width" value="0.11" />
 	<xacro:property name="fork_height" value="0.015" />
-	<xacro:property name="fork_mass" value="10.0" />
+	<xacro:property name="fork_mass" value="2.0" />
 	<xacro:property name="fork_separation" value="0.116" />
 	<xacro:property name="support_wheel_radius" value="${wheel_radius/4.0}" />
 	<xacro:property name="support_wheel_length" value="${fork_width}" />
-  <xacro:property name="support_wheel_mass" value="10.0" />
+  <xacro:property name="support_wheel_mass" value="2.0" />
 	<xacro:property name="support_wheel_joint_x" value="${0.16-fork_length}" />
 	<xacro:property name="support_wheel_joint_y" value="0.0" />
@@ -61,12 +62,15 @@
 		</inertial>
 	</link>
-	<joint name="${prefix}_support_wheel_joint" type="continuous">
- 			<origin xyz="${support_wheel_joint_x} ${support_wheel_joint_y} ${support_wheel_joint_z-0.05}" rpy="0 0 0"/>
+	<xacro:omni_wheel prefix="${prefix}omni" parent="${prefix}_platform_link" hq="${hq}">
+			<origin xyz="${support_wheel_joint_x} ${support_wheel_joint_y} ${support_wheel_joint_z-0.01}" rpy="0 0 0"/>
+	</xacro:omni_wheel>
+	<!--joint name="${prefix}_support_wheel_joint" type="continuous">
+ 			<origin xyz="${support_wheel_joint_x} ${support_wheel_joint_y} ${support_wheel_joint_z-0.01}" rpy="0 0 0"/>
 			<parent link="${prefix}_platform_link"/>
 			<child link="${prefix}_support_wheel_link" />
 			<limit effort="1000.0" velocity="100.0"/>
-			<axis xyz="0 1 0" rpy="0 0 0" />
+			<axis xyz="0 -1 0" rpy="0 0 0" />
 	</joint>
-	<!--transmission name="${prefix}_support_wheel_joint_transmission">
+	<transmission name="${prefix}_support_wheel_joint_transmission">
 		<type>transmission_interface/SimpleTransmission</type>
 		<joint name="${prefix}_support_wheel_joint">
@@ -77,8 +81,8 @@
 			<mechanicalReduction>$1</mechanicalReduction>
 		</actuator>
-	</transmission-->
+	</transmission>
 	<link name="${prefix}_support_wheel_link">
 		<visual>
-				<origin xyz="0 0 0.01" rpy="${M_PI/2} 0 0" />
+				<origin xyz="0 0 0" rpy="${M_PI/2} 0 0" />
 				<geometry>
 					<cylinder radius="${support_wheel_radius}" length="${support_wheel_length}"/>
@@ -86,5 +90,5 @@
 		</visual>
 		<collision>
-			<origin xyz="0 0 +0.01" rpy="${M_PI/2} 0 0" />
+			<origin xyz="0 0 0" rpy="${M_PI/2} 0 0" />
 			<geometry>
 				<cylinder radius="${support_wheel_radius}" length="${support_wheel_length}"/>
@@ -96,5 +100,5 @@
 			<cylinder_inertia m="${support_wheel_mass}" r="${support_wheel_length}" h="${support_wheel_length}" />
 		</inertial>
-	</link>
+	</link-->
 	<!--xacro:elevator_transmission prefix="${prefix}" /-->
 	<!--xacro:elevator_gazebo prefix="${prefix}" /-->

File: hr_recycler_common/hr_recycler_description/urdf/wheels/motor_wheel.urdf.xacro (robot description, xacro)
@@ -5,5 +5,5 @@
   <xacro:property name="wheel_radius" value="0.1" />
   <xacro:property name="wheel_height" value="0.14" />
-  <xacro:property name="wheel_mass" value="5.0" />
+  <xacro:property name="wheel_mass" value="4.0" />
   <!-- in kg-->
   <xacro:property name="steer_joint_damping" value="2000.0" />
@@ -16,5 +16,6 @@
   <xacro:property name="traction_joint_friction" value="1000.0" />
   <xacro:property name="traction_joint_effort_limit" value="100000.0" />
-  <xacro:property name="traction_joint_velocity_limit" value="6.28" />
+  <xacro:property name="traction_joint_velocity_limit" value="100" />
+  <!--xacro:property name="traction_joint_velocity_limit" value="6.28" /-->
   <xacro:property name="traction_mechanical_reduction" value="1.0" />
   <xacro:property name="traction_joint_position_limit" value="1000.0" />
@@ -97,5 +98,5 @@
     </link>
     <gazebo reference="${prefix}wheel_traction_link">
-      <mu1>2</mu1>
+      <mu1>3</mu1>
       <mu2>2</mu2>
       <material>Gazebo/Black</material>

File: hr_recycler_common/hr_recycler_description/urdf/wheels/omni_wheel.urdf.xacro (robot description, xacro)
@@ -28,5 +28,5 @@
           <origin xyz="0 0 0" rpy="0 0 0" />
           <geometry>
-				    <mesh filename="package://hr_recycler_description/meshes/wheels/hr_recycler_omni_wheel_fake.dae" />
+				    <mesh filename="package://hr_recycler_description/meshes/wheels/hr_recycler_omni_wheel_fake.dae" scale="0.5 0.6 0.5"/>
           </geometry>
         </xacro:if>
@@ -42,5 +42,5 @@
       <origin xyz="0 0 0" rpy="${M_PI/2} 0 0" />
       <geometry>
-         <sphere radius="${omni_wheel_radius}"/>
+         <sphere radius="${omni_wheel_radius*0.35}"/>
       </geometry>
       <surface>
