Commit message: Sim works well ( ͡❛ ‿っ ͡❛) At this point, xacros should be well defined.

File: hr_recycler_common/hr_recycler_description/robots/hr_recycler_std.urdf.xacro (robot description, xacro)
@@ -8,20 +8,16 @@
   <xacro:include filename="$(find hr_recycler_description)/urdf/bases/hr_recycler.urdf.xacro" />
 	<!-- Import HR-RECYCLER wheels -->
-	<xacro:include filename="$(find hr_recycler_description)/urdf/wheels/rubber_wheel.urdf.xacro" />
-	<xacro:include filename="$(find hr_recycler_description)/urdf/wheels/omni_wheel.urdf.xacro" />
 	<xacro:include filename="$(find hr_recycler_description)/urdf/wheels/motor_wheel.urdf.xacro" />
   <!-- Import HR-RECYCLER elevator -->
-	<xacro:include filename="$(find hr_recycler_description)/urdf/elevator/elevator.urdf.xacro" />
   <xacro:include filename="$(find hr_recycler_description)/urdf/elevator/both_elevator.urdf.xacro" />
-	<!-- Import all available sensors -->
+	<!-- Import sensors -->
 	<xacro:include filename="$(find robotnik_sensors)/urdf/all_sensors.urdf.xacro" />
-    <!-- Import Gazebo Stuff -->
+  <!-- Import Gazebo Stuff -->
   <xacro:include filename="$(find hr_recycler_description)/urdf/common.gazebo.xacro" />
-	<!-- ***************** -->
 	<!-- Global parameters -->
-	<!-- ***************** -->
 	<xacro:property name="PI" value="3.1415926535897931"/>
 	<!-- Wheel parameters -->
-	<xacro:property name="wheel_offset_x" value="0.1"/>    <!-- x,y,z in translation from base_link to the center of the wheel -->
+  <!-- x,y,z in translation from base_link to the center of the wheel -->
+	<xacro:property name="wheel_offset_x" value="0.1"/>
 	<xacro:property name="wheel_offset_y" value="0.0"/>
 	<xacro:property name="wheel_offset_z" value="${wheel_radius}"/>
@@ -31,26 +27,16 @@
   <xacro:property name="base_height" value="0.533" />
   <xacro:property name="base_width" value="0.754" />
-	<!-- Castor paramters -->
-	<!--xacro:property name="omni_x" value="0.296"/>
-	<xacro:property name="omni_y" value="0.249"/>
-	<xacro:property name="omni_z" value="0.010"/-->
 	<!-- Flag to select the high or low quality model -->
 	<xacro:property name="hq" value="true" />
-  <!-- ******************* -->
 	<!--  SENSOR PARAMETERS  -->
-	<!-- ******************* -->
   <xacro:property name="sensor_x" value="${base_length/2.0+sensor_length}" />
   <xacro:property name="sensor_y" value="0.0" />
   <xacro:property name="sensor_z" value="${wheel_radius+separation_wheel_box+0.087}" />
   <xacro:property name="sensor_length" value="0.055" />
-  <!-- ******************* -->
 	<!--  CAMERA PARAMETERS  -->
-	<!-- ******************* -->
   <xacro:property name="camera_x" value="-${fork_length+0.025}" />
   <xacro:property name="camera_y" value="0" />
   <xacro:property name="camera_z" value="0" />
-	<!-- ******************* -->
 	<!-- ELEVATOR PARAMETERS -->
-	<!-- ******************* -->
 	<xacro:property name="elevator_x" value="-${base_length/2.0}" />
 	<xacro:property name="elevator_y" value="0.0" />
@@ -62,22 +48,21 @@
 	<!-- *************** -->
 	<!-- Here we create the robot elements using the xacro:macros imported at the beggining of this file -->
-	<!-- HR-RECYCLER base -->
 	<xacro:arg name="prefix" default="hr_recycler_"/>
-	<xacro:hr_recycler prefix="$(arg prefix)" publish_bf="true" hq="${hq}" />
-	<xacro:motor_wheel prefix="$(arg prefix)back" parent="$(arg prefix)base_link" hq="${hq}">
+	<xacro:hr_recycler prefix="$(arg prefix)" publish_bf="true" hq="${hq}" /> <!-- BASE -->
+	<xacro:motor_wheel prefix="$(arg prefix)front_" parent="$(arg prefix)base_link" hq="${hq}"> <!-- WHEEL -->
 			<origin xyz="${wheel_offset_x} ${wheel_offset_y} ${wheel_offset_z}" rpy="0 0 0"/>
 	</xacro:motor_wheel>
-  <xacro:both_elevator prefix="$(arg prefix)both_forks" parent="$(arg prefix)base_link" hq="${hq}">
-      <origin xyz="${elevator_x} ${elevator_y} ${elevator_z+0.01}" rpy="0 0 0"/>
+  <xacro:both_elevator prefix="$(arg prefix)both_forks" parent="$(arg prefix)base_link" hq="${hq}"> <!-- ELEVATOR -->
+      <origin xyz="${elevator_x} ${elevator_y} ${elevator_z}" rpy="0 0 0"/>
   </xacro:both_elevator>
-  <xacro:sensor_sick_s300 prefix="$(arg prefix)front_laser" parent="$(arg prefix)base_link">
+  <xacro:sensor_sick_s300 prefix="$(arg prefix)front_laser" parent="$(arg prefix)base_link"> <!-- FRONT SENSOR -->
       <origin xyz="${sensor_x} ${sensor_y} ${sensor_z}" rpy="${PI} 0 0"/>
   </xacro:sensor_sick_s300>
-  <xacro:sensor_r430 prefix="$(arg prefix)right_fork_camera" parent="$(arg prefix)right_fork_platform_link" prefix_topic="front_right_rgbd_camera">
+  <xacro:sensor_r430 prefix="$(arg prefix)right_fork_camera" parent="$(arg prefix)right_foot_elevator_link" prefix_topic="front_right_rgbd_camera">
       <origin xyz="${camera_x} ${camera_y} ${camera_z}" rpy="0 0 ${PI}"/>
-  </xacro:sensor_r430>
-  <xacro:sensor_r430 prefix="$(arg prefix)left_fork_camera" parent="$(arg prefix)left_fork_platform_link" prefix_topic="front_left_rgbd_camera">
+  </xacro:sensor_r430> <!-- BACK CAMERA -->
+  <xacro:sensor_r430 prefix="$(arg prefix)left_fork_camera" parent="$(arg prefix)left_foot_elevator_link" prefix_topic="front_left_rgbd_camera">
       <origin xyz="${camera_x} ${camera_y} ${camera_z}" rpy="0 0 ${PI}"/>
-  </xacro:sensor_r430>
+  </xacro:sensor_r430> <!-- BACK CAMERA -->
 	<!-- Gazebo ros control pluggins -->
 	<xacro:ros_control/>

File: hr_recycler_common/hr_recycler_description/urdf/bases/hr_recycler.urdf.xacro (robot description, xacro)
@@ -4,5 +4,4 @@
   <!-- Robot mechanical and motor parameters -->
   <xacro:property name="PI" value="3.1415926535897931"/>
-  <xacro:property name="wheel_width" value="0.220" />
   <xacro:property name="wheel_radius" value="0.10" />
   <xacro:property name="base_length" value="0.679" />
@@ -10,10 +9,6 @@
   <xacro:property name="base_height" value="0.2" />
   <xacro:property name="base_mass" value="50"/>
-  <xacro:property name="visual_base_link_z" value="${wheel_radius+base_height/2.0+separation_wheel_box}" />
-  <xacro:property name="fork_length" value="1.176" />
-  <xacro:property name="fork_width" value="0.11" />
-  <xacro:property name="fork_height" value="0.05" />
-  <xacro:property name="fork_separation" value="0.116" />
-  <xacro:property name="separation_wheel_box" value="0.08" />
+  <xacro:property name="base_link_height" value="${wheel_radius+base_height/2.0+separation_wheel_box}" />
+  <xacro:property name="separation_wheel_box" value="0.07" />
   <xacro:macro name="box_inertia" params="m x y z">
     <inertia  ixx="${m*(y*y+z*z)/12}" ixy = "0" ixz = "0"
@@ -22,28 +17,26 @@
   </xacro:macro>
   <!-- BASE FOOTPRINT -->
-  <xacro:if value="${publish_bf}">
-    <link name="${prefix}base_footprint">
-      <visual>
-          <origin xyz="0 0 0" rpy="0 0 0" />
-          <geometry>
-             <box size="0.001 0.001 0.001" />
-          </geometry>
-      </visual>
-    </link>
-    <joint name="${prefix}base_footprint_joint" type="fixed">
-      <origin xyz="0 0 ${wheel_radius}" rpy="0 0 0" />
-      <parent link="${prefix}base_footprint"/>
-      <child link="${prefix}base_link" />
-    </joint>
-  </xacro:if>
-  <!-- BASE_LINK -->
+  <link name="${prefix}base_footprint">
+    <visual>
+      <origin xyz="0 0 0" rpy="0 0 0" />
+      <geometry>
+         <box size="0.001 0.001 0.001" />
+      </geometry>
+    </visual>
+  </link>
+  <joint name="${prefix}base_footprint_joint" type="fixed">
+    <origin xyz="0 0 0" rpy="0 0 0" />
+    <parent link="${prefix}base_footprint"/>
+    <child link="${prefix}base_link" />
+  </joint>
+  <!-- BASE LINK -->
   <link name="${prefix}base_link">
     <inertial>
       <mass value="${base_mass}" />
-      <origin xyz="0 0 -${wheel_radius}" />
+      <origin xyz="0 0 -${wheel_radius}" /><!-- Base_link's inertia origin ->  base_footprint -->
       <box_inertia  m="${base_mass}" x="${base_length}" y="${base_width}" z="${base_height}"/>
     </inertial>
     <visual>
-      <origin xyz="0 0 ${visual_base_link_z}" rpy="0 0 0" />
+      <origin xyz="0 0 ${base_link_height}" rpy="0 0 0" />
       <geometry>
 	       <box size="${base_length} ${base_width} ${base_height}"/>
@@ -54,5 +47,5 @@
     </visual>
     <collision>
-      <origin xyz="0 0 ${visual_base_link_z}" rpy="0 0 0" />
+      <origin xyz="0 0 ${base_link_height}" rpy="0 0 0" />
       <geometry>
 	       <box size="${base_length} ${base_width} ${base_height}"/>

File: hr_recycler_common/hr_recycler_description/urdf/elevator/both_elevator.urdf.xacro (robot description, xacro)
@@ -1,23 +1,84 @@
 <?xml version="1.0"?>
 <robot xmlns:xacro="http://www.ros.org/wiki/xacro">
-  <xacro:include filename="$(find hr_recycler_description)/urdf/elevator/elevator.urdf.xacro"/>
+  <xacro:include filename="$(find hr_recycler_description)/urdf/wheels/omni_wheel.urdf.xacro" />
+  <!-- Fork measurements -->
+  <xacro:property name="fork_length" value="1.176" />
+	<xacro:property name="fork_width" value="0.11" />
+	<xacro:property name="fork_height" value="0.015" />
+	<xacro:property name="fork_mass" value="2.0" />
+  <!-- Fork positions -->
+  <xacro:property name="fork_x" value="0.0" />
+  <xacro:property name="fork_y" value="0.195" />
+  <xacro:property name="upper_fork_z" value="${fork_height}" />
+  <xacro:property name="lower_fork_z" value="0.0" />
+  <xacro:property name="visual_fork_position" value="-${fork_length/2}" />
+  <!-- Support wheel measurements -->
+  <xacro:property name="support_wheel_radius" value="${wheel_radius/4.0}" />
+  <xacro:property name="support_wheel_length" value="${fork_width}" />
+  <xacro:property name="support_wheel_mass" value="2.0" />
+  <!-- Support wheel position -->
+  <xacro:property name="support_wheel_joint_x" value="${0.16-fork_length}" />
+  <xacro:property name="support_wheel_joint_y" value="0.0" />
+  <xacro:property name="support_wheel_joint_z" value="-${fork_height/2.0+support_wheel_radius}" />
+  <!-- Limit elevator -->
+  <xacro:property name="upper_limit_elevator" value="0.25" />
+  <!-- Inertial equation depending of forms -->
+  <xacro:macro name="solid_cuboid_inertia" params="m h d w">
+   <inertia  ixx="${(m*(h*h+d*d))/12}" ixy = "0" ixz = "0"
+             iyy="${(m*(w*w+d*d))/12}" iyz = "0"
+             izz="${(m*(w*w+h*h))/12}"
+    />
+  </xacro:macro>
+  <!-- Platform is divided into two parts: TOP PLATFORM with a prismatic
+   joint, BELOW PLATFORM which has the two support wheels.-->
+  <!-- ************ -->
+  <!-- TOP PLATFORM -->
+  <!-- ************ -->
+  <xacro:macro name="elevator_platform" params="prefix parent hq *origin">
+  	<joint name="${prefix}_foot_elevator_joint" type="fixed">
+  			<xacro:insert_block name="origin" />
+  			<parent link="${parent}"/>
+  			<child link="${prefix}_foot_elevator_link" />
+  	</joint>
+    <!--Fork -->
+  	<link name="${prefix}_foot_elevator_link">
+  		<visual>
+  			<origin xyz="${visual_fork_position} 0 0" rpy="0 0 0" />
+  			<geometry>
+  				<!--mesh filename="package://hr_recycler_description/meshes/elevator/hr_recycler_elevator.dae"/-->
+  				<box size="${fork_length} ${fork_width} ${fork_height}"/>
+  			</geometry>
+  			<material name="black">
+  				<color rgba="0.0 0.0 0.0 1"/>
+  			</material>
+  		</visual>
+  		<collision>
+  			<origin xyz="${visual_fork_position} 0 0" rpy="0 0 0" />
+  			<geometry>
+  				<box size="${fork_length} ${fork_width} ${fork_height}"/>
+  			</geometry>
+  		</collision>
+  		<inertial>
+  			<mass value="${fork_mass}" />
+  			<origin xyz="-${fork_length} 0 0" />
+  			<solid_cuboid_inertia m="${fork_mass}" h="${fork_height}" d="${fork_length}" w="${fork_width}"/>
+  		</inertial>
+  	</link>
+    <!-- Support wheel -->
+  	<xacro:omni_wheel prefix="${prefix}_omni" parent="${prefix}_foot_elevator_link" hq="${hq}">
+  			<origin xyz="${support_wheel_joint_x} ${support_wheel_joint_y} ${support_wheel_joint_z}" rpy="0 0 0"/>
+  	</xacro:omni_wheel>
+  </xacro:macro>
+  <!-- ************** -->
+  <!-- BELOW PLATFORM -->
+  <!-- ************** -->
   <xacro:macro name="both_elevator" params="prefix parent hq *origin" >
-    <xacro:property name="fork_length" value="1.176" />
-    <xacro:property name="elevator_x" value="0.0" />
-  	<xacro:property name="elevator_y" value="0.195" />
-  	<xacro:property name="elevator_z" value="${fork_height}" />
-  	<xacro:property name="fork_width" value="0.11" />
-  	<xacro:property name="fork_height" value="0.015" />
-  	<xacro:property name="fork_mass" value="1.0" />
-    <xacro:property name="fork_separation" value="0.116" />
-    <xacro:property name="fork_x" value="0.0" />
-    <xacro:property name="fork_y" value="0.195" />
-    <xacro:property name="fork_z" value="0.0" />
-    <joint name="${prefix}_both_elevator_joint" type="fixed">
+    <joint name="${prefix}_base_elevator_joint" type="fixed">
         <xacro:insert_block name="origin" />
         <parent link="${parent}"/>
-        <child link="${prefix}_platform_link" />
+        <child link="${prefix}_base_elevator_link" />
     </joint>
-    <link name="${prefix}_platform_link">
+    <!-- This piece supports the two lower forks -->
+    <link name="${prefix}_base_elevator_link">
       <inertial>
         <mass value="1" />
@@ -26,54 +87,38 @@
       </inertial>
     </link>
-    <xacro:elevator_platform prefix="$(arg prefix)left_fork" parent="${prefix}_platform_link" hq="${hq}">
-        <origin xyz="${fork_x} ${fork_y} ${fork_z}" rpy="0 0 0"/>
+    <!-- Called two lower forks -->
+    <xacro:elevator_platform prefix="$(arg prefix)left" parent="${prefix}_base_elevator_link" hq="${hq}">
+        <origin xyz="${fork_x} ${fork_y} ${lower_fork_z}" rpy="0 0 0"/>
     </xacro:elevator_platform>
-    <xacro:elevator_platform prefix="$(arg prefix)right_fork" parent="${prefix}_platform_link" hq="${hq}">
-        <origin xyz="${fork_x} -${fork_y} ${fork_z}" rpy="0 0 0"/>
+    <xacro:elevator_platform prefix="$(arg prefix)right" parent="${prefix}_base_elevator_link" hq="${hq}">
+        <origin xyz="${fork_x} -${fork_y} ${lower_fork_z}" rpy="0 0 0"/>
     </xacro:elevator_platform>
-    <joint name="${prefix}_prismatic_both_forks_joint" type="prismatic">
+    <joint name="${prefix}_elevator_joint" type="prismatic">
          <origin xyz="0 0 0" rpy="0 0 0"/>
-         <parent link="${prefix}_platform_link"/>
-         <child link="${prefix}_prismatic_forks_link" />
+         <parent link="${prefix}_base_elevator_link"/>
+         <child link="${prefix}_elevator_link" />
          <axis xyz="0 0 1"/>
-         <limit effort="1000.0" lower="0.0" upper="0.25" velocity="1"/>
+         <limit effort="1000.0" lower="0.0" upper="${upper_limit_elevator}" velocity="1"/>
      </joint>
-     <transmission name="${prefix}_prismatic_both_forks_joint_transmission">
-       <type>transmission_interface/SimpleTransmission</type>
-       <joint name="${prefix}_prismatic_both_forks_joint">
-         <hardwareInterface>hardware_interface/PositionJointInterface</hardwareInterface>
-       </joint>
-       <actuator name="${prefix}_prismatic_both_forks_joint_motor">
-         <hardwareInterface>hardware_interface/PositionActuatorInterface</hardwareInterface>
-         <mechanicalReduction>${traction_mechanical_reduction}</mechanicalReduction>
-       </actuator>
-     </transmission>
-     <link name="${prefix}_prismatic_forks_link">
+     <!-- This piece holds the forks that are going to be elevated -->
+     <link name="${prefix}_elevator_link">
        <inertial>
          <mass value="${fork_mass}" />
          <origin xyz="0 0 1" />
-         <solid_cuboid_inertia m="${fork_mass/2.0}" h="${fork_height}" d="${fork_length}" w="${fork_width}"/>
+         <solid_cuboid_inertia m="${fork_mass}" h="${fork_height}" d="${fork_length}" w="${fork_width}"/>
        </inertial>
      </link>
-     <joint name="${prefix}_prismatic_left_fork_joint" type="fixed">
-         <origin xyz="${elevator_x} ${elevator_y} ${elevator_z}" rpy="0 0 0"/>
-         <parent link="${prefix}_prismatic_forks_link"/>
-         <child link="${prefix}_prismatic_left_fork" />
+     <joint name="${prefix}_left_fork_joint" type="fixed">
+         <origin xyz="${fork_x} ${fork_y} ${upper_fork_z}" rpy="0 0 0"/>
+         <parent link="${prefix}_elevator_link"/>
+         <child link="${prefix}_left_fork" />
      </joint>
-     <link name="${prefix}_prismatic_left_fork">
+     <link name="${prefix}_left_fork">
        <visual>
-         <origin xyz="-${fork_length/2} 0 0" rpy="0 0 0" />
-         <xacro:if value="${hq}">
-           <geometry>
-             <!--mesh filename="package://hr_recycler_description/meshes/elevator/hr_recycler_elevator.dae"/-->
-             <box size="${fork_length} ${fork_width} ${fork_height}"/>
-           </geometry>
-         </xacro:if>
-         <xacro:unless value="${hq}">
-           <geometry>
-             <!--mesh filename="package://hr_recycler_description/meshes/elevator/hr_recycler_elevator.stl"/-->
-             <box size="${fork_length} ${fork_width} ${fork_height}"/>
-           </geometry>
-         </xacro:unless>
+         <origin xyz="${visual_fork_position} 0 0" rpy="0 0 0" />
+         <geometry>
+          <!--mesh filename="package://hr_recycler_description/meshes/elevator/hr_recycler_elevator.stl"/-->
+           <box size="${fork_length} ${fork_width} ${fork_height}"/>
+         </geometry>
          <material name="black">
            <color rgba="0.0 0.0 0.0 1"/>
@@ -81,5 +126,5 @@
        </visual>
        <collision>
-         <origin xyz="-${fork_length/2} 0 0" rpy="0 0 0" />
+         <origin xyz="${visual_fork_position} 0 0" rpy="0 0 0" />
          <geometry>
            <box size="${fork_length} ${fork_width} ${fork_height}"/>
@@ -92,24 +137,16 @@
        </inertial>
      </link>
-     <joint name="${prefix}_prismatic_right_fork_joint" type="fixed">
-         <origin xyz="${elevator_x} -${elevator_y} ${elevator_z}" rpy="0 0 0"/>
-         <parent link="${prefix}_prismatic_forks_link"/>
-         <child link="${prefix}_prismatic_right_fork" />
+     <joint name="${prefix}_right_fork_joint" type="fixed">
+         <origin xyz="${fork_x} -${fork_y} ${upper_fork_z}" rpy="0 0 0"/>
+         <parent link="${prefix}_elevator_link"/>
+         <child link="${prefix}_right_fork" />
      </joint>
-     <link name="${prefix}_prismatic_right_fork">
+     <link name="${prefix}_right_fork">
        <visual>
-         <origin xyz="-${fork_length/2} 0 0" rpy="0 0 0" />
-         <xacro:if value="${hq}">
-           <geometry>
+         <origin xyz="${visual_fork_position} 0 0" rpy="0 0 0" />
+         <geometry>
              <!--mesh filename="package://hr_recycler_description/meshes/elevator/hr_recycler_elevator.dae"/-->
-             <box size="${fork_length} ${fork_width} ${fork_height}"/>
-           </geometry>
-         </xacro:if>
-         <xacro:unless value="${hq}">
-           <geometry>
-             <!--mesh filename="package://hr_recycler_description/meshes/elevator/hr_recycler_elevator.stl"/-->
-             <box size="${fork_length} ${fork_width} ${fork_height}"/>
-           </geometry>
-         </xacro:unless>
+           <box size="${fork_length} ${fork_width} ${fork_height}"/>
+         </geometry>
          <material name="black">
            <color rgba="0.0 0.0 0.0 1"/>
@@ -117,5 +154,5 @@
        </visual>
        <collision>
-         <origin xyz="-${fork_length/2} 0 0" rpy="0 0 0" />
+         <origin xyz="${visual_fork_position} 0 0" rpy="0 0 0" />
          <geometry>
            <box size="${fork_length} ${fork_width} ${fork_height}"/>
@@ -128,4 +165,17 @@
        </inertial>
      </link>
+    <!-- ************* -->
+    <!-- TRANSMISSIONS -->
+    <!-- ************* -->
+     <transmission name="${prefix}_elevator_joint_transmission">
+       <type>transmission_interface/SimpleTransmission</type>
+       <joint name="${prefix}_elevator_joint">
+         <hardwareInterface>hardware_interface/PositionJointInterface</hardwareInterface>
+       </joint>
+       <actuator name="${prefix}_elevator_joint_motor">
+         <hardwareInterface>hardware_interface/PositionActuatorInterface</hardwareInterface>
+         <mechanicalReduction>${traction_mechanical_reduction}</mechanicalReduction>
+       </actuator>
+     </transmission>
   </xacro:macro>
 </robot>
