Commit message: Added .stl, removed some .stl that never gonna be used, changed the schedule of joints, at this point it's like a new URDF, but it works :D

File: hr_recycler_common/hr_recycler_description/robots/hr_recycler_std.urdf.xacro (robot description, xacro)
@@ -19,5 +19,5 @@
 	<!-- Wheel parameters -->
   <!-- x,y,z in translation from base_link to the center of the wheel -->
-	<xacro:property name="wheel_offset_x" value="0.1"/>
+	<xacro:property name="wheel_offset_x" value="0.0"/>
 	<xacro:property name="wheel_offset_y" value="0.0"/>
 	<xacro:property name="wheel_offset_z" value="${wheel_radius}"/>
@@ -30,12 +30,10 @@
 	<xacro:property name="hq" value="true" />
 	<!--  SENSOR PARAMETERS  -->
-  <xacro:property name="sensor_x" value="${base_length/2.0+sensor_length}" />
-  <xacro:property name="sensor_y" value="0.0" />
-  <xacro:property name="sensor_z" value="${wheel_radius+separation_wheel_box+0.087}" />
   <xacro:property name="sensor_length" value="0.055" />
+  <xacro:property name="sensor" value="0.25294 0 0.200" />
 	<!--  CAMERA PARAMETERS  -->
-  <xacro:property name="camera_x" value="-${fork_length+0.025}" />
-  <xacro:property name="camera_y" value="0" />
-  <xacro:property name="camera_z" value="0" />
+  <xacro:property name="camera_x" value="-1.539" />
+  <xacro:property name="camera_y" value="0.195" />
+  <xacro:property name="camera_z" value="0.067" />
 	<!-- ELEVATOR PARAMETERS -->
 	<xacro:property name="elevator_x" value="-${base_length/2.0}" />
@@ -44,4 +42,5 @@
   <xacro:property name="fork_length" value="1.176" />
   <xacro:property name="fork_height" value="0.015" />
+  <xacro:property name="elevator" value="0 0 0" />
 	<!-- *************** -->
 	<!-- Robots Elements -->
@@ -51,17 +50,18 @@
 	<xacro:hr_recycler prefix="$(arg prefix)" publish_bf="true" hq="${hq}" /> <!-- BASE -->
 	<xacro:motor_wheel prefix="$(arg prefix)front_" parent="$(arg prefix)base_link" hq="${hq}"> <!-- WHEEL -->
-			<origin xyz="${wheel_offset_x} ${wheel_offset_y} ${wheel_offset_z}" rpy="0 0 0"/>
+			<!--origin xyz="${wheel_offset_x} ${wheel_offset_y} ${wheel_offset_z}" rpy="0 0 0"/-->
+      <origin xyz="0 0 0.460" rpy="0 0 0"/>
 	</xacro:motor_wheel>
   <xacro:both_elevator prefix="$(arg prefix)both_forks" parent="$(arg prefix)base_link" hq="${hq}"> <!-- ELEVATOR -->
-      <origin xyz="${elevator_x} ${elevator_y} ${elevator_z}" rpy="0 0 0"/>
+      <origin xyz="${elevator}" rpy="0 0 0"/>
   </xacro:both_elevator>
-  <xacro:sensor_sick_s300 prefix="$(arg prefix)front_laser" parent="$(arg prefix)base_link"> <!-- FRONT SENSOR -->
-      <origin xyz="${sensor_x} ${sensor_y} ${sensor_z}" rpy="${PI} 0 0"/>
+  <xacro:sensor_sick_s300 prefix="$(arg prefix)front_laser" parent="$(arg prefix)base_footprint"> <!-- BACK SENSOR -->
+      <origin xyz="${sensor}" rpy="${PI} 0 0"/>
   </xacro:sensor_sick_s300>
-  <xacro:sensor_r430 prefix="$(arg prefix)right_fork_camera" parent="$(arg prefix)right_foot_elevator_link" prefix_topic="front_right_rgbd_camera">
+  <xacro:sensor_r430 prefix="$(arg prefix)right_fork_camera" parent="$(arg prefix)both_forks_elevator_link" prefix_topic="front_right_rgbd_camera">
       <origin xyz="${camera_x} ${camera_y} ${camera_z}" rpy="0 0 ${PI}"/>
   </xacro:sensor_r430> <!-- BACK CAMERA -->
-  <xacro:sensor_r430 prefix="$(arg prefix)left_fork_camera" parent="$(arg prefix)left_foot_elevator_link" prefix_topic="front_left_rgbd_camera">
-      <origin xyz="${camera_x} ${camera_y} ${camera_z}" rpy="0 0 ${PI}"/>
+  <xacro:sensor_r430 prefix="$(arg prefix)left_fork_camera" parent="$(arg prefix)both_forks_elevator_link" prefix_topic="front_left_rgbd_camera">
+      <origin xyz="${camera_x} -${camera_y} ${camera_z}" rpy="0 0 ${PI}"/>
   </xacro:sensor_r430> <!-- BACK CAMERA -->
 	<!-- Gazebo ros control pluggins -->

File: hr_recycler_common/hr_recycler_description/urdf/bases/hr_recycler.urdf.xacro (robot description, xacro)
@@ -3,5 +3,4 @@
   <xacro:macro name="hr_recycler" params="prefix publish_bf hq">
   <!-- Robot mechanical and motor parameters -->
-  <xacro:property name="PI" value="3.1415926535897931"/>
   <xacro:property name="wheel_radius" value="0.10" />
   <xacro:property name="base_length" value="0.679" />
@@ -9,6 +8,6 @@
   <xacro:property name="base_height" value="0.2" />
   <xacro:property name="base_mass" value="50"/>
-  <xacro:property name="base_link_height" value="${wheel_radius+base_height/2.0+separation_wheel_box}" />
-  <xacro:property name="separation_wheel_box" value="0.07" />
+  <xacro:property name="base_link_origin" value="0 0 0.46" />
+  <!-- Inertial equation -->
   <xacro:macro name="box_inertia" params="m x y z">
     <inertia  ixx="${m*(y*y+z*z)/12}" ixy = "0" ixz = "0"
@@ -18,10 +17,4 @@
   <!-- BASE FOOTPRINT -->
   <link name="${prefix}base_footprint">
-    <visual>
-      <origin xyz="0 0 0" rpy="0 0 0" />
-      <geometry>
-         <box size="0.001 0.001 0.001" />
-      </geometry>
-    </visual>
   </link>
   <joint name="${prefix}base_footprint_joint" type="fixed">
@@ -34,22 +27,19 @@
     <inertial>
       <mass value="${base_mass}" />
-      <origin xyz="0 0 -${wheel_radius}" /><!-- Base_link's inertia origin ->  base_footprint -->
+      <origin xyz="${base_link_origin}" /><!-- Base_link's inertia origin ->  base_footprint -->
       <box_inertia  m="${base_mass}" x="${base_length}" y="${base_width}" z="${base_height}"/>
     </inertial>
     <visual>
-      <origin xyz="0 0 ${base_link_height}" rpy="0 0 0" />
+      <origin xyz="${base_link_origin}" rpy="0 0 0" />
       <geometry>
-	       <box size="${base_length} ${base_width} ${base_height}"/>
+        <mesh filename="package://hr_recycler_description/meshes/wheels/HR_recycler_steer.stl" scale="-1 1 1"/>
       </geometry>
-       <material name="darkgrey">
-         <color rgba="0.1 0.1 0.1 1"/>
-       </material>
     </visual>
-    <collision>
-      <origin xyz="0 0 ${base_link_height}" rpy="0 0 0" />
+    <!--collision>
+      <origin xyz="${base_link_origin}" rpy="0 0 0" />
       <geometry>
-	       <box size="${base_length} ${base_width} ${base_height}"/>
+        <mesh filename="package://hr_recycler_description/meshes/wheels/HR_recycler_steer.stl" scale="-1 1 1"/>
       </geometry>
-    </collision>
+    </collision-->
   </link>
   </xacro:macro>

File: hr_recycler_common/hr_recycler_description/urdf/elevator/both_elevator.urdf.xacro (robot description, xacro)
@@ -10,17 +10,9 @@
   <xacro:property name="fork_x" value="0.0" />
   <xacro:property name="fork_y" value="0.195" />
-  <xacro:property name="upper_fork_z" value="${fork_height}" />
-  <xacro:property name="lower_fork_z" value="0.0" />
-  <xacro:property name="visual_fork_position" value="-${fork_length/2}" />
-  <!-- Support wheel measurements -->
-  <xacro:property name="support_wheel_radius" value="${wheel_radius/4.0}" />
-  <xacro:property name="support_wheel_length" value="${fork_width}" />
-  <xacro:property name="support_wheel_mass" value="2.0" />
+  <xacro:property name="fork_z" value="0.0" />
   <!-- Support wheel position -->
-  <xacro:property name="support_wheel_joint_x" value="${0.16-fork_length}" />
-  <xacro:property name="support_wheel_joint_y" value="0.0" />
-  <xacro:property name="support_wheel_joint_z" value="-${fork_height/2.0+support_wheel_radius}" />
+  <xacro:property name="support_wheel_origin" value="-1.5 0.0 ${wheel_radius/4.0}" />
   <!-- Limit elevator -->
-  <xacro:property name="upper_limit_elevator" value="0.25" />
+  <xacro:property name="upper_limit_elevator" value="0.07" />
   <!-- Inertial equation depending of forms -->
   <xacro:macro name="solid_cuboid_inertia" params="m h d w">
@@ -32,7 +24,7 @@
   <!-- Platform is divided into two parts: TOP PLATFORM with a prismatic
    joint, BELOW PLATFORM which has the two support wheels.-->
-  <!-- ************ -->
-  <!-- TOP PLATFORM -->
-  <!-- ************ -->
+  <!-- ************** -->
+  <!-- BELOW PLATFORM -->
+  <!-- ************** -->
   <xacro:macro name="elevator_platform" params="prefix parent hq *origin">
   	<joint name="${prefix}_foot_elevator_joint" type="fixed">
@@ -41,35 +33,13 @@
   			<child link="${prefix}_foot_elevator_link" />
   	</joint>
-    <!--Fork -->
   	<link name="${prefix}_foot_elevator_link">
-  		<visual>
-  			<origin xyz="${visual_fork_position} 0 0" rpy="0 0 0" />
-  			<geometry>
-  				<!--mesh filename="package://hr_recycler_description/meshes/elevator/hr_recycler_elevator.dae"/-->
-  				<box size="${fork_length} ${fork_width} ${fork_height}"/>
-  			</geometry>
-  			<material name="black">
-  				<color rgba="0.0 0.0 0.0 1"/>
-  			</material>
-  		</visual>
-  		<collision>
-  			<origin xyz="${visual_fork_position} 0 0" rpy="0 0 0" />
-  			<geometry>
-  				<box size="${fork_length} ${fork_width} ${fork_height}"/>
-  			</geometry>
-  		</collision>
-  		<inertial>
-  			<mass value="${fork_mass}" />
-  			<origin xyz="-${fork_length} 0 0" />
-  			<solid_cuboid_inertia m="${fork_mass}" h="${fork_height}" d="${fork_length}" w="${fork_width}"/>
-  		</inertial>
   	</link>
     <!-- Support wheel -->
   	<xacro:omni_wheel prefix="${prefix}_omni" parent="${prefix}_foot_elevator_link" hq="${hq}">
-  			<origin xyz="${support_wheel_joint_x} ${support_wheel_joint_y} ${support_wheel_joint_z}" rpy="0 0 0"/>
+  			<origin xyz="${support_wheel_origin}" rpy="0 0 0"/>
   	</xacro:omni_wheel>
   </xacro:macro>
   <!-- ************** -->
-  <!-- BELOW PLATFORM -->
+  <!--    PLATFORM    -->
   <!-- ************** -->
   <xacro:macro name="both_elevator" params="prefix parent hq *origin" >
@@ -89,15 +59,15 @@
     <!-- Called two lower forks -->
     <xacro:elevator_platform prefix="$(arg prefix)left" parent="${prefix}_base_elevator_link" hq="${hq}">
-        <origin xyz="${fork_x} ${fork_y} ${lower_fork_z}" rpy="0 0 0"/>
+        <origin xyz="${fork_x} ${fork_y} ${fork_z}" rpy="0 0 0"/>
     </xacro:elevator_platform>
     <xacro:elevator_platform prefix="$(arg prefix)right" parent="${prefix}_base_elevator_link" hq="${hq}">
-        <origin xyz="${fork_x} -${fork_y} ${lower_fork_z}" rpy="0 0 0"/>
+        <origin xyz="${fork_x} -${fork_y} ${fork_z}" rpy="0 0 0"/>
     </xacro:elevator_platform>
     <joint name="${prefix}_elevator_joint" type="prismatic">
-         <origin xyz="0 0 0" rpy="0 0 0"/>
-         <parent link="${prefix}_base_elevator_link"/>
-         <child link="${prefix}_elevator_link" />
-         <axis xyz="0 0 1"/>
-         <limit effort="1000.0" lower="0.0" upper="${upper_limit_elevator}" velocity="1"/>
+       <xacro:insert_block name="origin" />
+       <parent link="${parent}"/>
+       <child link="${prefix}_elevator_link" />
+       <axis xyz="0 0 1"/>
+       <limit effort="1000.0" lower="0.0" upper="${upper_limit_elevator}" velocity="1"/>
      </joint>
      <!-- This piece holds the forks that are going to be elevated -->
@@ -108,60 +78,19 @@
          <solid_cuboid_inertia m="${fork_mass}" h="${fork_height}" d="${fork_length}" w="${fork_width}"/>
        </inertial>
-     </link>
-     <joint name="${prefix}_left_fork_joint" type="fixed">
-         <origin xyz="${fork_x} ${fork_y} ${upper_fork_z}" rpy="0 0 0"/>
-         <parent link="${prefix}_elevator_link"/>
-         <child link="${prefix}_left_fork" />
-     </joint>
-     <link name="${prefix}_left_fork">
        <visual>
-         <origin xyz="${visual_fork_position} 0 0" rpy="0 0 0" />
+         <origin xyz="0 0 0.410" rpy="0 0 0" />
          <geometry>
-          <!--mesh filename="package://hr_recycler_description/meshes/elevator/hr_recycler_elevator.stl"/-->
-           <box size="${fork_length} ${fork_width} ${fork_height}"/>
+           <mesh filename="package://hr_recycler_description/meshes/bases/HR_recycler_base_forks.stl" scale="-1 1 1"/>
          </geometry>
-         <material name="black">
-           <color rgba="0.0 0.0 0.0 1"/>
-         </material>
+          <material name="darkgrey">
+            <color rgba="0.1 0.1 0.1 1"/>
+          </material>
        </visual>
        <collision>
-         <origin xyz="${visual_fork_position} 0 0" rpy="0 0 0" />
+         <origin xyz="0 0 0.410" rpy="0 0 0" />
          <geometry>
-           <box size="${fork_length} ${fork_width} ${fork_height}"/>
+           <mesh filename="package://hr_recycler_description/meshes/bases/HR_recycler_base_forks.stl" scale="-1 1 1"/>
          </geometry>
        </collision>
-       <inertial>
-         <mass value="${fork_mass}" />
-         <origin xyz="-1 0 0" />
-         <solid_cuboid_inertia m="${fork_mass}" h="${fork_height}" d="${fork_length}" w="${fork_width}"/>
-       </inertial>
-     </link>
-     <joint name="${prefix}_right_fork_joint" type="fixed">
-         <origin xyz="${fork_x} -${fork_y} ${upper_fork_z}" rpy="0 0 0"/>
-         <parent link="${prefix}_elevator_link"/>
-         <child link="${prefix}_right_fork" />
-     </joint>
-     <link name="${prefix}_right_fork">
-       <visual>
-         <origin xyz="${visual_fork_position} 0 0" rpy="0 0 0" />
-         <geometry>
-             <!--mesh filename="package://hr_recycler_description/meshes/elevator/hr_recycler_elevator.dae"/-->
-           <box size="${fork_length} ${fork_width} ${fork_height}"/>
-         </geometry>
-         <material name="black">
-           <color rgba="0.0 0.0 0.0 1"/>
-         </material>
-       </visual>
-       <collision>
-         <origin xyz="${visual_fork_position} 0 0" rpy="0 0 0" />
-         <geometry>
-           <box size="${fork_length} ${fork_width} ${fork_height}"/>
-         </geometry>
-       </collision>
-       <inertial>
-         <mass value="${fork_mass}" />
-         <origin xyz="-1 0 0" />
-         <solid_cuboid_inertia m="${fork_mass}" h="${fork_height}" d="${fork_length}" w="${fork_width}"/>
-       </inertial>
      </link>
     <!-- ************* -->

File: hr_recycler_common/hr_recycler_description/urdf/wheels/motor_wheel.urdf.xacro (robot description, xacro)
@@ -1,9 +1,7 @@
 <?xml version="1.0"?>
 <robot xmlns:xacro="http://www.ros.org/wiki/xacro">
-  <xacro:property name="M_PI" value="3.1415926535897931" />
   <!-- Wheels -->
-  <xacro:property name="wheel_radius" value="0.1" />
+  <xacro:property name="wheel_radius" value="0.125" />
   <xacro:property name="wheel_width" value="0.1" />
-  <!--xacro:property name="wheel_width" value="0.14" /-->
   <xacro:property name="wheel_mass" value="4.0" /><!-- in kg-->
   <!-- Steer wheel properties -->
@@ -19,7 +17,8 @@
   <xacro:property name="traction_joint_effort_limit" value="100000.0" />
   <xacro:property name="traction_joint_velocity_limit" value="100" />
-  <!--xacro:property name="traction_joint_velocity_limit" value="6.28" -->
   <xacro:property name="traction_mechanical_reduction" value="1.0" />
-  <!-- inertial equation depending of forms -->
+  <xacro:property name="steer_origin" value="0 0 0.460"/>
+  <xacro:property name="traction_origin" value="0 0 -0.335"/>
+  <!-- inertial equation -->
   <xacro:macro name="cylinder_inertia" params="m r h">
     <inertia ixx="${m*(3*r*r+h*h)/12}" ixy = "0" ixz = "0" iyy="${m*(3*r*r+h*h)/12}" iyz = "0" izz="${m*r*r/2}" />
@@ -41,5 +40,5 @@
       <inertial>
         <mass value="${wheel_mass}" />
-        <origin xyz="0 0 0" />
+        <origin xyz="${steer_origin}" />
         <cylinder_inertia m="${wheel_mass}" r="${wheel_width}" h="${wheel_radius}" />
       </inertial>
@@ -49,5 +48,5 @@
       <parent link="${prefix}wheel_steer_link"/>
       <child link="${prefix}wheel_traction_link"/>
-      <origin xyz="0 0 -${wheel_radius}" rpy="0 0 ${M_PI}" />
+      <origin xyz="${traction_origin}" rpy="0 0 0" />
       <axis xyz="0 1 0" rpy="0 0 0" />
       <limit effort="${traction_joint_effort_limit}" velocity="${traction_joint_velocity_limit}" />
@@ -57,25 +56,25 @@
       <visual>
         <xacro:if value="${hq}">
-          <origin xyz="0 0 0" rpy="${M_PI/2} 0 0" />
+          <origin xyz="0 0 -0.125" rpy="0 0 0" />
           <geometry>
-            <cylinder radius="${wheel_radius}" length="${wheel_width}"/>
+            <mesh filename="package://hr_recycler_description/meshes/wheels/HR_recycler_wheel.stl" scale="1 -0.9 1"/>
           </geometry>
         </xacro:if>
         <xacro:unless value="${hq}">
-          <origin xyz="0 0 0" rpy="${M_PI/2} 0 0" />
+          <origin xyz="0 0 -0.125" rpy="0 0 0" />
           <geometry>
-            <cylinder radius="${wheel_radius}" length="${wheel_width}"/>
+            <mesh filename="package://hr_recycler_description/meshes/wheels/HR_recycler_wheel.stl" scale="1 -0.9 1"/>
           </geometry>
         </xacro:unless>
       </visual>
       <collision>
-        <origin xyz="0 0 0" rpy="${M_PI/2} 0 0" />
+        <origin xyz="0 0 -0.125" rpy="0 0 0" />
         <geometry>
-          <cylinder radius="${wheel_radius}" length="${wheel_width}"/>
+          <mesh filename="package://hr_recycler_description/meshes/wheels/HR_recycler_wheel.stl" scale="1 -0.9 1"/>
         </geometry>
       </collision>
       <inertial>
         <mass value="${wheel_mass}" />
-        <origin xyz="0 0 0" />
+        <origin xyz="0 0 0"/>
         <cylinder_inertia m="${wheel_mass}" r="${wheel_radius}" h="${wheel_width}" />
       </inertial>
