Commit message: work towards standarization
- all names and filenames in lowercase
- elevator as a simple element (everything in the same tree)
- simplified names

File: hr_recycler_common/hr_recycler_description/robots/hr_recycler_std.urdf.xacro (robot description, xacro)
@@ -10,5 +10,5 @@
 	<xacro:include filename="$(find hr_recycler_description)/urdf/wheels/motor_wheel.urdf.xacro" />
   <!-- Import HR-RECYCLER elevator -->
-  <xacro:include filename="$(find hr_recycler_description)/urdf/elevator/both_elevator.urdf.xacro" />
+  <xacro:include filename="$(find hr_recycler_description)/urdf/elevator/elevator.urdf.xacro" />
 	<!-- Import sensors -->
 	<xacro:include filename="$(find robotnik_sensors)/urdf/all_sensors.urdf.xacro" />
@@ -53,16 +53,16 @@
       <origin xyz="0 0 0.460" rpy="0 0 0"/>
 	</xacro:motor_wheel>
-  <xacro:both_elevator prefix="$(arg prefix)both_forks" parent="$(arg prefix)base_link" hq="${hq}"> <!-- ELEVATOR -->
-      <origin xyz="${elevator}" rpy="0 0 0"/>
-  </xacro:both_elevator>
-  <xacro:sensor_sick_s300 prefix="$(arg prefix)front_laser" parent="$(arg prefix)base_footprint"> <!-- BACK SENSOR -->
-      <origin xyz="${sensor}" rpy="${PI} 0 0"/>
-  </xacro:sensor_sick_s300>
-  <xacro:sensor_r430 prefix="$(arg prefix)right_fork_camera" parent="$(arg prefix)both_forks_elevator_link" prefix_topic="front_right_rgbd_camera">
-      <origin xyz="${camera_x} ${camera_y} ${camera_z}" rpy="0 0 ${PI}"/>
-  </xacro:sensor_r430> <!-- BACK CAMERA -->
-  <xacro:sensor_r430 prefix="$(arg prefix)left_fork_camera" parent="$(arg prefix)both_forks_elevator_link" prefix_topic="front_left_rgbd_camera">
-      <origin xyz="${camera_x} -${camera_y} ${camera_z}" rpy="0 0 ${PI}"/>
-  </xacro:sensor_r430> <!-- BACK CAMERA -->
+    <xacro:elevator prefix="$(arg prefix)" parent="$(arg prefix)base_link" hq="${hq}"> <!-- ELEVATOR -->
+        <origin xyz="${elevator}" rpy="0 0 0"/>
+    </xacro:elevator>
+    <xacro:sensor_sick_s300 prefix="$(arg prefix)front_laser" parent="$(arg prefix)base_footprint"> <!-- BACK SENSOR -->
+        <origin xyz="${sensor}" rpy="${PI} 0 0"/>
+    </xacro:sensor_sick_s300>
+    <xacro:sensor_r430 prefix="$(arg prefix)right_fork" parent="$(arg prefix)elevator_link" prefix_topic="front_right_rgbd_camera">
+        <origin xyz="${camera_x} ${camera_y} ${camera_z}" rpy="0 0 ${PI}"/>
+    </xacro:sensor_r430>
+    <xacro:sensor_r430 prefix="$(arg prefix)left_fork" parent="$(arg prefix)elevator_link" prefix_topic="front_left_rgbd_camera">
+        <origin xyz="${camera_x} -${camera_y} ${camera_z}" rpy="0 0 ${PI}"/>
+    </xacro:sensor_r430>
 	<!-- Gazebo ros control pluggins -->
 	<xacro:ros_control/>

File: hr_recycler_common/hr_recycler_description/urdf/bases/hr_recycler.urdf.xacro (robot description, xacro)
@@ -33,13 +33,7 @@
       <origin xyz="${base_link_origin}" rpy="0 0 0" />
       <geometry>
-        <mesh filename="package://hr_recycler_description/meshes/wheels/HR_recycler_steer.stl" scale="-1 1 1"/>
+        <mesh filename="package://hr_recycler_description/meshes/wheels/hr_recycler_steer.stl" scale="-1 1 1"/>
       </geometry>
     </visual>
-    <!--collision>
-      <origin xyz="${base_link_origin}" rpy="0 0 0" />
-      <geometry>
-        <mesh filename="package://hr_recycler_description/meshes/wheels/HR_recycler_steer.stl" scale="-1 1 1"/>
-      </geometry>
-    </collision-->
   </link>
   </xacro:macro>

File: hr_recycler_common/hr_recycler_description/urdf/elevator/elevator.urdf.xacro (robot description, xacro)
@@ -28,13 +28,13 @@
   <!-- ************** -->
   <xacro:macro name="elevator_platform" params="prefix parent hq *origin">
-  	<joint name="${prefix}_foot_elevator_joint" type="fixed">
+  	<joint name="${prefix}foot_elevator_joint" type="fixed">
   			<xacro:insert_block name="origin" />
   			<parent link="${parent}"/>
-  			<child link="${prefix}_foot_elevator_link" />
+  			<child link="${prefix}foot_elevator_link" />
   	</joint>
-  	<link name="${prefix}_foot_elevator_link">
+  	<link name="${prefix}foot_elevator_link">
   	</link>
     <!-- Support wheel -->
-  	<xacro:omni_wheel prefix="${prefix}_omni" parent="${prefix}_foot_elevator_link" hq="${hq}">
+  	<xacro:omni_wheel prefix="${prefix}omni" parent="${prefix}foot_elevator_link" hq="${hq}">
   			<origin xyz="${support_wheel_origin}" rpy="0 0 0"/>
   	</xacro:omni_wheel>
@@ -43,12 +43,12 @@
   <!--    PLATFORM    -->
   <!-- ************** -->
-  <xacro:macro name="both_elevator" params="prefix parent hq *origin" >
-    <joint name="${prefix}_base_elevator_joint" type="fixed">
+  <xacro:macro name="elevator" params="prefix parent hq *origin" >
+    <joint name="${prefix}base_elevator_joint" type="fixed">
         <xacro:insert_block name="origin" />
         <parent link="${parent}"/>
-        <child link="${prefix}_base_elevator_link" />
+        <child link="${prefix}base_elevator_link" />
     </joint>
     <!-- This piece supports the two lower forks -->
-    <link name="${prefix}_base_elevator_link">
+    <link name="${prefix}base_elevator_link">
       <inertial>
         <mass value="1" />
@@ -57,20 +57,13 @@
       </inertial>
     </link>
-    <!-- Called two lower forks -->
-    <xacro:elevator_platform prefix="$(arg prefix)left" parent="${prefix}_base_elevator_link" hq="${hq}">
-        <origin xyz="${fork_x} ${fork_y} ${fork_z}" rpy="0 0 0"/>
-    </xacro:elevator_platform>
-    <xacro:elevator_platform prefix="$(arg prefix)right" parent="${prefix}_base_elevator_link" hq="${hq}">
-        <origin xyz="${fork_x} -${fork_y} ${fork_z}" rpy="0 0 0"/>
-    </xacro:elevator_platform>
-    <joint name="${prefix}_elevator_joint" type="prismatic">
+    <joint name="${prefix}elevator_joint" type="prismatic">
        <xacro:insert_block name="origin" />
-       <parent link="${parent}"/>
-       <child link="${prefix}_elevator_link" />
+       <parent link="${prefix}base_elevator_link"/>
+       <child link="${prefix}elevator_link" />
        <axis xyz="0 0 1"/>
        <limit effort="1000.0" lower="0.0" upper="${upper_limit_elevator}" velocity="1"/>
      </joint>
      <!-- This piece holds the forks that are going to be elevated -->
-     <link name="${prefix}_elevator_link">
+     <link name="${prefix}elevator_link">
        <inertial>
          <mass value="${fork_mass}" />
@@ -81,5 +74,5 @@
          <origin xyz="0 0 0.410" rpy="0 0 0" />
          <geometry>
-           <mesh filename="package://hr_recycler_description/meshes/bases/HR_recycler_base_forks.stl" scale="-1 1 1"/>
+           <mesh filename="package://hr_recycler_description/meshes/bases/hr_recycler_base_forks.stl" scale="-1 1 1"/>
          </geometry>
           <material name="darkgrey">
@@ -90,17 +83,24 @@
          <origin xyz="0 0 0.410" rpy="0 0 0" />
          <geometry>
-           <mesh filename="package://hr_recycler_description/meshes/bases/HR_recycler_base_forks.stl" scale="-1 1 1"/>
+           <mesh filename="package://hr_recycler_description/meshes/bases/hr_recycler_base_forks.stl" scale="-1 1 1"/>
          </geometry>
        </collision>
      </link>
+    <!-- Called two lower forks -->
+    <xacro:elevator_platform prefix="$(arg prefix)left_" parent="${prefix}base_elevator_link" hq="${hq}">
+        <origin xyz="${fork_x} ${fork_y} ${fork_z}" rpy="0 0 0"/>
+    </xacro:elevator_platform>
+    <xacro:elevator_platform prefix="$(arg prefix)right_" parent="${prefix}base_elevator_link" hq="${hq}">
+        <origin xyz="${fork_x} -${fork_y} ${fork_z}" rpy="0 0 0"/>
+    </xacro:elevator_platform>
     <!-- ************* -->
     <!-- TRANSMISSIONS -->
     <!-- ************* -->
-     <transmission name="${prefix}_elevator_joint_transmission">
+     <transmission name="${prefix}elevator_joint_transmission">
        <type>transmission_interface/SimpleTransmission</type>
-       <joint name="${prefix}_elevator_joint">
+       <joint name="${prefix}elevator_joint">
          <hardwareInterface>hardware_interface/PositionJointInterface</hardwareInterface>
        </joint>
-       <actuator name="${prefix}_elevator_joint_motor">
+       <actuator name="${prefix}elevator_joint_motor">
          <hardwareInterface>hardware_interface/PositionActuatorInterface</hardwareInterface>
          <mechanicalReduction>${traction_mechanical_reduction}</mechanicalReduction>

File: hr_recycler_common/hr_recycler_description/urdf/wheels/motor_wheel.urdf.xacro (robot description, xacro)
@@ -58,5 +58,5 @@
           <origin xyz="0 0 -0.125" rpy="0 0 0" />
           <geometry>
-            <mesh filename="package://hr_recycler_description/meshes/wheels/HR_recycler_wheel.stl" scale="1 -0.9 1"/>
+            <mesh filename="package://hr_recycler_description/meshes/wheels/hr_recycler_wheel.stl" scale="1 -0.9 1"/>
           </geometry>
         </xacro:if>
@@ -64,5 +64,5 @@
           <origin xyz="0 0 -0.125" rpy="0 0 0" />
           <geometry>
-            <mesh filename="package://hr_recycler_description/meshes/wheels/HR_recycler_wheel.stl" scale="1 -0.9 1"/>
+            <mesh filename="package://hr_recycler_description/meshes/wheels/hr_recycler_wheel.stl" scale="1 -0.9 1"/>
           </geometry>
         </xacro:unless>
@@ -71,5 +71,5 @@
         <origin xyz="0 0 -0.125" rpy="0 0 0" />
         <geometry>
-          <mesh filename="package://hr_recycler_description/meshes/wheels/HR_recycler_wheel.stl" scale="1 -0.9 1"/>
+          <mesh filename="package://hr_recycler_description/meshes/wheels/hr_recycler_wheel.stl" scale="1 -0.9 1"/>
         </geometry>
       </collision>

Commit message: prefix is now a property of xacro

File: hr_recycler_common/hr_recycler_description/robots/hr_recycler_std.urdf.xacro (robot description, xacro)
@@ -48,19 +48,20 @@
 	<!-- Here we create the robot elements using the xacro:macros imported at the beggining of this file -->
 	<xacro:arg name="prefix" default="hr_recycler_"/>
-	<xacro:hr_recycler prefix="$(arg prefix)" publish_bf="true" hq="${hq}" /> <!-- BASE -->
-	<xacro:motor_wheel prefix="$(arg prefix)front_" parent="$(arg prefix)base_link" hq="${hq}"> <!-- WHEEL -->
+    <xacro:property name="prefix" value="$(arg prefix)" />
+	<xacro:hr_recycler prefix="${prefix}" publish_bf="true" hq="${hq}" /> <!-- BASE -->
+	<xacro:motor_wheel prefix="${prefix}front_" parent="${prefix}base_link" hq="${hq}"> <!-- WHEEL -->
 			<!--origin xyz="${wheel_offset_x} ${wheel_offset_y} ${wheel_offset_z}" rpy="0 0 0"/-->
       <origin xyz="0 0 0.460" rpy="0 0 0"/>
 	</xacro:motor_wheel>
-    <xacro:elevator prefix="$(arg prefix)" parent="$(arg prefix)base_link" hq="${hq}"> <!-- ELEVATOR -->
+    <xacro:elevator prefix="${prefix}" parent="${prefix}base_link" hq="${hq}"> <!-- ELEVATOR -->
         <origin xyz="${elevator}" rpy="0 0 0"/>
     </xacro:elevator>
-    <xacro:sensor_sick_s300 prefix="$(arg prefix)front_laser" parent="$(arg prefix)base_footprint"> <!-- BACK SENSOR -->
+    <xacro:sensor_sick_s300 prefix="${prefix}front_laser" parent="${prefix}base_footprint"> <!-- BACK SENSOR -->
         <origin xyz="${sensor}" rpy="${PI} 0 0"/>
     </xacro:sensor_sick_s300>
-    <xacro:sensor_r430 prefix="$(arg prefix)right_fork" parent="$(arg prefix)elevator_link" prefix_topic="front_right_rgbd_camera">
+    <xacro:sensor_r430 prefix="${prefix}right_fork" parent="${prefix}elevator_link" prefix_topic="front_right_rgbd_camera">
         <origin xyz="${camera_x} ${camera_y} ${camera_z}" rpy="0 0 ${PI}"/>
     </xacro:sensor_r430>
-    <xacro:sensor_r430 prefix="$(arg prefix)left_fork" parent="$(arg prefix)elevator_link" prefix_topic="front_left_rgbd_camera">
+    <xacro:sensor_r430 prefix="${prefix}left_fork" parent="${prefix}elevator_link" prefix_topic="front_left_rgbd_camera">
         <origin xyz="${camera_x} -${camera_y} ${camera_z}" rpy="0 0 ${PI}"/>
     </xacro:sensor_r430>

File: hr_recycler_common/hr_recycler_description/urdf/common.gazebo.xacro (robot description, xacro)
@@ -14,11 +14,11 @@
    </xacro:macro>
    <xacro:macro name="gazebo_colors" params="prefix">
-		<gazebo reference="$(arg prefix)base_footprint">
+		<gazebo reference="${prefix}base_footprint">
 			<material>Gazebo/Green</material>
 		</gazebo>
-		<gazebo reference="$(arg prefix)base_link">
+		<gazebo reference="${prefix}base_link">
 			<material>Gazebo/Grey</material>
 		</gazebo>
-		<gazebo reference="$(arg prefix)front_cover_link">
+		<gazebo reference="${prefix}front_cover_link">
 			<material>Gazebo/Black</material>
 		</gazebo>

File: hr_recycler_common/hr_recycler_description/urdf/elevator/elevator.urdf.xacro (robot description, xacro)
@@ -88,8 +88,8 @@
      </link>
     <!-- Called two lower forks -->
-    <xacro:elevator_platform prefix="$(arg prefix)left_" parent="${prefix}base_elevator_link" hq="${hq}">
+    <xacro:elevator_platform prefix="${prefix}left_" parent="${prefix}base_elevator_link" hq="${hq}">
         <origin xyz="${fork_x} ${fork_y} ${fork_z}" rpy="0 0 0"/>
     </xacro:elevator_platform>
-    <xacro:elevator_platform prefix="$(arg prefix)right_" parent="${prefix}base_elevator_link" hq="${hq}">
+    <xacro:elevator_platform prefix="${prefix}right_" parent="${prefix}base_elevator_link" hq="${hq}">
         <origin xyz="${fork_x} -${fork_y} ${fork_z}" rpy="0 0 0"/>
     </xacro:elevator_platform>

Commit message: wip to solve physics issue

File: hr_recycler_common/hr_recycler_description/robots/hr_recycler_std.urdf.xacro (robot description, xacro)
@@ -48,5 +48,5 @@
 	<!-- Here we create the robot elements using the xacro:macros imported at the beggining of this file -->
 	<xacro:arg name="prefix" default="hr_recycler_"/>
-    <xacro:property name="prefix" value="$(arg prefix)" />
+  <xacro:property name="prefix" value="$(arg prefix)" />
 	<xacro:hr_recycler prefix="${prefix}" publish_bf="true" hq="${hq}" /> <!-- BASE -->
 	<xacro:motor_wheel prefix="${prefix}front_" parent="${prefix}base_link" hq="${hq}"> <!-- WHEEL -->

File: hr_recycler_common/hr_recycler_description/urdf/bases/hr_recycler.urdf.xacro (robot description, xacro)
@@ -7,5 +7,5 @@
   <xacro:property name="base_width" value="0.754" />
   <xacro:property name="base_height" value="0.2" />
-  <xacro:property name="base_mass" value="50"/>
+  <xacro:property name="base_mass" value="1"/>
   <xacro:property name="base_link_origin" value="0 0 0.46" />
   <!-- Inertial equation -->

File: hr_recycler_common/hr_recycler_description/urdf/elevator/elevator.urdf.xacro (robot description, xacro)
@@ -44,35 +44,50 @@
   <!-- ************** -->
   <xacro:macro name="elevator" params="prefix parent hq *origin" >
-    <joint name="${prefix}base_elevator_joint" type="fixed">
+    <joint name="${prefix}base_elevator_joint" type="prismatic">
         <xacro:insert_block name="origin" />
         <parent link="${parent}"/>
         <child link="${prefix}base_elevator_link" />
+        <axis xyz="0 0 1"/>
+        <limit effort="1000.0" lower="0.0" upper="${upper_limit_elevator}" velocity="1"/>
     </joint>
     <!-- This piece supports the two lower forks -->
     <link name="${prefix}base_elevator_link">
+      <visual>
+        <origin xyz="0 0 0.410" rpy="0 0 0" />
+        <geometry>
+          <mesh filename="package://hr_recycler_description/meshes/bases/base.stl" scale="-1 1 1"/>
+        </geometry>
+         <material name="darkgrey">
+           <color rgba="0.1 0.1 0.1 1"/>
+         </material>
+      </visual>
       <inertial>
         <mass value="1" />
-        <origin xyz="0 0 0" />
-        <cylinder_inertia m="7" r="1" h="1" />
+        <origin xyz="-0.8 0 0" />
+        <box_inertia  m="1" x="1.67" y="0.1" z="0.03"/>
       </inertial>
+      <collision>
+        <origin xyz="0 0 0.410" rpy="0 0 0" />
+        <geometry>
+          <mesh filename="package://hr_recycler_description/meshes/bases/base.stl" scale="-1 1 1"/>
+        </geometry>
+      </collision>
     </link>
-    <joint name="${prefix}elevator_joint" type="prismatic">
+    <joint name="${prefix}elevator_joint" type="fixed">
        <xacro:insert_block name="origin" />
        <parent link="${prefix}base_elevator_link"/>
        <child link="${prefix}elevator_link" />
-       <axis xyz="0 0 1"/>
-       <limit effort="1000.0" lower="0.0" upper="${upper_limit_elevator}" velocity="1"/>
      </joint>
      <!-- This piece holds the forks that are going to be elevated -->
      <link name="${prefix}elevator_link">
        <inertial>
-         <mass value="${fork_mass}" />
-         <origin xyz="0 0 1" />
+         <mass value="1" />
+         <origin xyz="-0.2 0 0" />
          <solid_cuboid_inertia m="${fork_mass}" h="${fork_height}" d="${fork_length}" w="${fork_width}"/>
        </inertial>
        <visual>
-         <origin xyz="0 0 0.410" rpy="0 0 0" />
+         <origin xyz="-1.3725 0 0.080" rpy="0 0 0" />
          <geometry>
-           <mesh filename="package://hr_recycler_description/meshes/bases/hr_recycler_base_forks.stl" scale="-1 1 1"/>
+           <mesh filename="package://hr_recycler_description/meshes/elevator/hr_recycler_forks.stl" scale="-1 1 1"/>
          </geometry>
           <material name="darkgrey">
@@ -81,15 +96,15 @@
        </visual>
        <collision>
-         <origin xyz="0 0 0.410" rpy="0 0 0" />
+         <origin xyz="-1.3725 0 0.080" rpy="0 0 0" />
          <geometry>
-           <mesh filename="package://hr_recycler_description/meshes/bases/hr_recycler_base_forks.stl" scale="-1 1 1"/>
+           <mesh filename="package://hr_recycler_description/meshes/elevator/hr_recycler_forks.stl" scale="-1 1 1"/>
          </geometry>
        </collision>
      </link>
     <!-- Called two lower forks -->
-    <xacro:elevator_platform prefix="${prefix}left_" parent="${prefix}base_elevator_link" hq="${hq}">
+    <xacro:elevator_platform prefix="${prefix}left_" parent="${prefix}base_footprint" hq="${hq}">
         <origin xyz="${fork_x} ${fork_y} ${fork_z}" rpy="0 0 0"/>
     </xacro:elevator_platform>
-    <xacro:elevator_platform prefix="${prefix}right_" parent="${prefix}base_elevator_link" hq="${hq}">
+    <xacro:elevator_platform prefix="${prefix}right_" parent="${prefix}base_footprint" hq="${hq}">
         <origin xyz="${fork_x} -${fork_y} ${fork_z}" rpy="0 0 0"/>
     </xacro:elevator_platform>
@@ -97,10 +112,10 @@
     <!-- TRANSMISSIONS -->
     <!-- ************* -->
-     <transmission name="${prefix}elevator_joint_transmission">
+     <transmission name="${prefix}base_elevator_joint_transmission">
        <type>transmission_interface/SimpleTransmission</type>
-       <joint name="${prefix}elevator_joint">
+       <joint name="${prefix}base_elevator_joint">
          <hardwareInterface>hardware_interface/PositionJointInterface</hardwareInterface>
        </joint>
-       <actuator name="${prefix}elevator_joint_motor">
+       <actuator name="${prefix}base_elevator_joint_motor">
          <hardwareInterface>hardware_interface/PositionActuatorInterface</hardwareInterface>
          <mechanicalReduction>${traction_mechanical_reduction}</mechanicalReduction>

File: hr_recycler_common/hr_recycler_description/urdf/wheels/motor_wheel.urdf.xacro (robot description, xacro)
@@ -18,5 +18,5 @@
   <xacro:property name="traction_joint_velocity_limit" value="100" />
   <xacro:property name="traction_mechanical_reduction" value="1.0" />
-  <xacro:property name="steer_origin" value="0 0 0.460"/>
+  <xacro:property name="steer_origin" value="0 0 -0.210"/>
   <xacro:property name="traction_origin" value="0 0 -0.335"/>
   <!-- inertial equation -->
@@ -40,5 +40,5 @@
       <inertial>
         <mass value="${wheel_mass}" />
-        <origin xyz="${steer_origin}" />
+        <origin xyz="${steer_origin}"/>
         <cylinder_inertia m="${wheel_mass}" r="${wheel_width}" h="${wheel_radius}" />
       </inertial>
