Commit message: cleaned xacro properties

File: hr_recycler_common/hr_recycler_description/robots/hr_recycler_std.urdf.xacro (robot description, xacro)
@@ -21,26 +21,15 @@
 	<xacro:property name="wheel_offset_x" value="0.0"/>
 	<xacro:property name="wheel_offset_y" value="0.0"/>
-	<xacro:property name="wheel_offset_z" value="${wheel_radius}"/>
-  <xacro:property name="separation_wheel_box" value="0.08" />
-  <!-- Base parameters -->
-  <xacro:property name="base_length" value="0.679" />
-  <xacro:property name="base_height" value="0.533" />
-  <xacro:property name="base_width" value="0.754" />
+	<xacro:property name="wheel_offset_z" value="0.46"/>
 	<!-- Flag to select the high or low quality model -->
 	<xacro:property name="hq" value="true" />
-	<!--  SENSOR PARAMETERS  -->
-  <xacro:property name="sensor_length" value="0.055" />
-  <xacro:property name="sensor" value="0.25294 0 0.200" />
-	<!--  CAMERA PARAMETERS  -->
-  <xacro:property name="camera_x" value="-1.539" />
-  <xacro:property name="camera_y" value="0.195" />
-  <xacro:property name="camera_z" value="0.067" />
-	<!-- ELEVATOR PARAMETERS -->
-	<xacro:property name="elevator_x" value="-${base_length/2.0}" />
-	<xacro:property name="elevator_y" value="0.0" />
-	<xacro:property name="elevator_z" value="${-wheel_radius/2.0+fork_height/2.0}" />
-  <xacro:property name="fork_length" value="1.176" />
-  <xacro:property name="fork_height" value="0.015" />
-  <xacro:property name="elevator" value="0 0 0" />
+	<!--  FORK CAMERAS  -->
+  <xacro:property name="fork_camera_x" value="-1.539" />
+  <xacro:property name="fork_camera_y" value="0.195" />
+  <xacro:property name="fork_camera_z" value="0.067" />
+   <!-- FRONT LASER -->
+ <xacro:property name="front_laser_x" value="0.25294" />
+ <xacro:property name="front_laser_y" value="0.000" />
+ <xacro:property name="front_laser_z" value="0.200" />
 	<!-- *************** -->
 	<!-- Robots Elements -->
@@ -51,18 +40,17 @@
 	<xacro:hr_recycler prefix="${prefix}" publish_bf="true" hq="${hq}" /> <!-- BASE -->
 	<xacro:motor_wheel prefix="${prefix}front_" parent="${prefix}base_link" hq="${hq}"> <!-- WHEEL -->
-			<!--origin xyz="${wheel_offset_x} ${wheel_offset_y} ${wheel_offset_z}" rpy="0 0 0"/-->
-      <origin xyz="0 0 0.460" rpy="0 0 0"/>
+			<origin xyz="${wheel_offset_x} ${wheel_offset_y} ${wheel_offset_z}" rpy="0 0 0"/>
 	</xacro:motor_wheel>
     <xacro:elevator prefix="${prefix}" parent="${prefix}base_link" hq="${hq}"> <!-- ELEVATOR -->
-        <origin xyz="${elevator}" rpy="0 0 0"/>
+        <origin xyz="0 0 0" rpy="0 0 0"/>
     </xacro:elevator>
-    <xacro:sensor_sick_s300 prefix="${prefix}front_laser" parent="${prefix}base_footprint"> <!-- BACK SENSOR -->
-        <origin xyz="${sensor}" rpy="${PI} 0 0"/>
+    <xacro:sensor_sick_s300 prefix="${prefix}front_laser" parent="${prefix}base_footprint"> <!-- FRONT LIDAR -->
+        <origin xyz="${front_laser_x} ${front_laser_y} ${front_laser_z}" rpy="${PI} 0 0"/>
     </xacro:sensor_sick_s300>
-    <xacro:sensor_r430 prefix="${prefix}right_fork" parent="${prefix}elevator_link" prefix_topic="front_right_rgbd_camera">
-        <origin xyz="${camera_x} ${camera_y} ${camera_z}" rpy="0 0 ${PI}"/>
+    <xacro:sensor_r430 prefix="${prefix}right_fork" parent="${prefix}elevator_link" prefix_topic="right_fork_rgbd_camera">
+        <origin xyz="${fork_camera_x} ${fork_camera_y} ${fork_camera_z}" rpy="0 0 ${PI}"/>
     </xacro:sensor_r430>
-    <xacro:sensor_r430 prefix="${prefix}left_fork" parent="${prefix}elevator_link" prefix_topic="front_left_rgbd_camera">
-        <origin xyz="${camera_x} -${camera_y} ${camera_z}" rpy="0 0 ${PI}"/>
+    <xacro:sensor_r430 prefix="${prefix}left_fork" parent="${prefix}elevator_link" prefix_topic="left_fork_rgbd_camera">
+        <origin xyz="${fork_camera_x} -${fork_camera_y} ${fork_camera_z}" rpy="0 0 ${PI}"/>
     </xacro:sensor_r430>
 	<!-- Gazebo ros control pluggins -->

File: hr_recycler_common/hr_recycler_description/urdf/bases/hr_recycler.urdf.xacro (robot description, xacro)
@@ -4,5 +4,4 @@
   <xacro:macro name="hr_recycler" params="prefix publish_bf hq">
   <!-- Robot mechanical and motor parameters -->
-  <xacro:property name="wheel_radius" value="0.10" />
   <xacro:property name="base_length" value="0.679" />
   <xacro:property name="base_width" value="0.754" />

File: hr_recycler_common/hr_recycler_description/urdf/epal_pallet/epal_pallet.urdf.xacro (robot description, xacro)
@@ -15,5 +15,7 @@
       <mass value="5" />
       <origin xyz="0 0 0" />
-      <solid_cuboid_inertia m="5" h="0.044" d="1.2" w="0.8"/> <!-- h = z, d = y, w = x -->
+      <!-- yes, axis in solid_cuboid_inertia are changed, w relates to X axis, d to Z axis, and h to Y axis -->
+      <!-- Keep this comment -->
+      <solid_cuboid_inertia m="5" h="0.8" d="0.044" w="1.2"/> <!-- h = z, d = y, w = x -->
     </inertial>
     <visual>
@@ -47,5 +49,7 @@
       <mass value="1" />
       <origin xyz="0 0 0" />
-      <solid_cuboid_inertia m="1" h="0.1" d="1.2" w="0.1"/> <!-- h = z, d = y, w = x -->
+      <!-- yes, axis in solid_cuboid_inertia are changed, w relates to X axis, d to Z axis, and h to Y axis -->
+      <!-- Keep this comment -->
+      <solid_cuboid_inertia m="1" h="0.1" d="0.1" w="1.2"/> <!-- h = z, d = y, w = x -->
     </inertial>
     <visual>
@@ -71,5 +75,7 @@
       <mass value="1" />
       <origin xyz="0 0 0" />
-      <solid_cuboid_inertia m="1" h="0.1" d="1.2" w="0.1"/> <!-- h = z, d = y, w = x -->
+      <!-- yes, axis in solid_cuboid_inertia are changed, w relates to X axis, d to Z axis, and h to Y axis -->
+      <!-- Keep this comment -->
+      <solid_cuboid_inertia m="1" h="0.1" d="0.1" w="1.2"/> <!-- h = z, d = y, w = x -->
     </inertial>
     <visual>
@@ -95,5 +101,7 @@
       <mass value="1" />
       <origin xyz="0 0 0" />
-      <solid_cuboid_inertia m="1" h="0.1" d="1.2" w="0.1"/> <!-- h = z, d = y, w = x -->
+      <!-- yes, axis in solid_cuboid_inertia are changed, w relates to X axis, d to Z axis, and h to Y axis -->
+      <!-- Keep this comment -->
+      <solid_cuboid_inertia m="1" h="0.1" d="0.1" w="1.2"/> <!-- h = z, d = y, w = x -->
     </inertial>
     <visual>
