Commit message: Added elevator transmission

File: pallet_truck_common/pallet_truck_description/urdf/bases/pallet_truck.urdf.xacro (robot description, xacro)
@@ -3,4 +3,5 @@
   <xacro:include filename="$(find pallet_truck_description)/urdf/inertia.urdf.xacro" />
   <xacro:macro name="pallet_truck" params="prefix publish_bf hq">
+	<xacro:property name="PI" value="3.1415926535897931"/>
   <!-- Robot mechanical and motor parameters -->
   <xacro:property name="base_length" value="0.35" />
@@ -32,5 +33,5 @@
     </inertial>
     <visual>
-      <origin xyz="0 0 0" rpy="0 0 0" />
+      <origin xyz="0 0 0" rpy="0 0 ${M_PI}" />
       <geometry>
         <mesh filename="package://pallet_truck_description/meshes/bases/base.stl"/>
@@ -38,5 +39,5 @@
     </visual>
     <collision>
-      <origin xyz="0 0 0" rpy="0 0 0" />
+      <origin xyz="0 0 0" rpy="0 0 ${M_PI}" />
       <geometry>
         <mesh filename="package://pallet_truck_description/meshes/bases/base.stl"/>

File: pallet_truck_common/pallet_truck_description/urdf/elevator/elevator.urdf.xacro (robot description, xacro)
@@ -81,4 +81,14 @@
        <limit effort="1000.0" lower="0.0" upper="0" velocity="1"/>
      </joint>
+     <transmission name="${prefix}fork_joint_transmission">
+       <type>transmission_interface/SimpleTransmission</type>
+       <joint name="${prefix}fork_joint">
+         <hardwareInterface>hardware_interface/VelocityJointInterface</hardwareInterface>
+       </joint>
+       <actuator name="${prefix}fork_joint_motor">
+         <hardwareInterface>hardware_interface/VelocityActuatorInterface</hardwareInterface>
+         <mechanicalReduction>${traction_mechanical_reduction}</mechanicalReduction>
+       </actuator>
+     </transmission>
      <!-- This piece holds the forks that are going to be elevated -->
      <link name="${prefix}fork_link">
@@ -174,9 +184,9 @@
     </xacro:fork>
     <!-- Called two support wheels -->
-    <xacro:support_wheel prefix="${prefix}left_" parent="${prefix}base_footprint" hq="${hq}">
-        <origin xyz="1.3725 0.195 0.04" rpy="0 0 0"/>
+    <xacro:support_wheel prefix="${prefix}left_" parent="${prefix}central_link" hq="${hq}">
+        <origin xyz="1.3725 0.195 -0.42" rpy="0 0 0"/>
     </xacro:support_wheel>
-    <xacro:support_wheel prefix="${prefix}right_" parent="${prefix}base_footprint" hq="${hq}">
-        <origin xyz="1.3725 -0.195 0.04" rpy="0 0 0"/>
+    <xacro:support_wheel prefix="${prefix}right_" parent="${prefix}central_link" hq="${hq}">
+        <origin xyz="1.3725 -0.195 -0.42" rpy="0 0 0"/>
     </xacro:support_wheel>
     <!-- ************* -->
