Commit message: 2 focus, only one blinks

File: pallet_truck_common/pallet_truck_description/urdf/bases/front_case.urdf.xacro (robot description, xacro)
@@ -37,11 +37,80 @@
        </collision>
      </link>
-		 <!--gazebo reference="${prefix}front_case_link">
-			 <mu1 value="1"/>
-			 <mu2 value="1"/>
-			 <kp>100000000.0</kp>
-			 <!- -kd value="10.0"/- ->
-			 <material>Gazebo/Black</material>
-		 </gazebo-->
+		 <gazebo>
+		   <model name='light_model'>
+		     <pose>1.5207 0.281 0.7 0 0 0</pose>
+		     <link name='light_link'>
+		       <visual name='light_source'>
+		         <pose>0 0 0 0 0 0</pose>
+		         <geometry>
+		           <box>
+		             <size>0.35 0.005 0.01</size>
+		           </box>
+		         </geometry>
+		         <material>
+		           <ambient>1 1 1 1</ambient>
+		           <diffuse>1 1 1 1</diffuse>
+		           <specular>1 1 1 1</specular>
+		           <emissive>0 0 0 1</emissive>
+		         </material>
+		       </visual>
+		       <light name='light_source' type='spot'>
+		         <pose>0 0 0 0 0 0</pose>
+		         <attenuation>
+		           <range>0.2</range>
+		           <!--linear>0.10</linear-->
+		         </attenuation>
+		         <diffuse>0 0 0 1</diffuse>
+		         <specular>0 0 0 1</specular>
+		       </light>
+			       <visual name='light_source2'>
+			         <pose>0 0 0 0 0 0</pose>
+			         <geometry>
+			           <box>
+			             <size>0.35 0.005 0.01</size>
+			           </box>
+			         </geometry>
+			         <material>
+			           <ambient>1 1 1 1</ambient>
+			           <diffuse>1 1 1 1</diffuse>
+			           <specular>1 1 1 1</specular>
+			           <emissive>0 0 0 1</emissive>
+			         </material>
+			       </visual>
+			       <light name='light_source2' type='spot'>
+			         <pose>0 -0.564 0 0 0 0</pose>
+			         <attenuation>
+			           <range>0.2</range>
+			           <!--linear>0.10</linear-->
+			         </attenuation>
+			         <diffuse>0 0 0 1</diffuse>
+			         <specular>0 0 0 1</specular>
+			       </light>
+		     </link>
+		     <plugin name='light_control' filename='libLedPlugin.so'>
+		 			<enable>true</enable>
+		       <light>
+		         <id>light_link/light_source</id>
+		         <enable>true</enable>
+		         <duration>1</duration>
+		         <interval>0.5</interval>
+		         <color>1 0 0</color>
+		       </light>
+					 <light>
+						 <id>light_link/light_source2</id>
+						 <enable>true</enable>
+						 <duration>1</duration>
+						 <interval>0.5</interval>
+						 <color>1 0 0</color>
+					 </light>
+		     </plugin>
+		   </model>
+		   </gazebo>
+		   <gazebo>
+		     <joint name='light_joint' type='fixed'>
+		       <parent>${prefix}front_case_link</parent>
+		       <child>light_model::light_link</child>
+		     </joint>
+		   </gazebo>
   </xacro:macro>
 </robot>

Commit message: Changed package.xml for projecting, 1 focus static light without beam

File: pallet_truck_common/pallet_truck_description/urdf/bases/front_case.urdf.xacro (robot description, xacro)
@@ -39,6 +39,6 @@
 		 <gazebo>
 		   <model name='light_model'>
-		     <pose>1.5207 0.281 0.7 0 0 0</pose>
 		     <link name='light_link'>
+					 <pose>1.5207 0.281 0.7 0 0 0</pose>
 		       <visual name='light_source'>
 		         <pose>0 0 0 0 0 0</pose>
@@ -64,27 +64,30 @@
 		         <specular>0 0 0 1</specular>
 		       </light>
-			       <visual name='light_source2'>
-			         <pose>0 0 0 0 0 0</pose>
-			         <geometry>
-			           <box>
-			             <size>0.35 0.005 0.01</size>
-			           </box>
-			         </geometry>
-			         <material>
-			           <ambient>1 1 1 1</ambient>
-			           <diffuse>1 1 1 1</diffuse>
-			           <specular>1 1 1 1</specular>
-			           <emissive>0 0 0 1</emissive>
-			         </material>
-			       </visual>
-			       <light name='light_source2' type='spot'>
-			         <pose>0 -0.564 0 0 0 0</pose>
-			         <attenuation>
-			           <range>0.2</range>
-			           <!--linear>0.10</linear-->
-			         </attenuation>
-			         <diffuse>0 0 0 1</diffuse>
-			         <specular>0 0 0 1</specular>
-			       </light>
+		     </link>
+				 <link name='light_link_2"'>
+					 <pose>1.5207 -0.281 0.7 0 0 0</pose>
+		       <visual name='light_source'>
+		         <pose>0 0 0 0 0 0</pose>
+		         <geometry>
+		           <box>
+		             <size>0.35 0.005 0.01</size>
+		           </box>
+		         </geometry>
+		         <material>
+		           <ambient>1 1 1 1</ambient>
+		           <diffuse>1 1 1 1</diffuse>
+		           <specular>1 1 1 1</specular>
+		           <emissive>0 0 0 1</emissive>
+		         </material>
+		       </visual>
+		       <light name='light_source' type='spot'>
+		         <pose>0 0 0 0 0 0</pose>
+		         <attenuation>
+		           <range>20</range>
+		           <linear>0.10</linear>
+		         </attenuation>
+		         <diffuse>0 0 0 1</diffuse>
+		         <specular>0 0 0 1</specular>
+		       </light>
 		     </link>
 		     <plugin name='light_control' filename='libLedPlugin.so'>
@@ -92,25 +95,73 @@
 		       <light>
 		         <id>light_link/light_source</id>
-		         <enable>true</enable>
-		         <duration>1</duration>
-		         <interval>0.5</interval>
-		         <color>1 0 0</color>
-		       </light>
-					 <light>
-						 <id>light_link/light_source2</id>
-						 <enable>true</enable>
-						 <duration>1</duration>
-						 <interval>0.5</interval>
-						 <color>1 0 0</color>
+						 <block>
+						 		<enable>true</enable>
+						 		<duration>1</duration>
+						 		<interval>0</interval>
+						 		<color>1 0 0</color>
+								<attenuation>
+									<range>20</range>
+									<linear>0.10</linear>
+								</attenuation>
+						 </block>
+						 <block>
+							 <duration>1</duration>
+							 <interval>0</interval>
+							 <color>1 0 0</color>
+							 <attenuation>
+								 <range>20</range>
+								 <linear>0.10</linear>
+							 </attenuation>
+						 </block>
+						 <block>
+							 <duration>1</duration>
+							 <interval>0</interval>
+							 <color>1 0 0</color>
+							 <attenuation>
+								 <range>20</range>
+								 <linear>0.10</linear>
+							 </attenuation>
+						 </block>
+						 <light>
+							 <id>light_link_2/light_source_2</id>
+							 <duration>0.3</duration>
+							 <interval>0.4</interval>
+							 <enable>true</enable>
+							 <color>1 0 0</color>
+						 </light>
 					 </light>
 		     </plugin>
 		   </model>
-		   </gazebo>
-		   <gazebo>
-		     <joint name='light_joint' type='fixed'>
-		       <parent>${prefix}front_case_link</parent>
-		       <child>light_model::light_link</child>
-		     </joint>
-		   </gazebo>
+		 </gazebo>
+		 <gazebo>
+		   <joint name='light_joint' type='fixed'>
+		     <parent>${prefix}front_case_link</parent>
+		     <child>light_model::light_link</child>
+		   </joint>
+		 </gazebo>
+		 <!--joint name="projector_joint" type="revolute">
+        <origin xyz="0 0 0.5" />
+        <parent link="${prefix}front_case_link"/>
+        <child link="projector_link" />
+				<limit effort="0" velocity="0" lower="0" upper="0"/>
+      </joint>
+      <link name="projector_link">
+      </link>
+		 <gazebo reference="projector_link">
+		     <projector name="projector_wg6802418">
+		         <pose>0 0 0 0 0 ${pi/2}</pose>
+		         <texture>package://pallet_truck_description/meshes/red.png</texture>
+		         <fov>0.5</fov>
+		         <near_clip>1</near_clip>
+		         <far_clip>10</far_clip>
+		      </projector>
+     			<plugin name="gazebo_ros_projector_controller" filename="libgazebo_ros_projector.so">
+         		<projector>projector/projector_wg6802418</projector>
+						<alwaysOn>true</alwaysOn>
+         		<updateRate>10.0</updateRate>
+         		<textureTopicName>/projector/image</textureTopicName>
+         		<projectorTopicName>/projector/projector</projectorTopicName>
+     			</plugin>
+	 		</gazebo-->
   </xacro:macro>
 </robot>

Commit message: 2focus and 2leds working

File: pallet_truck_common/pallet_truck_description/urdf/bases/front_case.urdf.xacro (robot description, xacro)
@@ -39,11 +39,11 @@
 		 <gazebo>
 		   <model name='light_model'>
+		     <pose>1.5207 0 0.68 0 0 0</pose>
 		     <link name='light_link'>
-					 <pose>1.5207 0.281 0.7 0 0 0</pose>
 		       <visual name='light_source'>
 		         <pose>0 0 0 0 0 0</pose>
 		         <geometry>
 		           <box>
-		             <size>0.35 0.005 0.01</size>
+		             <size>0.35 0.568 0.01</size>
 		           </box>
 		         </geometry>
@@ -56,37 +56,30 @@
 		       </visual>
 		       <light name='light_source' type='spot'>
-		         <pose>0 0 0 0 0 0</pose>
+		         <pose>0 0.35 0 0 0 0</pose>
 		         <attenuation>
-		           <range>0.2</range>
+		           <range>20</range>
 		           <!--linear>0.10</linear-->
 		         </attenuation>
 		         <diffuse>0 0 0 1</diffuse>
 		         <specular>0 0 0 1</specular>
+						 <spot>
+							 <inner_angle>0.1</inner_angle>
+							 <outer_angle>0.15</outer_angle>
+							 <falloff>1</falloff>
+						 </spot>
 		       </light>
-		     </link>
-				 <link name='light_link_2"'>
-					 <pose>1.5207 -0.281 0.7 0 0 0</pose>
-		       <visual name='light_source'>
-		         <pose>0 0 0 0 0 0</pose>
-		         <geometry>
-		           <box>
-		             <size>0.35 0.005 0.01</size>
-		           </box>
-		         </geometry>
-		         <material>
-		           <ambient>1 1 1 1</ambient>
-		           <diffuse>1 1 1 1</diffuse>
-		           <specular>1 1 1 1</specular>
-		           <emissive>0 0 0 1</emissive>
-		         </material>
-		       </visual>
-		       <light name='light_source' type='spot'>
-		         <pose>0 0 0 0 0 0</pose>
+					 <light name='light_source2' type='spot'>
+		         <pose>0 -0.35 0 0 0 0</pose>
 		         <attenuation>
 		           <range>20</range>
-		           <linear>0.10</linear>
+		           <!--linear>0.10</linear-->
 		         </attenuation>
 		         <diffuse>0 0 0 1</diffuse>
 		         <specular>0 0 0 1</specular>
+						 <spot>
+							 <inner_angle>0.1</inner_angle>
+							 <outer_angle>0.15</outer_angle>
+							 <falloff>1</falloff>
+						 </spot>
 		       </light>
 		     </link>
@@ -96,20 +89,33 @@
 		         <id>light_link/light_source</id>
 						 <block>
-						 		<enable>true</enable>
-						 		<duration>1</duration>
-						 		<interval>0</interval>
-						 		<color>1 0 0</color>
-								<attenuation>
-									<range>20</range>
-									<linear>0.10</linear>
-								</attenuation>
+							 <enable>true</enable>
+						 	 <duration>1</duration>
+						 	 <interval>0</interval>
+						 	 <color>1 0 0</color>
+						 	 <attenuation>
+						 	 		<range>20</range>
+						 	 		<linear>0.10</linear>
+						 	 </attenuation>
 						 </block>
 						 <block>
+						 	 <duration>1</duration>
+						 	 <interval>0</interval>
+						   <color>1 0 0</color>
+						 	 <attenuation>
+						 			 <range>20</range>
+						 			 <linear>0.10</linear>
+						 	 </attenuation>
+						  </block>
+					 </light>
+					 <light>
+						 <id>light_link/light_source2</id>
+						 <block>
+							 <enable>true</enable>
 							 <duration>1</duration>
 							 <interval>0</interval>
 							 <color>1 0 0</color>
 							 <attenuation>
-								 <range>20</range>
-								 <linear>0.10</linear>
+									<range>20</range>
+									<linear>0.10</linear>
 							 </attenuation>
 						 </block>
@@ -119,49 +125,18 @@
 							 <color>1 0 0</color>
 							 <attenuation>
-								 <range>20</range>
-								 <linear>0.10</linear>
+									 <range>20</range>
+									 <linear>0.10</linear>
 							 </attenuation>
-						 </block>
-						 <light>
-							 <id>light_link_2/light_source_2</id>
-							 <duration>0.3</duration>
-							 <interval>0.4</interval>
-							 <enable>true</enable>
-							 <color>1 0 0</color>
-						 </light>
+							</block>
 					 </light>
 		     </plugin>
 		   </model>
-		 </gazebo>
-		 <gazebo>
-		   <joint name='light_joint' type='fixed'>
-		     <parent>${prefix}front_case_link</parent>
-		     <child>light_model::light_link</child>
-		   </joint>
-		 </gazebo>
-		 <!--joint name="projector_joint" type="revolute">
-        <origin xyz="0 0 0.5" />
-        <parent link="${prefix}front_case_link"/>
-        <child link="projector_link" />
-				<limit effort="0" velocity="0" lower="0" upper="0"/>
-      </joint>
-      <link name="projector_link">
-      </link>
-		 <gazebo reference="projector_link">
-		     <projector name="projector_wg6802418">
-		         <pose>0 0 0 0 0 ${pi/2}</pose>
-		         <texture>package://pallet_truck_description/meshes/red.png</texture>
-		         <fov>0.5</fov>
-		         <near_clip>1</near_clip>
-		         <far_clip>10</far_clip>
-		      </projector>
-     			<plugin name="gazebo_ros_projector_controller" filename="libgazebo_ros_projector.so">
-         		<projector>projector/projector_wg6802418</projector>
-						<alwaysOn>true</alwaysOn>
-         		<updateRate>10.0</updateRate>
-         		<textureTopicName>/projector/image</textureTopicName>
-         		<projectorTopicName>/projector/projector</projectorTopicName>
-     			</plugin>
-	 		</gazebo-->
+		   </gazebo>
+		   <gazebo>
+		     <joint name='light_joint' type='fixed'>
+		       <parent>${prefix}front_case_link</parent>
+		       <child>light_model::light_link</child>
+		     </joint>
+		   </gazebo>
   </xacro:macro>
 </robot>

Commit message: Projects red image, but background black. TODO: Remove testing links, and project another image

File: pallet_truck_common/pallet_truck_description/urdf/bases/front_case.urdf.xacro (robot description, xacro)
@@ -37,5 +37,117 @@
        </collision>
      </link>
+		 <!--PROJECTOR -->
+		 <joint name="${prefix}projector_joint" type="fixed">
+				 <origin xyz="1 1 1" rpy="0 0 0"/>
+				 <parent link="${prefix}front_case_link"/>
+				 <child link="head"/>
+		</joint>
+		<link name="head">
+		    <visual>
+		        <origin xyz="0 0 0" rpy="0 0 0" />
+		        <geometry>
+							<box size="0.1 0.1 0.1"/>
+		        </geometry>
+		    </visual>
+		    <collision>
+		      <origin xyz="0 0 0" rpy="0 0 0" />
+		      <geometry>
+						<box size="0.1 0.1 0.1"/>
+		      </geometry>
+		    </collision>
+		    <inertial>
+		        <origin xyz="0 0 0" rpy="0 0 0" />
+		        <mass value="1" />
+		        <inertia
+		          ixx="1.0" ixy="0.0" ixz="0.0"
+		          iyy="1.0" iyz="0.0"
+		          izz="1.0" />
+		    </inertial>
+		</link>
+		<!-- this one doesn't work correctly because it is attached to a fixed link -->
+		<gazebo reference="head">
+		  <projector name="projector_test_head">
+		    <!-- none of the translations or rotations applied here have any effect -->
+		    <pose>0 0 0 1.57 0 0</pose>
+		    <texture>red.png</texture>
+		    <fov>0.95</fov>
+		    <near_clip>0.1</near_clip>
+		    <far_clip>10.0</far_clip>
+				<!--texture>stereo_projection_pattern_high_res_red.png</texture-->
+		  </projector>
+		</gazebo>
+		<!-- try putting a projector onto another link -->
+		<joint name="joint_projector_test_1" type="revolute">
+		  <parent link="head" />
+		  <child link="link_projector_test_1" />
+		  <origin xyz="0 0.23 0" rpy="0 0 0" />
+		  <axis xyz="0 1 0" />
+		  <limit effort="1000.0" upper="0.0001" lower="-0.0001" velocity="0.5" />
+		</joint>
+		<!-- this works fine because it is attached to a revolute jointed link-->
+		<link name="link_projector_test_1">
+		    <visual>
+		      <origin xyz="0 0 0" rpy="0 0 0" />
+		      <geometry>
+		        <box size="0.05 0.05 0.05"/>
+		      </geometry>
+		    </visual>
+		    <collision>
+		      <origin xyz="0 0 0" rpy="0 0 0" />
+		      <geometry>
+		        <box size="0.05 0.05 0.05"/>
+		      </geometry>
+		    </collision>
+		    <inertial>
+		        <origin xyz="0 0 0" rpy="0 0 0" />
+		        <mass value="1" />
+		        <inertia
+		          ixx="1.0" ixy="0.0" ixz="0.0"
+		          iyy="1.0" iyz="0.0"
+		          izz="1.0" />
+		    </inertial>
+		</link>
+		<gazebo reference="link_projector_test_1">
+		  <projector name="projector_test_1">
+		    <!-- setting the pose will produce glitches even when attached to a revolute joint -->
+		    <pose>0 0 0 0 1.57 0</pose>
+		    <texture>red.png</texture>
+		    <!--texture>stereo_projection_pattern_high_res_red.png</texture-->
+		    <fov>0.95</fov>
+		    <near_clip>0.1</near_clip>
+		    <far_clip>10.0</far_clip>
+		  </projector>
+		</gazebo>
+		 <!--PROJECTOR no funciona-->
+		 <!--joint name="${prefix}projector_joint" type="revolute">
+        <origin xyz="0 0 0" rpy="0 0 0"/>
+        <parent link="${prefix}front_case_link"/>
+        <child link="${prefix}projector_link"/>
+				<limit effort="0.01" velocity="0.01" upper="0.0001" lower="-0.0001"/>
+      </joint>
+			<link name="${prefix}projector_link">
+			</link>
+		 <gazebo reference="${prefix}projector_link">
+			 <projector name="projector">
+				 <pose>0 0 0 0 0 0</pose>
+         <texture>red.png</texture>
+         <fov>0.95</fov>
+         <near_clip>0.1</near_clip>
+         <far_clip>10</far_clip>
+     	 </projector>
+		 </gazebo>
 		 <gazebo>
+     		<plugin name="projector" filename="libgazebo_ros_projector.so">
+         	<projector>${prefix}projector_link/projector</projector>
+         	<alwaysOn>true</alwaysOn>
+         	<updateRate>10.0</updateRate>
+					<textureName>red.png</textureName>
+					<filterTextureName>red.png</filterTextureName>
+         	<textureTopicName>/projector/image</textureTopicName>
+         	<projectorTopicName>/projector/projector</projectorTopicName>
+     		</plugin>
+			</gazebo-->
+<!-- LEDS -->
+		 <!--gazebo>
 		   <model name='light_model'>
 		     <pose>1.5207 0 0.68 0 0 0</pose>
@@ -59,5 +171,5 @@
 		         <attenuation>
 		           <range>20</range>
-		           <!--linear>0.10</linear-->
+		           <!- -linear>0.10</linear- ->
 		         </attenuation>
 		         <diffuse>0 0 0 1</diffuse>
@@ -73,5 +185,5 @@
 		         <attenuation>
 		           <range>20</range>
-		           <!--linear>0.10</linear-->
+		           <!- -linear>0.10</linear- ->
 		         </attenuation>
 		         <diffuse>0 0 0 1</diffuse>
@@ -132,5 +244,5 @@
 		     </plugin>
 		   </model>
-		   </gazebo>
+		 </gazebo>
 		   <gazebo>
 		     <joint name='light_joint' type='fixed'>
@@ -138,5 +250,5 @@
 		       <child>light_model::light_link</child>
 		     </joint>
-		   </gazebo>
+		   </gazebo-->
   </xacro:macro>
 </robot>

Commit message: Changed to a relative path for the image. Added led xacro. For lighting -> service call.

File: pallet_truck_common/pallet_truck_description/urdf/bases/front_case.urdf.xacro (robot description, xacro)
@@ -2,4 +2,5 @@
 <robot xmlns:xacro="http://www.ros.org/wiki/xacro">
 	<xacro:include filename="$(find pallet_truck_description)/urdf/projector/projector.urdf.xacro" />
+	<xacro:include filename="$(find pallet_truck_description)/urdf/led/led2.urdf.xacro" />
 	<xacro:property name="front_case_mass" value="10" />
 	<xacro:property name="PI" value="3.1415926535897931"/>
@@ -39,112 +40,13 @@
      </link>
 		 <xacro:line_projector prefix="${prefix}left_" parent="${prefix}front_case_link">
-	      <origin xyz="-0.2 -0.5 0.2" rpy="0 0 0" />
+	      <origin xyz="0.2 -0.5 0.2" rpy="0 0 0" />
 	   </xacro:line_projector>
 		 <xacro:line_projector prefix="${prefix}right_" parent="${prefix}battery_case_link">
-				<origin xyz="-0.1993 0.43 0.197" rpy="0 0 0" />
+				<origin xyz="0.1993 0.43 0.197" rpy="0 0 0" />
 		 </xacro:line_projector>
-<!-- LEDS -->
-		 <gazebo>
-		   <model name='light_model'>
-		     <pose>1.5207 0 0.68 0 0 0</pose>
-		     <link name='light_link'>
-		       <visual name='light_source'>
-		         <pose>0 0 0 0 0 0</pose>
-		         <geometry>
-		           <box>
-		             <size>0.35 0.568 0.01</size>
-		           </box>
-		         </geometry>
-		         <material>
-		           <ambient>1 1 1 1</ambient>
-		           <diffuse>1 1 1 1</diffuse>
-		           <specular>1 1 1 1</specular>
-		           <emissive>0 0 0 1</emissive>
-		         </material>
-		       </visual>
-		       <light name='light_source' type='point'>
-		         <pose>0 0.276 0 0 0 0</pose>
-		         <attenuation>
-		           <range>20</range>
-		           <!--linear>0.10</linear-->
-		         </attenuation>
-		         <diffuse>0 0 0 1</diffuse>
-		         <specular>0 0 0 1</specular>
-						 <spot>
-							 <inner_angle>0.1</inner_angle>
-							 <outer_angle>0.15</outer_angle>
-							 <falloff>1</falloff>
-						 </spot>
-		       </light>
-					 <light name='light_source2' type='point'>
-		         <pose>0 -0.276 0 0 0 0</pose>
-		         <attenuation>
-		           <range>20</range>
-		           <!--linear>0.10</linear-->
-		         </attenuation>
-		         <diffuse>0 0 0 1</diffuse>
-		         <specular>0 0 0 1</specular>
-						 <spot>
-							 <inner_angle>0.1</inner_angle>
-							 <outer_angle>0.15</outer_angle>
-							 <falloff>1</falloff>
-						 </spot>
-		       </light>
-		     </link>
-		     <plugin name='light_control' filename='libLedPlugin.so'>
-		 			<enable>true</enable>
-		       <light>
-		         <id>light_link/light_source</id>
-						 <block>
-							 <enable>true</enable>
-						 	 <duration>1</duration>
-						 	 <interval>0.5</interval>
-						 	 <color>1 0 0</color>
-						 	 <attenuation>
-						 	 		<range>20</range>
-						 	 		<linear>0.10</linear>
-						 	 </attenuation>
-						 </block>
-						 <block>
-						 	 <duration>1</duration>
-						 	 <interval>0.5</interval>
-						   <color>1 0 0</color>
-						 	 <attenuation>
-						 			 <range>20</range>
-						 			 <linear>0.10</linear>
-						 	 </attenuation>
-						  </block>
-					 </light>
-					 <light>
-						 <id>light_link/light_source2</id>
-						 <block>
-							 <enable>true</enable>
-							 <duration>1</duration>
-							 <interval>0.5</interval>
-							 <color>1 0 0</color>
-							 <attenuation>
-									<range>20</range>
-									<linear>0.10</linear>
-							 </attenuation>
-						 </block>
-						 <block>
-							 <duration>1</duration>
-							 <interval>0.5</interval>
-							 <color>1 0 0</color>
-							 <attenuation>
-									 <range>20</range>
-									 <linear>0.10</linear>
-							 </attenuation>
-							</block>
-					 </light>
-		     </plugin>
-		   </model>
-		 </gazebo>
-		   <gazebo>
-		     <joint name='light_joint' type='fixed'>
-		       <parent>${prefix}front_case_link</parent>
-		       <child>light_model::light_link</child>
-		     </joint>
-		   </gazebo>
+		 <!--xacro:led prefix="${prefix}">
+		 </xacro:led-->
+		 <xacro:led prefix="${prefix}">
+		 </xacro:led>
   </xacro:macro>
 </robot>
