Commit message: Inertia is calculated with inertia's macro

File: pallet_truck_common/pallet_truck_description/urdf/bases/battery_case.urdf.xacro (robot description, xacro)
@@ -5,9 +5,18 @@
       <!-- Robot mechanical and motor parameters -->
   <xacro:property name="battery_case_mass" value="10"/>
+  <xacro:property name="battery_case_size_x" value="0.38"/>
+  <xacro:property name="battery_case_size_y" value="0.57"/>
+  <xacro:property name="battery_case_size_z" value="0.68"/>
   <xacro:property name="fork_offset_x" value="-0.4325"/>
   <xacro:property name="fork_offset_y" value="0.201"/>
   <xacro:property name="fork_offset_z" value="-0.662"/>
   <xacro:property name="PI" value="3.1415926535897931"/>
-  <xacro:macro name="battery_case" params="prefix parent *origin">
+  <xacro:macro name="solid_cuboid_inertia" params="m h d w">
+    <inertia  ixx="${(m*(h*h+d*d))/12}" ixy = "0" ixz = "0"
+              iyy="${(m*(w*w+d*d))/12}" iyz = "0"
+              izz="${(m*(w*w+h*h))/12}"
+     />
+  </xacro:macro>
+ <xacro:macro name="battery_case" params="prefix parent *origin">
   <joint name="${prefix}elevator_joint" type="prismatic">
     <xacro:insert_block name="origin" />
@@ -16,5 +25,5 @@
     <axis xyz="0 0 1"/>
     <limit effort="1000.0" lower="0" upper="0.106" velocity="1"/>
-</joint>
+  </joint>
   <link name="${prefix}battery_case_link">
     <visual>
@@ -32,7 +41,6 @@
     <inertial>
       <mass value="${battery_case_mass}" />
-      <origin xyz="-0.249758 0.0 -0.416592"/>
-      <!--inertia ixx="0.001371" ixy="-0.000021" ixz="-0.000146" iyy="0.000854" iyz="-0.000068" izz="0.000925"/-->
-      <inertia ixx="0.5824" ixy="0.0" ixz="0.0" iyy="0.5824" iyz="0.0" izz="0.4166"/>  <!-- Multiplicar por la masa -->
+      <origin xyz="-0.2 0.0 -0.35"/>
+      <solid_cuboid_inertia m="${battery_case_mass}" h="${battery_case_size_y}" d="${battery_case_size_z}" w="${battery_case_size_x}"/>
     </inertial>
   </link>
@@ -43,4 +51,11 @@
      <origin xyz="${fork_offset_x} -${fork_offset_y} ${fork_offset_z}" rpy="0 0 0" />
   </xacro:fork>
+  <!--gazebo reference="${prefix}battery_case_link">
+    <mu1 value="1"/>
+    <mu2 value="1"/>
+    <!- -kp>100000000.0</kp- ->
+    <!- -kd value="10.0"/- ->
+    <material>Gazebo/Black</material>
+  </gazebo-->
   <transmission name="${prefix}elevator_transmission">
     <type>transmission_interface/SimpleTransmission</type>

File: pallet_truck_common/pallet_truck_description/urdf/bases/front_case.urdf.xacro (robot description, xacro)
@@ -2,4 +2,14 @@
 <robot xmlns:xacro="http://www.ros.org/wiki/xacro">
 	<xacro:property name="front_case_mass" value="10" />
+	<xacro:property name="PI" value="3.1415926535897931"/>
+  <xacro:macro name="solid_cuboid_inertia" params="m h d w">
+    <inertia  ixx="${(m*(h*h+d*d))/12}" ixy = "0" ixz = "0"
+              iyy="${(m*(w*w+d*d))/12}" iyz = "0"
+              izz="${(m*(w*w+h*h))/12}"
+     />
+  </xacro:macro>
+	<xacro:property name="front_case_size_x" value="0.5"/>
+	<xacro:property name="front_case_size_y" value="0.5"/>
+	<xacro:property name="front_case_size_z" value="0.5"/>
   <xacro:macro name="front_case" params="prefix parent *origin">
     <joint name="${prefix}front_case_joint" type="fixed">
@@ -11,6 +21,6 @@
        <inertial>
          <mass value="${front_case_mass}" />
-         <origin xyz="0.226093 0.0 -0.285579" />
-         <inertia ixx="0.644" ixy="0.0" ixz="0.0" iyy="0.4944" iyz="0.0" izz="0.391"/>  <!-- Multiplicar por la masa -->
+         <origin xyz="0.226093 0.0 -0.31" />
+				 <solid_cuboid_inertia m="${front_case_mass}" h="${front_case_size_y}" d="${front_case_size_z}" w="${front_case_size_x}"/>
        </inertial>
        <visual>
@@ -27,4 +37,11 @@
        </collision>
      </link>
+		 <!--gazebo reference="${prefix}front_case_link">
+			 <mu1 value="1"/>
+			 <mu2 value="1"/>
+			 <kp>100000000.0</kp>
+			 <!- -kd value="10.0"/- ->
+			 <material>Gazebo/Black</material>
+		 </gazebo-->
   </xacro:macro>
 </robot>

File: pallet_truck_common/pallet_truck_description/urdf/bases/pallet_truck.urdf.xacro (robot description, xacro)
@@ -25,7 +25,6 @@
   <link name="${prefix}base_link">
     <inertial>
-      <mass value="${base_mass}" />
-      <origin xyz="0 0 0" />
-      <solid_cuboid_inertia  m="${base_mass}" d="${base_length}" w="${base_length}" h="${base_length}"/>
+      <mass value="0.0001"/>
+      <inertia ixx="0.4" ixy="0.0" ixz="0.0" iyy="0.4" iyz="0.0" izz="0.2"/>
     </inertial>
   </link>

Commit message: Changed mass values (correct the sliding)

File: pallet_truck_common/pallet_truck_description/urdf/bases/battery_case.urdf.xacro (robot description, xacro)
@@ -4,5 +4,5 @@
   <xacro:include filename="$(find pallet_truck_description)/urdf/elevator/fork.urdf.xacro" />
       <!-- Robot mechanical and motor parameters -->
-  <xacro:property name="battery_case_mass" value="10"/>
+  <xacro:property name="battery_case_mass" value="5"/>
   <xacro:property name="battery_case_size_x" value="0.38"/>
   <xacro:property name="battery_case_size_y" value="0.57"/>

File: pallet_truck_common/pallet_truck_description/urdf/bases/front_case.urdf.xacro (robot description, xacro)
@@ -1,5 +1,5 @@
 <?xml version="1.0"?>
 <robot xmlns:xacro="http://www.ros.org/wiki/xacro">
-	<xacro:property name="front_case_mass" value="10" />
+	<xacro:property name="front_case_mass" value="5" />
 	<xacro:property name="PI" value="3.1415926535897931"/>
   <xacro:macro name="solid_cuboid_inertia" params="m h d w">

File: pallet_truck_common/pallet_truck_description/urdf/wheels/motor_wheel.urdf.xacro (robot description, xacro)
@@ -4,5 +4,5 @@
   <xacro:property name="wheel_radius" value="0.122" />
   <xacro:property name="wheel_width" value="0.1" />
-  <xacro:property name="wheel_mass" value="1" /><!-- in kg-->
+  <xacro:property name="wheel_mass" value="10" /><!-- in kg-->
   <!-- Steer wheel properties -->
   <xacro:property name="steer_joint_damping" value="1000" />

Commit message: Changed masses and added a protection for battery-case

File: pallet_truck_common/pallet_truck_description/urdf/bases/battery_case.urdf.xacro (robot description, xacro)
@@ -3,6 +3,7 @@
   <xacro:include filename="$(find pallet_truck_description)/urdf/inertia.urdf.xacro" />
   <xacro:include filename="$(find pallet_truck_description)/urdf/elevator/fork.urdf.xacro" />
+  <xacro:include filename="$(find pallet_truck_description)/urdf/bases/protection.urdf.xacro" />
       <!-- Robot mechanical and motor parameters -->
-  <xacro:property name="battery_case_mass" value="5"/>
+  <xacro:property name="battery_case_mass" value="10"/>
   <xacro:property name="battery_case_size_x" value="0.38"/>
   <xacro:property name="battery_case_size_y" value="0.57"/>
@@ -24,5 +25,5 @@
     <child link="${prefix}battery_case_link" />
     <axis xyz="0 0 1"/>
-    <limit effort="1000.0" lower="0" upper="0.106" velocity="1"/>
+    <limit effort="1000.0" lower="0" upper="0.106" velocity="0.1"/>
   </joint>
   <link name="${prefix}battery_case_link">
@@ -51,4 +52,7 @@
      <origin xyz="${fork_offset_x} -${fork_offset_y} ${fork_offset_z}" rpy="0 0 0" />
   </xacro:fork>
+  <xacro:protection prefix="${prefix}battery_case_" parent="${prefix}battery_case_link" measurement="0.001 0.52 0.5204">
+     <origin xyz="-0.439 0 -0.42" rpy="0 0 0" />
+  </xacro:protection>
   <!--gazebo reference="${prefix}battery_case_link">
     <mu1 value="1"/>

File: pallet_truck_common/pallet_truck_description/urdf/bases/front_case.urdf.xacro (robot description, xacro)
@@ -1,5 +1,5 @@
 <?xml version="1.0"?>
 <robot xmlns:xacro="http://www.ros.org/wiki/xacro">
-	<xacro:property name="front_case_mass" value="5" />
+	<xacro:property name="front_case_mass" value="10" />
 	<xacro:property name="PI" value="3.1415926535897931"/>
   <xacro:macro name="solid_cuboid_inertia" params="m h d w">
@@ -21,5 +21,5 @@
        <inertial>
          <mass value="${front_case_mass}" />
-         <origin xyz="0.226093 0.0 -0.31" />
+         <origin xyz="0.226093 0.0 -0.31"/>
 				 <solid_cuboid_inertia m="${front_case_mass}" h="${front_case_size_y}" d="${front_case_size_z}" w="${front_case_size_x}"/>
        </inertial>

File: pallet_truck_common/pallet_truck_description/urdf/bases/pallet_truck.urdf.xacro (robot description, xacro)
@@ -3,9 +3,4 @@
   <xacro:include filename="$(find pallet_truck_description)/urdf/inertia.urdf.xacro" />
 	<xacro:property name="PI" value="3.1415926535897931"/>
-  <!-- Robot mechanical and motor parameters -->
-  <xacro:property name="base_length" value="0.0001" />
-  <xacro:property name="base_width" value="0.0001" />
-  <xacro:property name="base_height" value="0.0001" />
-  <xacro:property name="base_mass" value="0.0001"/>
   <xacro:property name="base_link_origin" value="0 0 0.040" /> <!--base_link (0,0,fork_wheel_radius) RF-> Base_Footprint. Align with the centers of fork_wheels.-->
   <xacro:macro name="pallet_truck" params="prefix publish_bf">

File: pallet_truck_common/pallet_truck_description/urdf/elevator/fork.urdf.xacro (robot description, xacro)
@@ -31,4 +31,10 @@
            <mesh filename="package://pallet_truck_description/meshes/elevator/single_fork.stl"/>
          </geometry>
+         <friction>
+           <ode>
+             <mu>100</mu>
+             <mu2>100</mu2>
+           </ode>
+         </friction>
        </collision>
      </link>
@@ -48,6 +54,6 @@
      <!-- FORK LINK -->
      <gazebo reference="${prefix}fork_link">
-       <mu1>100000</mu1>
-       <mu2>100000</mu2>
+       <mu1>100</mu1>
+       <mu2>100</mu2>
        <material>Gazebo/Black</material>
      </gazebo>

Commit message: Projector works, two lines

File: pallet_truck_common/pallet_truck_description/urdf/bases/battery_case.urdf.xacro (robot description, xacro)
@@ -55,4 +55,20 @@
      <origin xyz="-0.439 0 -0.42" rpy="0 0 0" />
   </xacro:protection>
+  		<!--joint name="${prefix}right_projector_joint" type="fixed">
+  			<origin xyz="1 -1 1" rpy="0 0 0"/>
+  			<parent link="${prefix}battery_case_link"/>
+  			<child link="${prefix}right_line_projector"/>
+  		</joint>
+  		<link name="${prefix}right_line_projector">
+  		</link>
+  		<gazebo reference="${prefix}right_line_projector">
+  			<projector name="projector_test_right">
+  	    	<pose>0 0 0 1.57 0 0</pose>
+  	    	<texture>red1.png</texture>
+  	    	<fov>0.95</fov>
+  	    	<near_clip>0.1</near_clip>
+        	<far_clip>10.0</far_clip>
+  			</projector>
+  		</gazebo-->
   <!--gazebo reference="${prefix}battery_case_link">
     <mu1 value="1"/>

File: pallet_truck_common/pallet_truck_description/urdf/bases/front_case.urdf.xacro (robot description, xacro)
@@ -1,4 +1,5 @@
 <?xml version="1.0"?>
 <robot xmlns:xacro="http://www.ros.org/wiki/xacro">
+	<xacro:include filename="$(find pallet_truck_description)/urdf/projector/projector.urdf.xacro" />
 	<xacro:property name="front_case_mass" value="10" />
 	<xacro:property name="PI" value="3.1415926535897931"/>
@@ -37,115 +38,10 @@
        </collision>
      </link>
-		 <!--PROJECTOR -->
-		 <joint name="${prefix}projector_joint" type="fixed">
-				 <origin xyz="1 1 1" rpy="0 0 0"/>
-				 <parent link="${prefix}front_case_link"/>
-				 <child link="head"/>
-		</joint>
-		<link name="head">
-		    <visual>
-		        <origin xyz="0 0 0" rpy="0 0 0" />
-		        <geometry>
-							<box size="0.1 0.1 0.1"/>
-		        </geometry>
-		    </visual>
-		    <collision>
-		      <origin xyz="0 0 0" rpy="0 0 0" />
-		      <geometry>
-						<box size="0.1 0.1 0.1"/>
-		      </geometry>
-		    </collision>
-		    <inertial>
-		        <origin xyz="0 0 0" rpy="0 0 0" />
-		        <mass value="1" />
-		        <inertia
-		          ixx="1.0" ixy="0.0" ixz="0.0"
-		          iyy="1.0" iyz="0.0"
-		          izz="1.0" />
-		    </inertial>
-		</link>
-		<!-- this one doesn't work correctly because it is attached to a fixed link -->
-		<gazebo reference="head">
-		  <projector name="projector_test_head">
-		    <!-- none of the translations or rotations applied here have any effect -->
-		    <pose>0 0 0 1.57 0 0</pose>
-		    <texture>red.png</texture>
-		    <fov>0.95</fov>
-		    <near_clip>0.1</near_clip>
-		    <far_clip>10.0</far_clip>
-				<!--texture>stereo_projection_pattern_high_res_red.png</texture-->
-		  </projector>
-		</gazebo>
-		<!-- try putting a projector onto another link -->
-		<joint name="joint_projector_test_1" type="revolute">
-		  <parent link="head" />
-		  <child link="link_projector_test_1" />
-		  <origin xyz="0 0.23 0" rpy="0 0 0" />
-		  <axis xyz="0 1 0" />
-		  <limit effort="1000.0" upper="0.0001" lower="-0.0001" velocity="0.5" />
-		</joint>
-		<!-- this works fine because it is attached to a revolute jointed link-->
-		<link name="link_projector_test_1">
-		    <visual>
-		      <origin xyz="0 0 0" rpy="0 0 0" />
-		      <geometry>
-		        <box size="0.05 0.05 0.05"/>
-		      </geometry>
-		    </visual>
-		    <collision>
-		      <origin xyz="0 0 0" rpy="0 0 0" />
-		      <geometry>
-		        <box size="0.05 0.05 0.05"/>
-		      </geometry>
-		    </collision>
-		    <inertial>
-		        <origin xyz="0 0 0" rpy="0 0 0" />
-		        <mass value="1" />
-		        <inertia
-		          ixx="1.0" ixy="0.0" ixz="0.0"
-		          iyy="1.0" iyz="0.0"
-		          izz="1.0" />
-		    </inertial>
-		</link>
-		<gazebo reference="link_projector_test_1">
-		  <projector name="projector_test_1">
-		    <!-- setting the pose will produce glitches even when attached to a revolute joint -->
-		    <pose>0 0 0 0 1.57 0</pose>
-		    <texture>red.png</texture>
-		    <!--texture>stereo_projection_pattern_high_res_red.png</texture-->
-		    <fov>0.95</fov>
-		    <near_clip>0.1</near_clip>
-		    <far_clip>10.0</far_clip>
-		  </projector>
-		</gazebo>
-		 <!--PROJECTOR no funciona-->
-		 <!--joint name="${prefix}projector_joint" type="revolute">
-        <origin xyz="0 0 0" rpy="0 0 0"/>
-        <parent link="${prefix}front_case_link"/>
-        <child link="${prefix}projector_link"/>
-				<limit effort="0.01" velocity="0.01" upper="0.0001" lower="-0.0001"/>
-      </joint>
-			<link name="${prefix}projector_link">
-			</link>
-		 <gazebo reference="${prefix}projector_link">
-			 <projector name="projector">
-				 <pose>0 0 0 0 0 0</pose>
-         <texture>red.png</texture>
-         <fov>0.95</fov>
-         <near_clip>0.1</near_clip>
-         <far_clip>10</far_clip>
-     	 </projector>
-		 </gazebo>
-		 <gazebo>
-     		<plugin name="projector" filename="libgazebo_ros_projector.so">
-         	<projector>${prefix}projector_link/projector</projector>
-         	<alwaysOn>true</alwaysOn>
-         	<updateRate>10.0</updateRate>
-					<textureName>red.png</textureName>
-					<filterTextureName>red.png</filterTextureName>
-         	<textureTopicName>/projector/image</textureTopicName>
-         	<projectorTopicName>/projector/projector</projectorTopicName>
-     		</plugin>
-			</gazebo-->
+		 <xacro:line_projector prefix="${prefix}left_" parent="${prefix}front_case_link">
+	      <origin xyz="-0.2 -0.5 0.2" rpy="0 0 0" />
+	   </xacro:line_projector>
+		 <xacro:line_projector prefix="${prefix}right_" parent="${prefix}battery_case_link">
+				<origin xyz="-0.1993 0.43 0.197" rpy="0 0 0" />
+		 </xacro:line_projector>
 <!-- LEDS -->
 		 <!--gazebo>

Commit message: added materials to urdf, from gazebo

File: pallet_truck_common/pallet_truck_description/urdf/bases/battery_case.urdf.xacro (robot description, xacro)
@@ -33,4 +33,7 @@
         <mesh filename="package://pallet_truck_description/meshes/bases/battery_case.stl"/>
       </geometry>
+     <material name="black">
+       <color rgba="0.0 0.0 0.0 1.0"/>
+     </material>
     </visual>
     <collision>

File: pallet_truck_common/pallet_truck_description/urdf/bases/front_case.urdf.xacro (robot description, xacro)
@@ -31,4 +31,7 @@
            <mesh filename="package://pallet_truck_description/meshes/bases/front_case.stl"/>
          </geometry>
+         <material name="black">
+           <color rgba="0.0 0.0 0.0 1.0"/>
+         </material>
        </visual>
        <collision>

File: pallet_truck_common/pallet_truck_description/urdf/elevator/fork.urdf.xacro (robot description, xacro)
@@ -25,4 +25,7 @@
            <mesh filename="package://pallet_truck_description/meshes/elevator/single_fork.stl"/>
          </geometry>
+         <material name="dark_grey">
+           <color rgba="0.2 0.2 0.2 1.0"/>
+         </material>
        </visual>
        <collision>
@@ -56,5 +59,4 @@
        <mu1>100</mu1>
        <mu2>100</mu2>
-       <material>Gazebo/Black</material>
      </gazebo>
     <joint name="${prefix}fork_sensor_joint" type="fixed">

File: pallet_truck_common/pallet_truck_description/urdf/wheels/castor_wheel.urdf.xacro (robot description, xacro)
@@ -26,7 +26,10 @@
         <origin xyz="0 0 0" rpy="0 0 0" />
         <geometry>
-				  <!--mesh filename="package://pallet_truck_description/meshes/wheels/pallet_truck_wheel_fake.dae"/-->
+		  <!--mesh filename="package://pallet_truck_description/meshes/wheels/pallet_truck_wheel_fake.dae"/-->
           <sphere radius="${castor_wheel_radius}"/>
         </geometry>
+        <material name="black">
+          <color rgba="0.0 0.0 0.0 1.0"/>
+        </material>
       </visual>
       <collision>
@@ -56,5 +59,4 @@
 		    <mu2 value="0.0"/>
 		    <fdir1 value="1 0 0"/>
-		    <material>Gazebo/Black</material>
         <turnGravityOff>false</turnGravityOff>
     </gazebo>

File: pallet_truck_common/pallet_truck_description/urdf/wheels/fork_wheel.urdf.xacro (robot description, xacro)
@@ -29,4 +29,7 @@
           <sphere radius="${fork_wheel_radius}"/>
         </geometry>
+        <material name="black">
+          <color rgba="0.0 0.0 0.0 1.0"/>
+        </material>
       </visual>
       <collision>
@@ -56,5 +59,4 @@
 		    <mu2 value="0.5"/>
 		    <fdir1 value="1 0 0"/>
-		    <material>Gazebo/Black</material>
         <turnGravityOff>false</turnGravityOff>
     </gazebo>

File: pallet_truck_common/pallet_truck_description/urdf/wheels/motor_wheel.urdf.xacro (robot description, xacro)
@@ -64,4 +64,7 @@
           <!--cylinder length="${wheel_width}" radius="${0.12675}"/-->
         </geometry>
+        <material name="black">
+          <color rgba="0.0 0.0 0.0 1.0"/>
+        </material>
       </visual>
       <collision>
@@ -88,5 +91,4 @@
       <kp>100000000</kp>
       <kd>10</kd>
-      <material>Gazebo/Black</material>
     </gazebo>
     <!-- ************* -->

Commit message: switched from black to gray

File: pallet_truck_common/pallet_truck_description/urdf/bases/battery_case.urdf.xacro (robot description, xacro)
@@ -33,7 +33,7 @@
         <mesh filename="package://pallet_truck_description/meshes/bases/battery_case.stl"/>
       </geometry>
-     <material name="black">
-       <color rgba="0.0 0.0 0.0 1.0"/>
-     </material>
+      <material name="dark_grey">
+        <color rgba="0.4 0.4 0.4 1.0"/>
+      </material>
     </visual>
     <collision>

File: pallet_truck_common/pallet_truck_description/urdf/bases/front_case.urdf.xacro (robot description, xacro)
@@ -31,6 +31,6 @@
            <mesh filename="package://pallet_truck_description/meshes/bases/front_case.stl"/>
          </geometry>
-         <material name="black">
-           <color rgba="0.0 0.0 0.0 1.0"/>
+         <material name="dark_grey">
+           <color rgba="0.4 0.4 0.4 1.0"/>
          </material>
        </visual>

File: pallet_truck_common/pallet_truck_description/urdf/elevator/fork.urdf.xacro (robot description, xacro)
@@ -26,5 +26,5 @@
          </geometry>
          <material name="dark_grey">
-           <color rgba="0.2 0.2 0.2 1.0"/>
+           <color rgba="0.4 0.4 0.4 1.0"/>
          </material>
        </visual>

File: pallet_truck_common/pallet_truck_description/urdf/wheels/castor_wheel.urdf.xacro (robot description, xacro)
@@ -29,6 +29,6 @@
           <sphere radius="${castor_wheel_radius}"/>
         </geometry>
-        <material name="black">
-          <color rgba="0.0 0.0 0.0 1.0"/>
+        <material name="dark_grey">
+          <color rgba="0.4 0.4 0.4 1.0"/>
         </material>
       </visual>

File: pallet_truck_common/pallet_truck_description/urdf/wheels/fork_wheel.urdf.xacro (robot description, xacro)
@@ -29,6 +29,6 @@
           <sphere radius="${fork_wheel_radius}"/>
         </geometry>
-        <material name="black">
-          <color rgba="0.0 0.0 0.0 1.0"/>
+        <material name="dark_grey">
+          <color rgba="0.4 0.4 0.4 1.0"/>
         </material>
       </visual>

File: pallet_truck_common/pallet_truck_description/urdf/wheels/motor_wheel.urdf.xacro (robot description, xacro)
@@ -64,6 +64,6 @@
           <!--cylinder length="${wheel_width}" radius="${0.12675}"/-->
         </geometry>
-        <material name="black">
-          <color rgba="0.0 0.0 0.0 1.0"/>
+        <material name="dark_grey">
+          <color rgba="0.4 0.4 0.4 1.0"/>
         </material>
       </visual>
