Commit message: Changed the names of the xacro-properties
At each wheel xacro the name of the wheel properties was the same and this produced that sometimes the value of certain parameters was not the desired one.

File: pallet_truck_common/pallet_truck_description/urdf/elevator/fork.urdf.xacro (robot description, xacro)
@@ -16,6 +16,6 @@
      <link name="${prefix}fork_link">
        <inertial>
+         <origin xyz="-0.581270 0.00000 0.012941" />
          <mass value="${fork_mass}" />
-         <origin xyz="-0.581270 0.000014 0.012941" />
          <solid_cuboid_inertia m="${fork_mass}" h="${fork_width}" d="${fork_height}" w="${fork_length}"/>
        </inertial>

File: pallet_truck_common/pallet_truck_description/urdf/wheels/castor_wheel.urdf.xacro (robot description, xacro)
@@ -3,7 +3,7 @@
   <xacro:property name="M_PI" value="3.1415926535897931" />
   <!-- Wheels -->
-  <xacro:property name="wheel_radius" value="0.040" />
-  <xacro:property name="wheel_height" value="0.080" />
-  <xacro:property name="wheel_mass" value="0.5" />
+  <xacro:property name="castor_wheel_radius" value="0.040" />
+  <xacro:property name="castor_wheel_height" value="0.080" />
+  <xacro:property name="castor_wheel_mass" value="0.5" />
   <xacro:macro name="cylinder_inertia" params="m r h">
     <inertia  ixx="${m*(3*r*r+h*h)/12}" ixy = "0" ixz = "0"
@@ -27,5 +27,5 @@
         <geometry>
 				  <!--mesh filename="package://pallet_truck_description/meshes/wheels/pallet_truck_wheel_fake.dae"/-->
-          <sphere radius="${wheel_radius}"/>
+          <sphere radius="${castor_wheel_radius}"/>
         </geometry>
       </visual>
@@ -33,9 +33,9 @@
         <origin xyz="0 0 0" rpy="${M_PI/2} 0 0" />
         <geometry>
-          <sphere radius="${wheel_radius}"/>
+          <sphere radius="${castor_wheel_radius}"/>
         </geometry>
       </collision>
       <inertial>
-        <mass value="${wheel_mass}" />
+        <mass value="${castor_wheel_mass}" />
         <origin xyz="0 0 0" />
         <inertia  ixx="0.00064" ixy="0.0"  ixz="0.0"  iyy="0.00064"  iyz="0.0"  izz="0.00064" />

File: pallet_truck_common/pallet_truck_description/urdf/wheels/fork_wheel.urdf.xacro (robot description, xacro)
@@ -4,10 +4,10 @@
   <!-- Wheels -->
   <xacro:property name="fork_wheel_radius" value="0.040" />
-  <xacro:property name="fork_wheel_height" value="0.080" />
+  <xacro:property name="fork_wheel_length" value="0.080" />
   <xacro:property name="fork_wheel_mass" value="0.5" />
   <xacro:macro name="cylinder_inertia" params="m r h">
     <inertia  ixx="${m*(3*r*r+h*h)/12}" ixy = "0" ixz = "0"
-              iyy="${m*(3*r*r+h*h)/12}" iyz = "0"
-              izz="${m*r*r/2}"
+              iyy="${m*r*r/2}" iyz = "0"
+              izz="${m*(3*r*r+h*h)/12}"
      />
   </xacro:macro>
@@ -37,7 +37,7 @@
       </collision>
       <inertial>
-        <mass value="${wheel_mass}" />
+        <mass value="${fork_wheel_mass}" />
         <origin xyz="0 0 0" />
-        <inertia  ixx="0.00064" ixy="0.0"  ixz="0.0"  iyy="0.00064"  iyz="0.0"  izz="0.00064" />
+        <cylinder_inertia  m="${fork_wheel_mass}" r="${fork_wheel_radius}" h="${fork_wheel_length}" />
       </inertial>
     </link>
