Commit message: Direction of moved has been changed

File: pallet_truck_common/pallet_truck_description/urdf/wheels/motor_wheel.urdf.xacro (robot description, xacro)
@@ -49,5 +49,5 @@
       <child link="${prefix}wheel_traction_link"/>
       <origin xyz="${traction_origin}" rpy="0 0 0" />
-      <axis xyz="0 1 0" rpy="0 0 0" />
+      <axis xyz="0 -1 0" rpy="0 0 0" />
       <limit effort="${traction_joint_effort_limit}" velocity="${traction_joint_velocity_limit}" />
       <dynamics damping="${traction_joint_damping}" friction="${traction_joint_friction}"/>

Commit message: Changed friction values.
The simulation is working well (it's necessary to check the odometry)

File: pallet_truck_common/pallet_truck_description/urdf/wheels/motor_wheel.urdf.xacro (robot description, xacro)
@@ -22,5 +22,8 @@
   <!-- inertial equation -->
   <xacro:macro name="cylinder_inertia" params="m r h">
-    <inertia ixx="${m*(3*r*r+h*h)/12}" ixy = "0" ixz = "0" iyy="${m*(3*r*r+h*h)/12}" iyz = "0" izz="${m*r*r/2}" />
+    <inertia  ixx="${m*(3*r*r+h*h)/12}" ixy = "0" ixz = "0"
+              iyy="${m*r*r/2}" iyz = "0"
+              izz="${m*(3*r*r+h*h)/12}"
+     />
   </xacro:macro>
   <!-- *********** -->
@@ -73,5 +76,5 @@
         <mass value="${wheel_mass}" />
         <origin xyz="0.000063 0 0.000465"/>
-        <inertia ixx="0.0064" ixy="0.0" ixz="0.0" iyy="0.00496" iyz="0.0" izz="0.0064"/>  <!-- Multiplicar por la masa -->
+        <cylinder_inertia  m="${wheel_mass}" r="${wheel_radius}" h="${wheel_width}" />
       </inertial>
     </link>
@@ -81,6 +84,8 @@
     <!-- TRACTION LINK -->
     <gazebo reference="${prefix}front_wheel_link">
-      <mu1>1000</mu1>
-      <mu2>1000</mu2>
+      <mu1>1</mu1>
+      <mu2>1</mu2>
+      <kp>100000000</kp>
+      <kd>10</kd>
       <material>Gazebo/Black</material>
     </gazebo>
