Commit message: Working on it. Additional wheels have continuous joints, normally these are fixed, but there's a bug with the inertia here. When the joint is fixed, inertia is like a big box with wrong directions, when the joint is revolute it has a normal behavior.

File: pallet_truck_common/pallet_truck_description/robots/pallet_truck_std.urdf.xacro (robot description, xacro)
@@ -9,4 +9,6 @@
 	<!-- Import HR-RECYCLER wheels -->
 	<xacro:include filename="$(find pallet_truck_description)/urdf/wheels/motor_wheel.urdf.xacro" />
+  <!-- Import HR-RECYCLER additional wheels -->
+  <xacro:include filename="$(find pallet_truck_description)/urdf/wheels/additional_wheel.urdf.xacro" />
   <!-- Import HR-RECYCLER elevator -->
   <xacro:include filename="$(find pallet_truck_description)/urdf/elevator/elevator.urdf.xacro" />
@@ -21,13 +23,13 @@
 	<xacro:property name="wheel_offset_x" value="0.0"/>
 	<xacro:property name="wheel_offset_y" value="0.0"/>
-	<xacro:property name="wheel_offset_z" value="0.46"/>
+	<xacro:property name="wheel_offset_z" value="0.0"/>
 	<!-- Flag to select the high or low quality model -->
 	<xacro:property name="hq" value="true" />
 	<!--  FORK CAMERAS  -->
-  <xacro:property name="fork_camera_x" value="-1.539" />
+  <xacro:property name="fork_camera_x" value="1.525" />
   <xacro:property name="fork_camera_y" value="0.195" />
-  <xacro:property name="fork_camera_z" value="0.067" />
+  <xacro:property name="fork_camera_z" value="0.0825" />
    <!-- FRONT LASER -->
- <xacro:property name="front_laser_x" value="0.25294" />
+ <xacro:property name="front_laser_x" value="-0.2529" />
  <xacro:property name="front_laser_y" value="0.000" />
  <xacro:property name="front_laser_z" value="0.200" />
@@ -42,16 +44,22 @@
 			<origin xyz="${wheel_offset_x} ${wheel_offset_y} ${wheel_offset_z}" rpy="0 0 0"/>
 	</xacro:motor_wheel>
-    <xacro:elevator prefix="${prefix}" parent="${prefix}base_link" hq="${hq}"> <!-- ELEVATOR -->
-        <origin xyz="0 0 0" rpy="0 0 0"/>
-    </xacro:elevator>
-    <xacro:sensor_sick_s300 prefix="${prefix}front_laser" parent="${prefix}base_footprint"> <!-- FRONT LIDAR -->
-        <origin xyz="${front_laser_x} ${front_laser_y} ${front_laser_z}" rpy="${PI} 0 0"/>
-    </xacro:sensor_sick_s300>
-    <xacro:sensor_r430 prefix="${prefix}right_fork" parent="${prefix}elevator_link" prefix_topic="right_fork_rgbd_camera">
-        <origin xyz="${fork_camera_x} ${fork_camera_y} ${fork_camera_z}" rpy="0 0 ${PI}"/>
-    </xacro:sensor_r430>
-    <xacro:sensor_r430 prefix="${prefix}left_fork" parent="${prefix}elevator_link" prefix_topic="left_fork_rgbd_camera">
-        <origin xyz="${fork_camera_x} -${fork_camera_y} ${fork_camera_z}" rpy="0 0 ${PI}"/>
-    </xacro:sensor_r430>
+  <!--xacro:additional_wheel prefix="${prefix}front_left" parent="${prefix}base_link" hq="${hq}">
+			<origin xyz="1 1 1" rpy="0 0 0"/>
+	</xacro:additional_wheel-->
+  <!--xacro:additional_wheel prefix="${prefix}front_right" parent="${prefix}base_link" hq="${hq}">
+      <origin xyz="1 -1 1" rpy="0 0 0"/>
+  </xacro:additional_wheel-->
+  <xacro:elevator prefix="${prefix}" parent="${prefix}base_link" hq="${hq}"> <!-- ELEVATOR -->
+      <origin xyz="0 0 0" rpy="0 0 0"/>
+  </xacro:elevator>
+  <!--xacro:sensor_sick_s300 prefix="${prefix}front_laser" parent="${prefix}base_footprint"> <!- - FRONT LIDAR - ->
+      <origin xyz="${front_laser_x} ${front_laser_y} ${front_laser_z}" rpy="${PI} 0 ${PI}"/>
+  </xacro:sensor_sick_s300>
+  <xacro:sensor_r430 prefix="${prefix}right_fork" parent="${prefix}elevator_link" prefix_topic="right_fork_rgbd_camera">
+      <origin xyz="${fork_camera_x} ${fork_camera_y} ${fork_camera_z}" rpy="0 0 ${PI}"/>
+  </xacro:sensor_r430>
+  <xacro:sensor_r430 prefix="${prefix}left_fork" parent="${prefix}elevator_link" prefix_topic="left_fork_rgbd_camera">
+      <origin xyz="${fork_camera_x} -${fork_camera_y} ${fork_camera_z}" rpy="0 0 ${PI}"/>
+  </xacro:sensor_r430-->
 	<!-- Gazebo ros control pluggins -->
 	<xacro:ros_control/>

File: pallet_truck_common/pallet_truck_description/urdf/bases/pallet_truck.urdf.xacro (robot description, xacro)
@@ -4,7 +4,7 @@
   <xacro:macro name="pallet_truck" params="prefix publish_bf hq">
   <!-- Robot mechanical and motor parameters -->
-  <xacro:property name="base_length" value="0.679" />
-  <xacro:property name="base_width" value="0.754" />
-  <xacro:property name="base_height" value="0.2" />
+  <xacro:property name="base_length" value="0.35" />
+  <xacro:property name="base_width" value="0.5" />
+  <xacro:property name="base_height" value="0.35" />
   <xacro:property name="base_mass" value="1"/>
   <xacro:property name="base_link_origin" value="0 0 0.46" />
@@ -13,5 +13,5 @@
   </link>
   <joint name="${prefix}base_footprint_joint" type="fixed">
-    <origin xyz="0 0 0" rpy="0 0 0" />
+    <origin xyz="${base_link_origin}" rpy="0 0 0" />
     <parent link="${prefix}base_footprint"/>
     <child link="${prefix}base_link" />
@@ -21,15 +21,22 @@
     <inertial>
       <mass value="${base_mass}" />
-      <origin xyz="${base_link_origin}" /><!-- Base_link's inertia origin ->  base_footprint -->
+      <origin xyz="0 0 -0.23" /><!-- Base_link's inertia origin ->  base_footprint -->
       <!-- yes, axis in solid_cuboid_inertia are changed, w relates to X axis, d to Z axis, and h to Y axis -->
       <!-- Keep this comment -->
-      <solid_cuboid_inertia  m="${base_mass}" d="${base_height}" w="${base_length}" h="${base_width}"/>
+      <solid_cuboid_inertia  m="${base_mass}" d="${base_length}" w="${base_length}" h="${base_length}"/>
+      <!--inertia ixx="0.0031" ixy="0" ixz="0" iyy="0.00204" iyz="0" izz="0.0031"/-->
     </inertial>
     <visual>
-      <origin xyz="${base_link_origin}" rpy="0 0 0" />
+      <origin xyz="0 0 0" rpy="0 0 0" />
       <geometry>
-        <mesh filename="package://pallet_truck_description/meshes/wheels/pallet_truck_steer.stl" scale="-1 1 1"/>
+        <mesh filename="package://pallet_truck_description/meshes/bases/base.stl"/>
       </geometry>
     </visual>
+    <collision>
+      <origin xyz="0 0 0" rpy="0 0 0" />
+      <geometry>
+        <mesh filename="package://pallet_truck_description/meshes/bases/base.stl"/>
+      </geometry>
+    </collision>
   </link>
   </xacro:macro>

File: pallet_truck_common/pallet_truck_description/urdf/elevator/elevator.urdf.xacro (robot description, xacro)
@@ -2,46 +2,83 @@
 <robot xmlns:xacro="http://www.ros.org/wiki/xacro">
   <xacro:include filename="$(find pallet_truck_description)/urdf/wheels/omni_wheel.urdf.xacro" />
+  <xacro:property name="PI" value="3.1415926535897931"/>
   <!-- Fork measurements -->
   <xacro:property name="fork_length" value="1.176" />
 	<xacro:property name="fork_width" value="0.11" />
 	<xacro:property name="fork_height" value="0.015" />
-	<xacro:property name="fork_mass" value="2.0" />
+	<xacro:property name="fork_mass" value="20" />
   <!-- Fork positions -->
   <xacro:property name="fork_x" value="0.0" />
   <xacro:property name="fork_y" value="0.195" />
   <xacro:property name="fork_z" value="0.0" />
-  <!-- Support wheel position -->
-  <xacro:property name="support_wheel_origin" value="-1.3175 0.0 ${wheel_radius/4.0-0.005}" />
+  <!-- Support wheel -->
+  <xacro:property name="support_wheel_mass" value="1" />
+  <xacro:property name="support_wheel_length" value="0.07" />
+  <xacro:property name="support_wheel_radius" value="0.04" />
   <!-- Limit elevator -->
   <xacro:property name="upper_limit_elevator" value="0.07" />
-  <!-- Platform is divided into two parts: TOP PLATFORM with a prismatic
-   joint, BELOW PLATFORM which has the two support wheels.-->
-  <!-- ************** -->
-  <!-- BELOW PLATFORM -->
-  <!-- ************** -->
-  <xacro:macro name="elevator_platform" params="prefix parent hq *origin">
-  	<joint name="${prefix}foot_elevator_joint" type="fixed">
+  <!-- *************** -->
+  <!--  SUPPORT WHEEL  -->
+  <!-- *************** -->
+  <xacro:macro name="support_wheel" params="prefix parent hq *origin">
+  	<joint name="${prefix}wheel_joint" type="continuous">
   			<xacro:insert_block name="origin" />
+        <axis xyz="0 1 0"/>
   			<parent link="${parent}"/>
-  			<child link="${prefix}foot_elevator_link" />
+  			<child link="${prefix}wheel_link" />
+        <limit effort="1.0" velocity="1"/>
   	</joint>
-  	<link name="${prefix}foot_elevator_link">
+  	<link name="${prefix}wheel_link">
+      <inertial>
+        <mass value="${support_wheel_mass}" />
+        <origin xyz="0 0 0" rpy="${PI/2.0} 0 0"/>
+        <cylinder_inertia  m="${support_wheel_mass}" r="${support_wheel_radius}" h="${support_wheel_length}" />
+      </inertial>
+      <visual>
+        <origin xyz="0 0 0" rpy="${PI/2.0} 0 0" />
+        <geometry>
+           <cylinder radius="${support_wheel_radius}" length="${support_wheel_length}" />
+        </geometry>
+        <material name="darkgrey">
+          <color rgba="0.1 0.1 0.1 1.0"/>
+        </material>
+      </visual>
+      <collision>
+        <origin xyz="0 0 0" rpy="${PI/2.0} 0 0"/>
+        <geometry>
+          <cylinder radius="${support_wheel_radius}" length="${support_wheel_length}" />
+        </geometry>
+        <surface>
+          <friction>
+            <ode>
+              <mu>100000</mu>
+              <mu2>1000000</mu2>
+            </ode>
+          </friction>
+        </surface>
+      </collision>
   	</link>
-    <!-- Support wheel -->
-  	<xacro:omni_wheel prefix="${prefix}omni" parent="${prefix}foot_elevator_link" hq="${hq}">
-  			<origin xyz="${support_wheel_origin}" rpy="0 0 0"/>
-  	</xacro:omni_wheel>
+    <!-- ***************** -->
+    <!-- GAZEBO PROPERTIES -->
+    <!-- ***************** -->
+    <!-- TRACTION LINK -->
+    <gazebo reference="${prefix}wheel_link">
+      <mu1>3</mu1>
+      <mu2>2</mu2>
+      <material>Gazebo/Black</material>
+    </gazebo>
   </xacro:macro>
   <xacro:macro name="fork" params="prefix parent hq *origin">
-    <joint name="${prefix}forks_joint" type="fixed">
+    <joint name="${prefix}fork_joint" type="prismatic">
   	   <xacro:insert_block name="origin" />
        <parent link="${parent}"/>
        <child link="${prefix}fork_link" />
+       <limit effort="1000.0" lower="0.0" upper="0" velocity="1"/>
      </joint>
      <!-- This piece holds the forks that are going to be elevated -->
      <link name="${prefix}fork_link">
        <inertial>
-         <mass value="1" />
-         <origin xyz="0 0 0" />
+         <mass value="${fork_mass}" />
+         <origin xyz="${fork_length/2.0} 0.0 0.0" />
          <!-- yes, axis in solid_cuboid_inertia are changed, w relates to X axis, d to Z axis, and h to Y axis -->
          <!-- Keep this comment -->
@@ -88,5 +125,5 @@
     <link name="${prefix}elevator_base_link" >
       <inertial>
-        <mass value="1" />
+        <mass value="0.001" />
         <origin xyz="0 0 0" />
          <!-- yes, axis in solid_cuboid_inertia are changed, w relates to X axis, d to Z axis, and h to Y axis -->
@@ -96,4 +133,5 @@
     </link>
     <joint name="${prefix}elevator_joint" type="prismatic">
+        <origin xyz="0 0 0" rpy="0 0 0" />
         <parent link="${prefix}elevator_base_link"/>
         <child link="${prefix}elevator_link" />
@@ -104,7 +142,6 @@
     <link name="${prefix}elevator_link">
       <visual>
-        <origin xyz="0 0 0.410" rpy="0 0 0" />
         <geometry>
-          <mesh filename="package://pallet_truck_description/meshes/bases/base.stl" scale="-1 1 1"/>
+          <mesh filename="package://pallet_truck_description/meshes/bases/cover.stl"/>
         </geometry>
         <material name="darkgrey">
@@ -113,30 +150,28 @@
       </visual>
       <inertial>
-        <mass value="1" />
-        <origin xyz="-0.8 0 0" />
+        <mass value="20" />
          <!-- yes, axis in solid_cuboid_inertia are changed, w relates to X axis, d to Z axis, and h to Y axis -->
          <!-- Keep this comment -->
-         <solid_cuboid_inertia m="0.001" h="0.1" d="0.03" w="1.67"/>
+         <solid_cuboid_inertia m="20" w="0.6" h="0.6" d="0.6"/>
       </inertial>
       <collision>
-        <origin xyz="0 0 0.410" rpy="0 0 0" />
         <geometry>
-          <mesh filename="package://pallet_truck_description/meshes/bases/base.stl" scale="-1 1 1"/>
+          <mesh filename="package://pallet_truck_description/meshes/bases/cover.stl"/>
         </geometry>
       </collision>
     </link>
     <xacro:fork prefix="${prefix}left_" parent="${prefix}elevator_link" hq="${hq}">
-       <origin xyz="-0.363 -0.195 0.080" rpy="0 0 3.1415" />
+       <origin xyz="0.349 -0.195 -0.3725" rpy="0 0 0" />
     </xacro:fork>
     <xacro:fork prefix="${prefix}right_" parent="${prefix}elevator_link" hq="${hq}">
-       <origin xyz="-0.363 0.195 0.080" rpy="0 0 3.1415" />
+       <origin xyz="0.349 0.195 -0.3725" rpy="0 0 0" />
     </xacro:fork>
-    <!-- Called two lower forks -->
-    <xacro:elevator_platform prefix="${prefix}left_" parent="${prefix}base_footprint" hq="${hq}">
-        <origin xyz="${fork_x} ${fork_y} ${fork_z}" rpy="0 0 0"/>
-    </xacro:elevator_platform>
-    <xacro:elevator_platform prefix="${prefix}right_" parent="${prefix}base_footprint" hq="${hq}">
-        <origin xyz="${fork_x} -${fork_y} ${fork_z}" rpy="0 0 0"/>
-    </xacro:elevator_platform>
+    <!-- Called two support wheels -->
+    <xacro:support_wheel prefix="${prefix}left_" parent="${prefix}base_footprint" hq="${hq}">
+        <origin xyz="1.3725 0.195 0.04" rpy="0 0 0"/>
+    </xacro:support_wheel>
+    <xacro:support_wheel prefix="${prefix}right_" parent="${prefix}base_footprint" hq="${hq}">
+        <origin xyz="1.3725 -0.195 0.04" rpy="0 0 0"/>
+    </xacro:support_wheel>
     <!-- ************* -->
     <!-- TRANSMISSIONS -->

File: pallet_truck_common/pallet_truck_description/urdf/epal_pallet/epal_pallet.urdf.xacro (robot description, xacro)
@@ -17,5 +17,5 @@
       <!-- yes, axis in solid_cuboid_inertia are changed, w relates to X axis, d to Z axis, and h to Y axis -->
       <!-- Keep this comment -->
-      <solid_cuboid_inertia m="5" h="0.8" d="0.044" w="1.2"/> <!-- h = z, d = y, w = x -->
+      <solid_cuboid_inertia m="5" h="0.044" d="0.8" w="1.2"/> <!-- h = z, d = y, w = x -->
     </inertial>
     <visual>

File: pallet_truck_common/pallet_truck_description/urdf/wheels/additional_wheel.urdf.xacro (robot description, xacro)
@@ -1,8 +1,8 @@
 <?xml version="1.0"?>
-<robot name="fixed_wheels" xmlns:xacro="http://www.ros.org/wiki/xacro">
+<robot name="additional_wheel" xmlns:xacro="http://www.ros.org/wiki/xacro">
   <xacro:property name="M_PI" value="3.1415926535897931" />
   <!-- Wheels -->
   <xacro:property name="support_wheel_radius" value="0.073" />
-  <xacro:property name="support_wheel_mass" value="0.01" />
+  <xacro:property name="support_wheel_mass" value="1" />
   <xacro:macro name="solid_sphere_inertia" params="m r">
     <inertia  ixx="${(2*r*r*m)/3}" ixy = "0" ixz = "0"
@@ -11,5 +11,5 @@
      />
   </xacro:macro>
-  <xacro:macro name="fixed_wheels" params="prefix parent *origin hq">
+  <xacro:macro name="additional_wheel" params="prefix parent *origin hq">
     <!--  -->
     <joint name="${prefix}wheel_joint" type="fixed">
@@ -22,5 +22,5 @@
         <mass value="${support_wheel_mass}" />
         <origin xyz="0 0 0" rpy="${PI/2.0} 0 0"/>
-        <sphere_inertia  m="${support_wheel_mass}" r="${support_wheel_radius}"/>
+        <solid_sphere_inertia  m="${support_wheel_mass}" r="${support_wheel_radius}"/>
       </inertial>
       <collision>

File: pallet_truck_common/pallet_truck_description/urdf/wheels/motor_wheel.urdf.xacro (robot description, xacro)
@@ -4,5 +4,5 @@
   <xacro:property name="wheel_radius" value="0.125" />
   <xacro:property name="wheel_width" value="0.1" />
-  <xacro:property name="wheel_mass" value="4.0" /><!-- in kg-->
+  <xacro:property name="wheel_mass" value="1.0" /><!-- in kg-->
   <!-- Steer wheel properties -->
   <xacro:property name="steer_joint_damping" value="1000" />

Commit message: Working on a slow move.
It works well but there's a small deviation in the movement that shouldn't appear

File: pallet_truck_common/pallet_truck_description/robots/pallet_truck_std.urdf.xacro (robot description, xacro)
@@ -45,8 +45,8 @@
 	</xacro:motor_wheel>
   <!--xacro:additional_wheel prefix="${prefix}front_left" parent="${prefix}base_link" hq="${hq}">
-			<origin xyz="1 1 1" rpy="0 0 0"/>
-	</xacro:additional_wheel-->
-  <!--xacro:additional_wheel prefix="${prefix}front_right" parent="${prefix}base_link" hq="${hq}">
-      <origin xyz="1 -1 1" rpy="0 0 0"/>
+			<origin xyz="-0.3 0.3 -0.4235" rpy="0 0 0"/>
+	</xacro:additional_wheel>
+  <xacro:additional_wheel prefix="${prefix}front_right" parent="${prefix}base_link" hq="${hq}">
+      <origin xyz="-0.3 -0.3 -0.4235" rpy="0 0 0"/>
   </xacro:additional_wheel-->
   <xacro:elevator prefix="${prefix}" parent="${prefix}base_link" hq="${hq}"> <!-- ELEVATOR -->

File: pallet_truck_common/pallet_truck_description/urdf/bases/pallet_truck.urdf.xacro (robot description, xacro)
@@ -7,8 +7,12 @@
   <xacro:property name="base_width" value="0.5" />
   <xacro:property name="base_height" value="0.35" />
-  <xacro:property name="base_mass" value="1"/>
+  <xacro:property name="base_mass" value="20"/>
   <xacro:property name="base_link_origin" value="0 0 0.46" />
   <!-- BASE FOOTPRINT -->
   <link name="${prefix}base_footprint">
+    <inertial>
+      <mass value="0.0001"/>
+      <inertia ixx="0.4" ixy="0.0" ixz="0.0" iyy="0.4" iyz="0.0" izz="0.2"/>
+    </inertial>
   </link>
   <joint name="${prefix}base_footprint_joint" type="fixed">

File: pallet_truck_common/pallet_truck_description/urdf/elevator/elevator.urdf.xacro (robot description, xacro)
@@ -68,4 +68,17 @@
       <material>Gazebo/Black</material>
     </gazebo>
+    <!-- ************* -->
+    <!-- TRANSMISSIONS -->
+    <!-- ************* -->
+     <transmission name="${prefix}wheel_joint_transmission">
+       <type>transmission_interface/SimpleTransmission</type>
+       <joint name="${prefix}wheel_joint">
+         <hardwareInterface>hardware_interface/VelocityJointInterface</hardwareInterface>
+       </joint>
+       <actuator name="${prefix}wheel_joint_motor">
+         <hardwareInterface>hardware_interface/VelocityActuatorInterface</hardwareInterface>
+         <mechanicalReduction>${traction_mechanical_reduction}</mechanicalReduction>
+       </actuator>
+     </transmission>
   </xacro:macro>
   <xacro:macro name="fork" params="prefix parent hq *origin">

File: pallet_truck_common/pallet_truck_description/urdf/wheels/additional_wheel.urdf.xacro (robot description, xacro)
@@ -5,4 +5,5 @@
   <xacro:property name="support_wheel_radius" value="0.073" />
   <xacro:property name="support_wheel_mass" value="1" />
+  <xacro:property name="wheel_mechanical_reduction" value="1" />
   <xacro:macro name="solid_sphere_inertia" params="m r">
     <inertia  ixx="${(2*r*r*m)/3}" ixy = "0" ixz = "0"
@@ -43,4 +44,17 @@
 		<turnGravityOff>false</turnGravityOff>
     </gazebo>
+    <!-- ***************** -->
+    <!--    TRANSMISSONS   -->
+    <!-- ***************** -->
+    <transmission name="${prefix}wheel_trans">
+      <type>transmission_interface/SimpleTransmission</type>
+      <joint name="${prefix}wheel_joint">
+        <hardwareInterface>hardware_interface/VelocityJointInterface</hardwareInterface>
+      </joint>
+      <actuator name="${prefix}wheel_joint_motor">
+        <hardwareInterface>hardware_interface/VelocityActuatorInterface</hardwareInterface>
+        <mechanicalReduction>${wheel_mechanical_reduction}</mechanicalReduction>
+      </actuator>
+    </transmission>
   </xacro:macro>
 </robot>

File: pallet_truck_common/pallet_truck_description/urdf/wheels/motor_wheel.urdf.xacro (robot description, xacro)
@@ -70,6 +70,8 @@
       <collision>
         <origin xyz="0 0 -0.125" rpy="0 0 0" />
+        <!--origin xyz="0 0 0" rpy="${PI/2.0} 0 0" /-->
         <geometry>
           <mesh filename="package://pallet_truck_description/meshes/wheels/pallet_truck_wheel.stl" scale="1 -0.9 1"/>
+          <!--cylinder length="${wheel_width}" radius="${0.125}"/-->
         </geometry>
       </collision>
