Commit message: Changed inertias

File: pallet_truck_common/pallet_truck_description/robots/pallet_truck_std.urdf.xacro (robot description, xacro)
@@ -11,4 +11,5 @@
   <!-- Import HR-RECYCLER additional wheels -->
   <xacro:include filename="$(find pallet_truck_description)/urdf/wheels/additional_wheel.urdf.xacro" />
+  <xacro:include filename="$(find pallet_truck_description)/urdf/wheels/omni_wheel.urdf.xacro" />
   <!-- Import HR-RECYCLER elevator -->
   <xacro:include filename="$(find pallet_truck_description)/urdf/elevator/elevator.urdf.xacro" />
@@ -27,7 +28,7 @@
 	<xacro:property name="hq" value="true" />
 	<!--  FORK CAMERAS  -->
-  <xacro:property name="fork_camera_x" value="1.525" />
+  <xacro:property name="fork_camera_x" value="1.54" />
   <xacro:property name="fork_camera_y" value="0.195" />
-  <xacro:property name="fork_camera_z" value="0.0825" />
+  <xacro:property name="fork_camera_z" value="0.375" />
    <!-- FRONT LASER -->
  <xacro:property name="front_laser_x" value="-0.2529" />
@@ -44,22 +45,28 @@
 			<origin xyz="${wheel_offset_x} ${wheel_offset_y} ${wheel_offset_z}" rpy="0 0 0"/>
 	</xacro:motor_wheel>
+  <xacro:additional_wheel1 prefix="${prefix}front_left" parent="${prefix}base_link" hq="${hq}">
+      <origin xyz="-0.2 0.2 -0.4235" rpy="0 0 0"/>
+  </xacro:additional_wheel1>
+  <xacro:additional_wheel1 prefix="${prefix}front_right" parent="${prefix}base_link" hq="${hq}">
+      <origin xyz="-0.2 -0.2 -0.4235" rpy="0 0 0"/>
+  </xacro:additional_wheel1>
   <!--xacro:additional_wheel prefix="${prefix}front_left" parent="${prefix}base_link" hq="${hq}">
-			<origin xyz="-0.3 0.3 -0.4235" rpy="0 0 0"/>
+			<origin xyz="-0.2 0.2 -0.4235" rpy="0 0 0"/>
 	</xacro:additional_wheel>
   <xacro:additional_wheel prefix="${prefix}front_right" parent="${prefix}base_link" hq="${hq}">
-      <origin xyz="-0.3 -0.3 -0.4235" rpy="0 0 0"/>
+      <origin xyz="-0.2 -0.2 -0.4235" rpy="0 0 0"/>
   </xacro:additional_wheel-->
   <xacro:elevator prefix="${prefix}" parent="${prefix}base_link" hq="${hq}"> <!-- ELEVATOR -->
       <origin xyz="0 0 0" rpy="0 0 0"/>
   </xacro:elevator>
-  <!--xacro:sensor_sick_s300 prefix="${prefix}front_laser" parent="${prefix}base_footprint"> <!- - FRONT LIDAR - ->
+  <xacro:sensor_sick_s300 prefix="${prefix}front_laser" parent="${prefix}base_footprint"> <!-- FRONT LIDAR -->
       <origin xyz="${front_laser_x} ${front_laser_y} ${front_laser_z}" rpy="${PI} 0 ${PI}"/>
   </xacro:sensor_sick_s300>
   <xacro:sensor_r430 prefix="${prefix}right_fork" parent="${prefix}elevator_link" prefix_topic="right_fork_rgbd_camera">
-      <origin xyz="${fork_camera_x} ${fork_camera_y} ${fork_camera_z}" rpy="0 0 ${PI}"/>
+      <origin xyz="${fork_camera_x} ${fork_camera_y} -${fork_camera_z}" rpy="0 0 0"/>
   </xacro:sensor_r430>
   <xacro:sensor_r430 prefix="${prefix}left_fork" parent="${prefix}elevator_link" prefix_topic="left_fork_rgbd_camera">
-      <origin xyz="${fork_camera_x} -${fork_camera_y} ${fork_camera_z}" rpy="0 0 ${PI}"/>
-  </xacro:sensor_r430-->
+      <origin xyz="${fork_camera_x} -${fork_camera_y} -${fork_camera_z}" rpy="0 0 0"/>
+  </xacro:sensor_r430>
 	<!-- Gazebo ros control pluggins -->
 	<xacro:ros_control/>

File: pallet_truck_common/pallet_truck_description/urdf/elevator/elevator.urdf.xacro (robot description, xacro)
@@ -49,12 +49,4 @@
           <cylinder radius="${support_wheel_radius}" length="${support_wheel_length}" />
         </geometry>
-        <surface>
-          <friction>
-            <ode>
-              <mu>100000</mu>
-              <mu2>1000000</mu2>
-            </ode>
-          </friction>
-        </surface>
       </collision>
   	</link>
@@ -116,14 +108,15 @@
             <box size="${fork_length} ${fork_width} ${fork_height}" />
          </geometry>
-         <surface>
-           <friction>
-             <ode>
-               <mu>100000</mu>
-               <mu2>50000</mu2>
-             </ode>
-           </friction>
-         </surface>
        </collision>
      </link>
+     <!-- ***************** -->
+     <!-- GAZEBO PROPERTIES -->
+     <!-- ***************** -->
+     <!-- FORK LINK -->
+     <gazebo reference="${prefix}fork_link">
+       <mu1>100000</mu1>
+       <mu2>100000</mu2>
+       <material>Gazebo/Black</material>
+     </gazebo>
   </xacro:macro>
   <!-- ************** -->

File: pallet_truck_common/pallet_truck_description/urdf/wheels/additional_wheel.urdf.xacro (robot description, xacro)
@@ -14,10 +14,10 @@
   <xacro:macro name="additional_wheel" params="prefix parent *origin hq">
     <!--  -->
-    <joint name="${prefix}wheel_joint" type="fixed">
+    <joint name="${prefix}_wheel_joint" type="fixed">
   			<xacro:insert_block name="origin" />
   			<parent link="${parent}"/>
-  			<child link="${prefix}wheel_base_link" />
+  			<child link="${prefix}_wheel_base_link" />
   	</joint>
-  	<link name="${prefix}wheel_base_link">
+  	<link name="${prefix}_wheel_base_link">
       <inertial>
         <mass value="${support_wheel_mass}" />
@@ -35,5 +35,5 @@
     <!-- GAZEBO PROPERTIES -->
     <!-- ***************** -->
-    <gazebo reference="${prefix}wheel_base_link">
+    <gazebo reference="${prefix}_wheel_base_link">
 		<mu1 value="0"/>
 		<mu2 value="0"/>
@@ -47,10 +47,10 @@
     <!--    TRANSMISSONS   -->
     <!-- ***************** -->
-    <transmission name="${prefix}wheel_trans">
+    <transmission name="${prefix}_wheel_trans">
       <type>transmission_interface/SimpleTransmission</type>
-      <joint name="${prefix}wheel_joint">
+      <joint name="${prefix}_wheel_joint">
         <hardwareInterface>hardware_interface/VelocityJointInterface</hardwareInterface>
       </joint>
-      <actuator name="${prefix}wheel_joint_motor">
+      <actuator name="${prefix}_wheel_joint_motor">
         <hardwareInterface>hardware_interface/VelocityActuatorInterface</hardwareInterface>
         <mechanicalReduction>${wheel_mechanical_reduction}</mechanicalReduction>

File: pallet_truck_common/pallet_truck_description/urdf/wheels/omni_wheel.urdf.xacro (robot description, xacro)
@@ -1,38 +1,66 @@
 <?xml version="1.0"?>
-<robot name="fixed_wheels" xmlns:xacro="http://www.ros.org/wiki/xacro">
+<robot name="additional_wheel1" xmlns:xacro="http://www.ros.org/wiki/xacro">
   <xacro:property name="M_PI" value="3.1415926535897931" />
   <!-- Wheels -->
-  <xacro:property name="support_wheel_radius" value="0.073" />
-  <xacro:property name="support_wheel_mass" value="0.01" />
-  <xacro:macro name="solid_sphere_inertia" params="m r">
-    <inertia  ixx="${(2*r*r*m)/3}" ixy = "0" ixz = "0"
-              iyy="${(2*r*r*m)/3}" iyz = "0"
-              izz="${(2*r*r*m)/3}"
+  <xacro:property name="omni_wheel_radius" value="0.036" />
+  <xacro:property name="omni_wheel_height" value="0.070" />
+  <xacro:property name="omni_wheel_mass" value="0.01" />
+  <xacro:macro name="cylinder_inertia" params="m r h">
+    <inertia  ixx="${m*(3*r*r+h*h)/12}" ixy = "0" ixz = "0"
+              iyy="${m*(3*r*r+h*h)/12}" iyz = "0"
+              izz="${m*r*r/2}"
      />
   </xacro:macro>
-  <xacro:macro name="fixed_wheels" params="prefix parent *origin hq">
-    <!--  -->
-    <joint name="${prefix}wheel_joint" type="fixed">
-  			<xacro:insert_block name="origin" />
-  			<parent link="${parent}"/>
-  			<child link="${prefix}wheel_base_link" />
-  	</joint>
-  	<link name="${prefix}wheel_base_link">
+  <xacro:macro name="additional_wheel1" params="prefix parent *origin hq">
+    <!--WHEEL TIRE -->
+    <joint name="${prefix}_wheel_joint" type="fixed">
+      <parent link="${parent}"/>
+      <child link="${prefix}_wheel_link"/>
+      <xacro:insert_block name="origin" />
+      <axis xyz="0 1 0" rpy="0 0 0" />
+      <limit effort="100" velocity="100"/>
+      <joint_properties damping="0.0" friction="0.0"/>
+    </joint>
+    <link name="${prefix}_wheel_link">
+      <visual>
+        <!-- HIGH RESOLUTION WHEELS -->
+        <xacro:if value="${hq}">
+          <origin xyz="0 0 0" rpy="0 0 0" />
+          <geometry>
+				    <!--mesh filename="package://pallet_truck_description/meshes/wheels/pallet_truck_omni_wheel_fake.dae"/-->
+            <sphere radius="${omni_wheel_radius}"/>
+          </geometry>
+        </xacro:if>
+       <!-- LOW RESOLUTION WHEELS -->
+        <xacro:unless value="${hq}">
+          <origin xyz="0 0 0" rpy="${M_PI/2} 0 0" />
+          <geometry>
+            <!--cylinder length="${omni_wheel_height}" radius="${omni_wheel_radius}" /-->
+            <sphere radius="${omni_wheel_radius}"/>
+          </geometry>
+        </xacro:unless>
+      </visual>
+      <collision>
+        <origin xyz="0 0 0" rpy="${M_PI/2} 0 0" />
+        <geometry>
+          <sphere radius="${omni_wheel_radius}"/>
+        </geometry>
+        <surface>
+          <friction>
+            <ode>
+              <mu>0.0001</mu>
+              <mu2>0.0001</mu2>
+            </ode>
+          </friction>
+			  </surface>
+      </collision>
       <inertial>
-        <mass value="${support_wheel_mass}" />
-        <origin xyz="0 0 0" rpy="${PI/2.0} 0 0"/>
-        <sphere_inertia  m="${support_wheel_mass}" r="${support_wheel_radius}"/>
+        <mass value="${wheel_mass}" />
+        <origin xyz="0 0 0" />
+        <cylinder_inertia  m="${omni_wheel_mass}" r="${omni_wheel_radius}" h="${omni_wheel_height}" />
+        <!-- inertia  ixx="0.001" ixy="0.0"  ixz="0.0"  iyy="0.001"  iyz="0.0"  izz="0.001" / -->
       </inertial>
-      <collision>
-        <origin xyz="0 0 0" rpy="${PI/2.0} 0 0"/>
-        <geometry>
-          <sphere radius="${support_wheel_radius}"/>
-        </geometry>
-      </collision>
-  	</link>
-    <!-- ***************** -->
-    <!-- GAZEBO PROPERTIES -->
-    <!-- ***************** -->
-    <gazebo reference="${prefix}wheel_base_link">
+    </link>
+    <gazebo reference="${prefix}wheel">
 		<mu1 value="0"/>
 		<mu2 value="0"/>

Commit message: Added Central_link

File: pallet_truck_common/pallet_truck_description/robots/pallet_truck_std.urdf.xacro (robot description, xacro)
@@ -10,5 +10,4 @@
 	<xacro:include filename="$(find pallet_truck_description)/urdf/wheels/motor_wheel.urdf.xacro" />
   <!-- Import HR-RECYCLER additional wheels -->
-  <xacro:include filename="$(find pallet_truck_description)/urdf/wheels/additional_wheel.urdf.xacro" />
   <xacro:include filename="$(find pallet_truck_description)/urdf/wheels/omni_wheel.urdf.xacro" />
   <!-- Import HR-RECYCLER elevator -->
@@ -28,5 +27,5 @@
 	<xacro:property name="hq" value="true" />
 	<!--  FORK CAMERAS  -->
-  <xacro:property name="fork_camera_x" value="1.54" />
+  <xacro:property name="fork_camera_x" value="1.545" />
   <xacro:property name="fork_camera_y" value="0.195" />
   <xacro:property name="fork_camera_z" value="0.375" />
@@ -34,5 +33,5 @@
  <xacro:property name="front_laser_x" value="-0.2529" />
  <xacro:property name="front_laser_y" value="0.000" />
- <xacro:property name="front_laser_z" value="0.200" />
+ <xacro:property name="front_laser_z" value="-0.26" />
 	<!-- *************** -->
 	<!-- Robots Elements -->
@@ -42,11 +41,22 @@
   <xacro:property name="prefix" value="$(arg prefix)" />
 	<xacro:pallet_truck prefix="${prefix}" publish_bf="true" hq="${hq}" /> <!-- BASE -->
-	<xacro:motor_wheel prefix="${prefix}front_" parent="${prefix}base_link" hq="${hq}"> <!-- WHEEL -->
+  <joint name="${prefix}central_joint" type="fixed">
+    <origin xyz="0 0 0" rpy="0 0 3.1415926535897931" />
+    <parent link="${prefix}base_link"/>
+    <child link="${prefix}central_link" />
+  </joint>
+  <link name="${prefix}central_link">
+    <inertial>
+      <mass value="0.0001"/>
+      <inertia ixx="0.4" ixy="0.0" ixz="0.0" iyy="0.4" iyz="0.0" izz="0.2"/>
+    </inertial>
+  </link>
+	<xacro:motor_wheel prefix="${prefix}front_" parent="${prefix}central_link" hq="${hq}"> <!-- WHEEL -->
 			<origin xyz="${wheel_offset_x} ${wheel_offset_y} ${wheel_offset_z}" rpy="0 0 0"/>
 	</xacro:motor_wheel>
-  <xacro:additional_wheel1 prefix="${prefix}front_left" parent="${prefix}base_link" hq="${hq}">
+  <xacro:additional_wheel1 prefix="${prefix}front_left" parent="${prefix}central_link" hq="${hq}">
       <origin xyz="-0.2 0.2 -0.4235" rpy="0 0 0"/>
   </xacro:additional_wheel1>
-  <xacro:additional_wheel1 prefix="${prefix}front_right" parent="${prefix}base_link" hq="${hq}">
+  <xacro:additional_wheel1 prefix="${prefix}front_right" parent="${prefix}central_link" hq="${hq}">
       <origin xyz="-0.2 -0.2 -0.4235" rpy="0 0 0"/>
   </xacro:additional_wheel1>
@@ -57,8 +67,8 @@
       <origin xyz="-0.2 -0.2 -0.4235" rpy="0 0 0"/>
   </xacro:additional_wheel-->
-  <xacro:elevator prefix="${prefix}" parent="${prefix}base_link" hq="${hq}"> <!-- ELEVATOR -->
+  <xacro:elevator prefix="${prefix}" parent="${prefix}central_link" hq="${hq}"> <!-- ELEVATOR -->
       <origin xyz="0 0 0" rpy="0 0 0"/>
   </xacro:elevator>
-  <xacro:sensor_sick_s300 prefix="${prefix}front_laser" parent="${prefix}base_footprint"> <!-- FRONT LIDAR -->
+  <xacro:sensor_sick_s300 prefix="${prefix}front_laser" parent="${prefix}central_link"> <!-- FRONT LIDAR -->
       <origin xyz="${front_laser_x} ${front_laser_y} ${front_laser_z}" rpy="${PI} 0 ${PI}"/>
   </xacro:sensor_sick_s300>
