Commit message: New pallet-truck version

File: pallet_truck_common/pallet_truck_description/robots/pallet_truck_std.urdf.xacro (robot description, xacro)
@@ -5,12 +5,16 @@
 	<!-- ***************** -->
 	<!-- First we import all posible elements defined in the urdf.xacro files. All these elements are defined as macro:xacros -->
-	<!-- Import HR-RECYCLER base elements -->
+	<!-- Import PALLET-TRUCK base elements -->
   <xacro:include filename="$(find pallet_truck_description)/urdf/bases/pallet_truck.urdf.xacro" />
-	<!-- Import HR-RECYCLER wheels -->
+	<!-- Import PALLET-TRUCK wheels -->
 	<xacro:include filename="$(find pallet_truck_description)/urdf/wheels/motor_wheel.urdf.xacro" />
-  <!-- Import HR-RECYCLER additional wheels -->
-  <xacro:include filename="$(find pallet_truck_description)/urdf/wheels/omni_wheel.urdf.xacro" />
-  <!-- Import HR-RECYCLER elevator -->
-  <xacro:include filename="$(find pallet_truck_description)/urdf/elevator/elevator.urdf.xacro" />
+  <!-- Import PALLET-TRUCK additional wheels -->
+  <xacro:include filename="$(find pallet_truck_description)/urdf/wheels/castor_wheel.urdf.xacro" />
+  <!-- Import PALLET-TRUCK additional wheels -->
+  <xacro:include filename="$(find pallet_truck_description)/urdf/wheels/fork_wheel.urdf.xacro" />
+  <!-- Import PALLET-TRUCK elevator -->
+  <xacro:include filename="$(find pallet_truck_description)/urdf/bases/front_case.urdf.xacro" />
+  <!-- Import PALLET-TRUCK battery_case -->
+  <xacro:include filename="$(find pallet_truck_description)/urdf/bases/battery_case.urdf.xacro" />
 	<!-- Import sensors -->
 	<xacro:include filename="$(find robotnik_sensors)/urdf/all_sensors.urdf.xacro" />
@@ -21,17 +25,35 @@
 	<!-- Wheel parameters -->
   <!-- x,y,z in translation from base_link to the center of the wheel -->
-	<xacro:property name="wheel_offset_x" value="0.0"/>
+	<xacro:property name="wheel_offset_x" value="0.077"/>
 	<xacro:property name="wheel_offset_y" value="0.0"/>
-	<xacro:property name="wheel_offset_z" value="0.0"/>
-	<!-- Flag to select the high or low quality model -->
-	<xacro:property name="hq" value="true" />
+	<xacro:property name="wheel_offset_z" value="-0.59"/>
+  <!-- Fork wheel -->
+  <xacro:property name="fork_wheel_offset_x" value="0.0"/>
+  <xacro:property name="fork_wheel_offset_y" value="0.201"/>
+  <xacro:property name="fork_wheel_offset_z" value="0.0"/>
+  <!-- Battery_case -->
+  <xacro:property name="battery_case_offset_x" value="1.2975"/>
+  <xacro:property name="battery_case_offset_y" value="0.0"/>
+  <xacro:property name="battery_case_offset_z" value="0.674"/>
+  <!-- Front_case -->
+  <xacro:property name="front_case_offset_x" value="1.2982"/>
+  <xacro:property name="front_case_offset_y" value="0.0"/>
+  <xacro:property name="front_case_offset_z" value="0.671"/>
+  <!-- Front support wheel -->
+  <xacro:property name="front_support_wheel_offset_x" value="0.340"/>
+  <xacro:property name="front_support_wheel_offset_y" value="0.180"/>
+  <xacro:property name="front_support_wheel_offset_z" value="-0.6685"/>
 	<!--  FORK CAMERAS  -->
   <xacro:property name="fork_camera_x" value="1.545" />
   <xacro:property name="fork_camera_y" value="0.195" />
   <xacro:property name="fork_camera_z" value="0.375" />
-   <!-- FRONT LASER -->
- <xacro:property name="front_laser_x" value="-0.2529" />
- <xacro:property name="front_laser_y" value="0.000" />
- <xacro:property name="front_laser_z" value="-0.26" />
+  <!-- FRONT LASER -->
+  <xacro:property name="front_laser_x" value="0.391" />
+  <xacro:property name="front_laser_y" value="0.0" />
+  <xacro:property name="front_laser_z" value="-0.38735" />
+  <!-- RS_lIDAR -->
+  <xacro:property name="lidar_offset_x" value="0.085" />
+  <xacro:property name="lidar_offset_y" value="0.0" />
+  <xacro:property name="lidar_offset_z" value="0.205" />
 	<!-- *************** -->
 	<!-- Robots Elements -->
@@ -40,43 +62,32 @@
 	<xacro:arg name="prefix" default="pallet_truck_"/>
   <xacro:property name="prefix" value="$(arg prefix)" />
-	<xacro:pallet_truck prefix="${prefix}" publish_bf="true" hq="${hq}" /> <!-- BASE -->
-  <joint name="${prefix}central_joint" type="fixed">
-    <origin xyz="0 0 0" rpy="0 0 3.1415926535897931" />
-    <parent link="${prefix}base_link"/>
-    <child link="${prefix}central_link" />
-  </joint>
-  <link name="${prefix}central_link">
-    <inertial>
-      <mass value="0.0001"/>
-      <inertia ixx="0.4" ixy="0.0" ixz="0.0" iyy="0.4" iyz="0.0" izz="0.2"/>
-    </inertial>
-  </link>
-	<xacro:motor_wheel prefix="${prefix}front_" parent="${prefix}central_link" hq="${hq}"> <!-- WHEEL -->
+	<xacro:pallet_truck prefix="${prefix}" publish_bf="true"/> <!-- BASE -->
+	<xacro:motor_wheel prefix="${prefix}" parent="${prefix}front_case_link">
 			<origin xyz="${wheel_offset_x} ${wheel_offset_y} ${wheel_offset_z}" rpy="0 0 0"/>
 	</xacro:motor_wheel>
-  <xacro:additional_wheel1 prefix="${prefix}front_left" parent="${prefix}central_link" hq="${hq}">
-      <origin xyz="-0.2 0.2 -0.4235" rpy="0 0 0"/>
-  </xacro:additional_wheel1>
-  <xacro:additional_wheel1 prefix="${prefix}front_right" parent="${prefix}central_link" hq="${hq}">
-      <origin xyz="-0.2 -0.2 -0.4235" rpy="0 0 0"/>
-  </xacro:additional_wheel1>
-  <!--xacro:additional_wheel prefix="${prefix}front_left" parent="${prefix}base_link" hq="${hq}">
-			<origin xyz="-0.2 0.2 -0.4235" rpy="0 0 0"/>
-	</xacro:additional_wheel>
-  <xacro:additional_wheel prefix="${prefix}front_right" parent="${prefix}base_link" hq="${hq}">
-      <origin xyz="-0.2 -0.2 -0.4235" rpy="0 0 0"/>
-  </xacro:additional_wheel-->
-  <xacro:elevator prefix="${prefix}" parent="${prefix}central_link" hq="${hq}"> <!-- ELEVATOR -->
-      <origin xyz="0 0 0" rpy="0 0 0"/>
-  </xacro:elevator>
-  <xacro:sensor_sick_s300 prefix="${prefix}front_laser" parent="${prefix}central_link"> <!-- FRONT LIDAR -->
-      <origin xyz="${front_laser_x} ${front_laser_y} ${front_laser_z}" rpy="${PI} 0 ${PI}"/>
+  <xacro:fork_wheel prefix="${prefix}left_fork_" parent="${prefix}base_link">
+      <origin xyz="${fork_wheel_offset_x} ${fork_wheel_offset_y} ${fork_wheel_offset_z}" rpy="0 0 0"/>
+  </xacro:fork_wheel>
+  <xacro:fork_wheel prefix="${prefix}right_fork_" parent="${prefix}base_link">
+      <origin xyz="${fork_wheel_offset_x} -${fork_wheel_offset_y} ${fork_wheel_offset_z}" rpy="0 0 0"/>
+  </xacro:fork_wheel>
+  <xacro:battery_case prefix="${prefix}" parent="${prefix}base_link">
+      <origin xyz="${battery_case_offset_x} -${battery_case_offset_y} ${battery_case_offset_z}" rpy="0 0 0"/>
+  </xacro:battery_case>
+  <xacro:front_case prefix="${prefix}" parent="${prefix}base_link">
+    <origin xyz="${front_case_offset_x} -${front_case_offset_y} ${front_case_offset_z}" rpy="0 0 0"/>
+	</xacro:front_case>
+  <xacro:support_wheel prefix="${prefix}front_left_" parent="${prefix}front_case_link">
+      <origin xyz="${front_support_wheel_offset_x} ${front_support_wheel_offset_x} ${front_support_wheel_offset_z}" rpy="0 0 0"/>
+  </xacro:support_wheel>
+  <xacro:support_wheel prefix="${prefix}front_right_" parent="${prefix}front_case_link">
+      <origin xyz="${front_support_wheel_offset_x} -${front_support_wheel_offset_x} ${front_support_wheel_offset_z}" rpy="0 0 0"/>
+  </xacro:support_wheel>
+  <xacro:sensor_rplidar prefix="${prefix}_rplidar" parent="${prefix}front_case_link">
+      <origin xyz="${lidar_offset_x} ${lidar_offset_y} ${lidar_offset_z}" rpy="0 0 0"/>
+  </xacro:sensor_rplidar>
+  <xacro:sensor_sick_s300 prefix="${prefix}_sick" parent="${prefix}front_case_link">
+      <origin xyz="${front_laser_x} ${front_laser_y} ${front_laser_z}" rpy="${PI} 0 0"/>
   </xacro:sensor_sick_s300>
-  <xacro:sensor_r430 prefix="${prefix}right_fork" parent="${prefix}elevator_link" prefix_topic="right_fork_rgbd_camera">
-      <origin xyz="${fork_camera_x} ${fork_camera_y} -${fork_camera_z}" rpy="0 0 0"/>
-  </xacro:sensor_r430>
-  <xacro:sensor_r430 prefix="${prefix}left_fork" parent="${prefix}elevator_link" prefix_topic="left_fork_rgbd_camera">
-      <origin xyz="${fork_camera_x} -${fork_camera_y} -${fork_camera_z}" rpy="0 0 0"/>
-  </xacro:sensor_r430>
 	<!-- Gazebo ros control pluggins -->
 	<xacro:ros_control/>

File: pallet_truck_common/pallet_truck_description/urdf/bases/pallet_truck.urdf.xacro (robot description, xacro)
@@ -2,17 +2,17 @@
 <robot name="pallet_truck" xmlns:xacro="http://www.ros.org/wiki/xacro">
   <xacro:include filename="$(find pallet_truck_description)/urdf/inertia.urdf.xacro" />
-  <xacro:macro name="pallet_truck" params="prefix publish_bf hq">
 	<xacro:property name="PI" value="3.1415926535897931"/>
   <!-- Robot mechanical and motor parameters -->
-  <xacro:property name="base_length" value="0.35" />
-  <xacro:property name="base_width" value="0.5" />
-  <xacro:property name="base_height" value="0.35" />
-  <xacro:property name="base_mass" value="20"/>
-  <xacro:property name="base_link_origin" value="0 0 0.46" />
+  <xacro:property name="base_length" value="0.0001" />
+  <xacro:property name="base_width" value="0.0001" />
+  <xacro:property name="base_height" value="0.0001" />
+  <xacro:property name="base_mass" value="0.0001"/>
+  <xacro:property name="base_link_origin" value="0 0 0.040" /> <!--base_link (0,0,fork_wheel_radius) RF-> Base_Footprint. Align with the centers of fork_wheels.-->
+  <xacro:macro name="pallet_truck" params="prefix publish_bf">
   <!-- BASE FOOTPRINT -->
   <link name="${prefix}base_footprint">
     <inertial>
       <mass value="0.0001"/>
-      <inertia ixx="0.4" ixy="0.0" ixz="0.0" iyy="0.4" iyz="0.0" izz="0.2"/>
+      <inertia ixx="0.0001" ixy="0" ixz="0" iyy="0.0001" iyz="0" izz="0.0001"/>
     </inertial>
   </link>
@@ -26,22 +26,7 @@
     <inertial>
       <mass value="${base_mass}" />
-      <origin xyz="0 0 -0.23" /><!-- Base_link's inertia origin ->  base_footprint -->
-      <!-- yes, axis in solid_cuboid_inertia are changed, w relates to X axis, d to Z axis, and h to Y axis -->
-      <!-- Keep this comment -->
+      <origin xyz="0 0 0" />
       <solid_cuboid_inertia  m="${base_mass}" d="${base_length}" w="${base_length}" h="${base_length}"/>
-      <!--inertia ixx="0.0031" ixy="0" ixz="0" iyy="0.00204" iyz="0" izz="0.0031"/-->
     </inertial>
-    <visual>
-      <origin xyz="0 0 0" rpy="0 0 ${M_PI}" />
-      <geometry>
-        <mesh filename="package://pallet_truck_description/meshes/bases/base.stl"/>
-      </geometry>
-    </visual>
-    <collision>
-      <origin xyz="0 0 0" rpy="0 0 ${M_PI}" />
-      <geometry>
-        <mesh filename="package://pallet_truck_description/meshes/bases/base.stl"/>
-      </geometry>
-    </collision>
   </link>
   </xacro:macro>

File: pallet_truck_common/pallet_truck_description/urdf/common.gazebo.xacro (robot description, xacro)
@@ -5,5 +5,4 @@
 	   <gazebo>
       <plugin name="ros_control" filename="libgazebo_ros_control.so">
-        <!--robotNamespace>/rb1</robotNamespace-->
         <robotParam>robot_description</robotParam>
         <controlPeriod>0.001</controlPeriod>

File: pallet_truck_common/pallet_truck_description/urdf/wheels/motor_wheel.urdf.xacro (robot description, xacro)
@@ -2,7 +2,7 @@
 <robot xmlns:xacro="http://www.ros.org/wiki/xacro">
   <!-- Wheels -->
-  <xacro:property name="wheel_radius" value="0.125" />
+  <xacro:property name="wheel_radius" value="0.122" />
   <xacro:property name="wheel_width" value="0.1" />
-  <xacro:property name="wheel_mass" value="1.0" /><!-- in kg-->
+  <xacro:property name="wheel_mass" value="1" /><!-- in kg-->
   <!-- Steer wheel properties -->
   <xacro:property name="steer_joint_damping" value="1000" />
@@ -18,6 +18,6 @@
   <xacro:property name="traction_joint_velocity_limit" value="100" />
   <xacro:property name="traction_mechanical_reduction" value="1.0" />
-  <xacro:property name="steer_origin" value="0 0 -0.210"/>
-  <xacro:property name="traction_origin" value="0 0 -0.335"/>
+  <xacro:property name="steer_origin" value="0 0 ${wheel_radius}"/>
+  <xacro:property name="front_wheel_origin" value="0 0 0"/>
   <!-- inertial equation -->
   <xacro:macro name="cylinder_inertia" params="m r h">
@@ -27,57 +27,51 @@
   <!-- MOTOR WHEEL -->
   <!-- *********** -->
-  <xacro:macro name="motor_wheel" params="prefix parent *origin hq">
+  <xacro:macro name="motor_wheel" params="prefix parent *origin">
     <!-- STEER -->
-    <joint name="${prefix}wheel_steer_joint" type="revolute">
+    <joint name="${prefix}steer_joint" type="revolute">
+      <xacro:insert_block name="origin" />
       <parent link="${parent}"/>
-      <child link="${prefix}wheel_steer_link"/>
-      <xacro:insert_block name="origin" />
+      <child link="${prefix}steer_link"/>
       <axis xyz="0 0 1" rpy="0 0 0" />
-      <limit effort="${steer_joint_effort_limit}" velocity="${steer_joint_velocity_limit}" lower="-${steer_joint_position_limit}" upper="${steer_joint_position_limit}"/>/>
+      <limit effort="${steer_joint_effort_limit}" velocity="${steer_joint_velocity_limit}" lower="-${steer_joint_position_limit}" upper="${steer_joint_position_limit}"/>
       <dynamics damping="${steer_joint_damping}" friction="${steer_joint_friction}"/>
     </joint>
-    <link name="${prefix}wheel_steer_link">
+    <link name="${prefix}steer_link">
       <inertial>
         <mass value="${wheel_mass}" />
-        <origin xyz="${steer_origin}"/>
+        <origin xyz="0 0 0"/>
         <cylinder_inertia m="${wheel_mass}" r="${wheel_width}" h="${wheel_radius}" />
       </inertial>
     </link>
     <!-- TRACTION -->
-    <joint name="${prefix}wheel_traction_joint" type="continuous">
-      <parent link="${prefix}wheel_steer_link"/>
-      <child link="${prefix}wheel_traction_link"/>
-      <origin xyz="${traction_origin}" rpy="0 0 0" />
-      <axis xyz="0 -1 0" rpy="0 0 0" />
+    <joint name="${prefix}traction_joint" type="continuous">
+      <parent link="${prefix}steer_link"/>
+      <child link="${prefix}front_wheel_link"/>
+      <origin xyz="0 0 0" rpy="0 0 0" />
+      <axis xyz="0 1 0" rpy="0 0 0" />
       <limit effort="${traction_joint_effort_limit}" velocity="${traction_joint_velocity_limit}" />
       <dynamics damping="${traction_joint_damping}" friction="${traction_joint_friction}"/>
     </joint>
-    <link name="${prefix}wheel_traction_link">
+    <link name="${prefix}front_wheel_link">
       <visual>
-        <xacro:if value="${hq}">
-          <origin xyz="0 0 -0.125" rpy="0 0 0" />
-          <geometry>
-            <mesh filename="package://pallet_truck_description/meshes/wheels/pallet_truck_wheel.stl" scale="1 -0.9 1"/>
-          </geometry>
-        </xacro:if>
-        <xacro:unless value="${hq}">
-          <origin xyz="0 0 -0.125" rpy="0 0 0" />
-          <geometry>
-            <mesh filename="package://pallet_truck_description/meshes/wheels/pallet_truck_wheel.stl" scale="1 -0.9 1"/>
-          </geometry>
-        </xacro:unless>
+        <!--origin xyz="0 0 0" rpy="${PI/2.0} 0 0" /-->
+        <origin xyz="0 0 0" rpy="0 0 0" />
+        <geometry>
+          <mesh filename="package://pallet_truck_description/meshes/wheels/pallet_truck_wheel.stl"/>
+          <!--cylinder length="${wheel_width}" radius="${0.12675}"/-->
+        </geometry>
       </visual>
       <collision>
-        <origin xyz="0 0 -0.125" rpy="0 0 0" />
-        <!--origin xyz="0 0 0" rpy="${PI/2.0} 0 0" /-->
+        <!--origin xyz="0 0 0" rpy="0 0 0" /-->
+        <origin xyz="0 0 0" rpy="${PI/2.0} 0 0" />
         <geometry>
-          <mesh filename="package://pallet_truck_description/meshes/wheels/pallet_truck_wheel.stl" scale="1 -0.9 1"/>
-          <!--cylinder length="${wheel_width}" radius="${0.125}"/-->
+          <!--mesh filename="package://pallet_truck_description/meshes/wheels/pallet_truck_wheel.stl"/-->
+          <cylinder length="${wheel_width}" radius="${0.125}"/>
         </geometry>
       </collision>
       <inertial>
         <mass value="${wheel_mass}" />
-        <origin xyz="0 0 0"/>
-        <cylinder_inertia m="${wheel_mass}" r="${wheel_radius}" h="${wheel_width}" />
+        <origin xyz="0.000063 0 0.000465"/>
+        <inertia ixx="0.0064" ixy="0.0" ixz="0.0" iyy="0.00496" iyz="0.0" izz="0.0064"/>  <!-- Multiplicar por la masa -->
       </inertial>
     </link>
@@ -86,7 +80,7 @@
     <!-- ***************** -->
     <!-- TRACTION LINK -->
-    <gazebo reference="${prefix}wheel_traction_link">
-      <mu1>3</mu1>
-      <mu2>2</mu2>
+    <gazebo reference="${prefix}front_wheel_link">
+      <mu1>1000</mu1>
+      <mu2>1000</mu2>
       <material>Gazebo/Black</material>
     </gazebo>
@@ -97,8 +91,8 @@
     <transmission name="${prefix}wheel_steer_trans">
       <type>transmission_interface/SimpleTransmission</type>
-      <joint name="${prefix}wheel_steer_joint">
+      <joint name="${prefix}steer_joint">
         <hardwareInterface>hardware_interface/PositionJointInterface</hardwareInterface>
       </joint>
-      <actuator name="${prefix}wheel_steer_motor">
+      <actuator name="${prefix}steer_motor">
         <hardwareInterface>hardware_interface/PositionActuatorInterface</hardwareInterface>
         <mechanicalReduction>${steer_mechanical_reduction}</mechanicalReduction>
@@ -106,10 +100,10 @@
     </transmission>
   <!-- TRACTION -->
-    <transmission name="${prefix}wheel_traction">
+    <transmission name="${prefix}_traction">
       <type>transmission_interface/SimpleTransmission</type>
-      <joint name="${prefix}wheel_traction_joint">
+      <joint name="${prefix}traction_joint">
         <hardwareInterface>hardware_interface/VelocityJointInterface</hardwareInterface>
       </joint>
-      <actuator name="${prefix}wheel_traction_motor">
+      <actuator name="${prefix}traction_motor">
         <hardwareInterface>hardware_interface/VelocityActuatorInterface</hardwareInterface>
         <mechanicalReduction>${traction_mechanical_reduction}</mechanicalReduction>

Commit message: Changed the distance between support wheel and floor

File: pallet_truck_common/pallet_truck_description/robots/pallet_truck_std.urdf.xacro (robot description, xacro)
@@ -43,5 +43,5 @@
   <xacro:property name="front_support_wheel_offset_x" value="0.340"/>
   <xacro:property name="front_support_wheel_offset_y" value="0.180"/>
-  <xacro:property name="front_support_wheel_offset_z" value="-0.6685"/>
+  <xacro:property name="front_support_wheel_offset_z" value="-0.675"/>
 	<!--  FORK CAMERAS  -->
   <xacro:property name="fork_camera_x" value="1.545" />

Commit message: Added registers

File: pallet_truck_common/pallet_truck_description/robots/pallet_truck_std.urdf.xacro (robot description, xacro)
@@ -56,4 +56,11 @@
   <xacro:property name="lidar_offset_y" value="0.0" />
   <xacro:property name="lidar_offset_z" value="0.205" />
+  <!-- REGISTERS -->
+  <xacro:property name="front_register_offset_x" value="0.452" />
+  <xacro:property name="front_register_offset_y" value="0.0" />
+  <xacro:property name="front_register_offset_z" value="-0.228" />
+  <xacro:property name="side_register_offset_x" value="0.1855" />
+  <xacro:property name="side_register_offset_y" value="0.276" />
+  <xacro:property name="side_register_offset_z" value="-0.228" />
 	<!-- *************** -->
 	<!-- Robots Elements -->
@@ -90,5 +97,30 @@
       <origin xyz="${front_laser_x} ${front_laser_y} ${front_laser_z}" rpy="${PI} 0 0"/>
   </xacro:sensor_sick_s300>
+  <!-- REGISTERS -->
+  <!-- Front -->
+  <joint name="${prefix}front_register_joint" type="fixed">
+     <origin xyz="${front_register_offset_x} ${front_register_offset_y} ${front_register_offset_z}" rpy="0 0 0"/>
+     <parent link="${prefix}front_case_link"/>
+     <child link="${prefix}front_register_link" />
+   </joint>
+   <link name="${prefix}front_register_link">
+   </link>
+   <!-- Right side -->
+   <joint name="${prefix}right_register_joint" type="fixed">
+     <origin xyz="${side_register_offset_x} -${side_register_offset_y} ${side_register_offset_z}" rpy="0 0 -${PI/2.0}"/>
+      <parent link="${prefix}front_case_link"/>
+      <child link="${prefix}right_register_link" />
+    </joint>
+    <link name="${prefix}right_register_link">
+    </link>
+   <!-- Left side -->
+   <joint name="${prefix}left_register_joint" type="fixed">
+      <origin xyz="${side_register_offset_x} ${side_register_offset_y} ${side_register_offset_z}" rpy="0 0 ${PI/2.0}"/>
+      <parent link="${prefix}front_case_link"/>
+      <child link="${prefix}left_register_link" />
+    </joint>
+    <link name="${prefix}left_register_link">
+    </link>
 	<!-- Gazebo ros control pluggins -->
-	<xacro:ros_control/>
+	<xacro:ros_control />
 </robot>

Commit message: added tricycle kinematics

File: pallet_truck_common/pallet_truck_description/robots/pallet_truck_std.urdf.xacro (robot description, xacro)
@@ -124,3 +124,21 @@
 	<!-- Gazebo ros control pluggins -->
 	<xacro:ros_control />
+	<xacro:sensor_imu_hector prefix="${prefix}imu" parent="${prefix}base_link">
+		<origin xyz="0.0 0.0 0.0" rpy="0 0 0"/>
+	</xacro:sensor_imu_hector>
+<gazebo>
+  <plugin name="ground_truth_controller" filename="librobotnik_gazebo_ground_truth_odom.so">
+    <alwaysOn>true</alwaysOn>
+    <updateRate>50.0</updateRate>
+    <bodyName>pallet_truck_base_link</bodyName> <!-- robot body to track, in gazebo -->
+    <frameName>pallet_truck_base_link_gt</frameName> <!-- frame name of robot body to be published in ros -->
+    <worldBodyName>world</worldBodyName> <!-- fixed body where body is tracked, in gazebo -->
+    <worldFrameName>pallet_truck_odom</worldFrameName> <!-- frame name of fixed body to be published in ros -->
+    <topicName>odom_gt</topicName>
+    <gaussianNoise>0.01</gaussianNoise>
+    <xyzOffsets>0 0 0</xyzOffsets>
+    <rpyOffsets>0 0 0</rpyOffsets>
+    <broadcastTF>True</broadcastTF>
+  </plugin>
+</gazebo>
 </robot>
