Commit message: Changed imu offset

File: pallet_truck_common/pallet_truck_description/robots/pallet_truck_std.urdf.xacro (robot description, xacro)
@@ -63,4 +63,8 @@
   <xacro:property name="side_register_offset_y" value="0.276" />
   <xacro:property name="side_register_offset_z" value="-0.228" />
+  <!-- IMU -->
+  <xacro:property name="imu_offset_x" value="1.2982" />
+  <xacro:property name="imu_offset_y" value="0.0" />
+  <xacro:property name="imu_offset_z" value="0.671" />
 	<!-- *************** -->
 	<!-- Robots Elements -->
@@ -125,20 +129,20 @@
 	<xacro:ros_control />
 	<xacro:sensor_imu_hector prefix="${prefix}imu" parent="${prefix}base_link">
-		<origin xyz="0.0 0.0 0.0" rpy="0 0 0"/>
+		<origin xyz="${imu_offset_x} -${imu_offset_y} ${imu_offset_z}" rpy="0 0 0"/>
 	</xacro:sensor_imu_hector>
-<gazebo>
-  <plugin name="ground_truth_controller" filename="librobotnik_gazebo_ground_truth_odom.so">
-    <alwaysOn>true</alwaysOn>
-    <updateRate>50.0</updateRate>
-    <bodyName>pallet_truck_base_link</bodyName> <!-- robot body to track, in gazebo -->
-    <frameName>pallet_truck_base_link_gt</frameName> <!-- frame name of robot body to be published in ros -->
-    <worldBodyName>world</worldBodyName> <!-- fixed body where body is tracked, in gazebo -->
-    <worldFrameName>pallet_truck_odom</worldFrameName> <!-- frame name of fixed body to be published in ros -->
-    <topicName>odom_gt</topicName>
-    <gaussianNoise>0.01</gaussianNoise>
-    <xyzOffsets>0 0 0</xyzOffsets>
-    <rpyOffsets>0 0 0</rpyOffsets>
-    <broadcastTF>True</broadcastTF>
-  </plugin>
-</gazebo>
+  <gazebo>
+    <plugin name="ground_truth_controller" filename="librobotnik_gazebo_ground_truth_odom.so">
+      <alwaysOn>true</alwaysOn>
+      <updateRate>50.0</updateRate>
+      <bodyName>pallet_truck_base_link</bodyName> <!-- robot body to track, in gazebo -->
+      <frameName>pallet_truck_base_link_gt</frameName> <!-- frame name of robot body to be published in ros -->
+      <worldBodyName>world</worldBodyName> <!-- fixed body where body is tracked, in gazebo -->
+      <worldFrameName>pallet_truck_odom</worldFrameName> <!-- frame name of fixed body to be published in ros -->
+      <topicName>odom_gt</topicName>
+      <gaussianNoise>0.01</gaussianNoise>
+      <xyzOffsets>0 0 0</xyzOffsets>
+      <rpyOffsets>0 0 0</rpyOffsets>
+      <broadcastTF>True</broadcastTF>
+    </plugin>
+  </gazebo>
 </robot>

Commit message: added rslidar and cleaned description

File: pallet_truck_common/pallet_truck_description/robots/pallet_truck_std.urdf.xacro (robot description, xacro)
@@ -1,12 +1,12 @@
 <?xml version="1.0"?>
 <robot name="pallet_truck" xmlns:xacro="http://www.ros.org/wiki/xacro">
-	<!-- ***************** -->
-	<!-- Imported elements -->
-	<!-- ***************** -->
-	<!-- First we import all posible elements defined in the urdf.xacro files. All these elements are defined as macro:xacros -->
-	<!-- Import PALLET-TRUCK base elements -->
+  <!-- ***************** -->
+  <!-- Imported elements -->
+  <!-- ***************** -->
+  <!-- First we import all posible elements defined in the urdf.xacro files. All these elements are defined as macro:xacros -->
+  <!-- Import PALLET-TRUCK base elements -->
   <xacro:include filename="$(find pallet_truck_description)/urdf/bases/pallet_truck.urdf.xacro" />
-	<!-- Import PALLET-TRUCK wheels -->
-	<xacro:include filename="$(find pallet_truck_description)/urdf/wheels/motor_wheel.urdf.xacro" />
+  <!-- Import PALLET-TRUCK wheels -->
+  <xacro:include filename="$(find pallet_truck_description)/urdf/wheels/motor_wheel.urdf.xacro" />
   <!-- Import PALLET-TRUCK additional wheels -->
   <xacro:include filename="$(find pallet_truck_description)/urdf/wheels/castor_wheel.urdf.xacro" />
@@ -17,15 +17,15 @@
   <!-- Import PALLET-TRUCK battery_case -->
   <xacro:include filename="$(find pallet_truck_description)/urdf/bases/battery_case.urdf.xacro" />
-	<!-- Import sensors -->
-	<xacro:include filename="$(find robotnik_sensors)/urdf/all_sensors.urdf.xacro" />
+  <!-- Import sensors -->
+  <xacro:include filename="$(find robotnik_sensors)/urdf/all_sensors.urdf.xacro" />
   <!-- Import Gazebo Stuff -->
   <xacro:include filename="$(find pallet_truck_description)/urdf/common.gazebo.xacro" />
-	<!-- Global parameters -->
-	<xacro:property name="PI" value="3.1415926535897931"/>
-	<!-- Wheel parameters -->
+  <!-- Global parameters -->
+  <xacro:property name="PI" value="3.1415926535897931"/>
+  <!-- Wheel parameters -->
   <!-- x,y,z in translation from base_link to the center of the wheel -->
-	<xacro:property name="wheel_offset_x" value="0.077"/>
-	<xacro:property name="wheel_offset_y" value="0.0"/>
-	<xacro:property name="wheel_offset_z" value="-0.59"/>
+  <xacro:property name="wheel_offset_x" value="0.077"/>
+  <xacro:property name="wheel_offset_y" value="0.0"/>
+  <xacro:property name="wheel_offset_z" value="-0.59"/>
   <!-- Fork wheel -->
   <xacro:property name="fork_wheel_offset_x" value="0.0"/>
@@ -44,5 +44,5 @@
   <xacro:property name="front_support_wheel_offset_y" value="0.180"/>
   <xacro:property name="front_support_wheel_offset_z" value="-0.675"/>
-	<!--  FORK CAMERAS  -->
+  <!--  FORK CAMERAS  -->
   <xacro:property name="fork_camera_x" value="1.545" />
   <xacro:property name="fork_camera_y" value="0.195" />
@@ -53,7 +53,7 @@
   <xacro:property name="front_laser_z" value="-0.38735" />
   <!-- RS_lIDAR -->
-  <xacro:property name="lidar_offset_x" value="0.085" />
-  <xacro:property name="lidar_offset_y" value="0.0" />
-  <xacro:property name="lidar_offset_z" value="0.205" />
+  <xacro:property name="top_lidar_offset_x" value="0.085" />
+  <xacro:property name="top_lidar_offset_y" value="0.0" />
+  <xacro:property name="top_lidar_offset_z" value="0.205" />
   <!-- REGISTERS -->
   <xacro:property name="front_register_offset_x" value="0.452" />
@@ -67,14 +67,14 @@
   <xacro:property name="imu_offset_y" value="0.0" />
   <xacro:property name="imu_offset_z" value="0.671" />
-	<!-- *************** -->
-	<!-- Robots Elements -->
-	<!-- *************** -->
-	<!-- Here we create the robot elements using the xacro:macros imported at the beggining of this file -->
-	<xacro:arg name="prefix" default="pallet_truck_"/>
+  <!-- *************** -->
+  <!-- Robots Elements -->
+  <!-- *************** -->
+  <!-- Here we create the robot elements using the xacro:macros imported at the beggining of this file -->
+  <xacro:arg name="prefix" default="pallet_truck_"/>
   <xacro:property name="prefix" value="$(arg prefix)" />
-	<xacro:pallet_truck prefix="${prefix}" publish_bf="true"/> <!-- BASE -->
-	<xacro:motor_wheel prefix="${prefix}" parent="${prefix}front_case_link">
-			<origin xyz="${wheel_offset_x} ${wheel_offset_y} ${wheel_offset_z}" rpy="0 0 0"/>
-	</xacro:motor_wheel>
+  <xacro:pallet_truck prefix="${prefix}" publish_bf="true"/> <!-- BASE -->
+  <xacro:motor_wheel prefix="${prefix}" parent="${prefix}front_case_link">
+      <origin xyz="${wheel_offset_x} ${wheel_offset_y} ${wheel_offset_z}" rpy="0 0 0"/>
+  </xacro:motor_wheel>
   <xacro:fork_wheel prefix="${prefix}left_fork_" parent="${prefix}base_link">
       <origin xyz="${fork_wheel_offset_x} ${fork_wheel_offset_y} ${fork_wheel_offset_z}" rpy="0 0 0"/>
@@ -88,5 +88,5 @@
   <xacro:front_case prefix="${prefix}" parent="${prefix}base_link">
     <origin xyz="${front_case_offset_x} -${front_case_offset_y} ${front_case_offset_z}" rpy="0 0 0"/>
-	</xacro:front_case>
+  </xacro:front_case>
   <xacro:support_wheel prefix="${prefix}front_left_" parent="${prefix}front_case_link">
       <origin xyz="${front_support_wheel_offset_x} ${front_support_wheel_offset_x} ${front_support_wheel_offset_z}" rpy="0 0 0"/>
@@ -95,8 +95,8 @@
       <origin xyz="${front_support_wheel_offset_x} -${front_support_wheel_offset_x} ${front_support_wheel_offset_z}" rpy="0 0 0"/>
   </xacro:support_wheel>
-  <xacro:sensor_rplidar prefix="${prefix}rplidar" parent="${prefix}front_case_link">
-      <origin xyz="${lidar_offset_x} ${lidar_offset_y} ${lidar_offset_z}" rpy="0 0 0"/>
-  </xacro:sensor_rplidar>
-  <xacro:sensor_sick_s300 prefix="${prefix}front_laser" parent="${prefix}front_case_link">
+  <xacro:sensor_rslidar_16 prefix="${prefix}top_lidar" parent="${prefix}front_case_link" prefix_topic="top_lidar" gpu="true">
+      <origin xyz="${top_lidar_offset_x} ${top_lidar_offset_y} ${top_lidar_offset_z}" rpy="0 0 0"/>
+  </xacro:sensor_rslidar_16>
+  <xacro:sensor_sick_s300 prefix="${prefix}front_laser" parent="${prefix}front_case_link" prefix_topic="front_laser" min_angle="-2.35" max_angle="2.35" >
       <origin xyz="${front_laser_x} ${front_laser_y} ${front_laser_z}" rpy="${PI} 0 0"/>
   </xacro:sensor_sick_s300>
@@ -104,31 +104,31 @@
   <!-- Front -->
   <joint name="${prefix}front_register_joint" type="fixed">
-     <origin xyz="${front_register_offset_x} ${front_register_offset_y} ${front_register_offset_z}" rpy="0 0 0"/>
+    <origin xyz="${front_register_offset_x} ${front_register_offset_y} ${front_register_offset_z}" rpy="0 0 0"/>
+    <parent link="${prefix}front_case_link"/>
+    <child link="${prefix}front_register_link" />
+  </joint>
+  <link name="${prefix}front_register_link">
+  </link>
+  <!-- Right side -->
+  <joint name="${prefix}right_register_joint" type="fixed">
+    <origin xyz="${side_register_offset_x} -${side_register_offset_y} ${side_register_offset_z}" rpy="0 0 -${PI/2.0}"/>
      <parent link="${prefix}front_case_link"/>
-     <child link="${prefix}front_register_link" />
-   </joint>
-   <link name="${prefix}front_register_link">
-   </link>
-   <!-- Right side -->
-   <joint name="${prefix}right_register_joint" type="fixed">
-     <origin xyz="${side_register_offset_x} -${side_register_offset_y} ${side_register_offset_z}" rpy="0 0 -${PI/2.0}"/>
-      <parent link="${prefix}front_case_link"/>
-      <child link="${prefix}right_register_link" />
-    </joint>
-    <link name="${prefix}right_register_link">
-    </link>
-   <!-- Left side -->
-   <joint name="${prefix}left_register_joint" type="fixed">
-      <origin xyz="${side_register_offset_x} ${side_register_offset_y} ${side_register_offset_z}" rpy="0 0 ${PI/2.0}"/>
-      <parent link="${prefix}front_case_link"/>
-      <child link="${prefix}left_register_link" />
-    </joint>
-    <link name="${prefix}left_register_link">
-    </link>
-	<!-- Gazebo ros control pluggins -->
-	<xacro:ros_control />
-	<xacro:sensor_imu_hector prefix="${prefix}imu" parent="${prefix}base_link">
-		<origin xyz="${imu_offset_x} -${imu_offset_y} ${imu_offset_z}" rpy="0 0 0"/>
-	</xacro:sensor_imu_hector>
+     <child link="${prefix}right_register_link" />
+  </joint>
+  <link name="${prefix}right_register_link">
+  </link>
+  <!-- Left side -->
+  <joint name="${prefix}left_register_joint" type="fixed">
+     <origin xyz="${side_register_offset_x} ${side_register_offset_y} ${side_register_offset_z}" rpy="0 0 ${PI/2.0}"/>
+     <parent link="${prefix}front_case_link"/>
+     <child link="${prefix}left_register_link" />
+  </joint>
+  <link name="${prefix}left_register_link">
+  </link>
+  <!-- Gazebo ros control pluggins -->
+  <xacro:ros_control />
+  <xacro:sensor_imu_hector prefix="${prefix}imu" parent="${prefix}base_link">
+    <origin xyz="${imu_offset_x} -${imu_offset_y} ${imu_offset_z}" rpy="0 0 0"/>
+  </xacro:sensor_imu_hector>
   <gazebo>
     <plugin name="ground_truth_controller" filename="librobotnik_gazebo_ground_truth_odom.so">

Commit message: added realsense simulation

File: pallet_truck_common/pallet_truck_description/robots/pallet_truck_std.urdf.xacro (robot description, xacro)
@@ -101,4 +101,13 @@
       <origin xyz="${front_laser_x} ${front_laser_y} ${front_laser_z}" rpy="${PI} 0 0"/>
   </xacro:sensor_sick_s300>
+  <xacro:sensor_intel_d435 prefix="${prefix}left_fork_camera" parent="${prefix}left_fork_sensor_link" prefix_topic="left_fork_camera" use_nominal_extrinsics="true" >
+        <origin xyz="0 0 0" rpy="0 0 0"/>
+  </xacro:sensor_intel_d435>
+  <xacro:sensor_intel_d435 prefix="${prefix}right_fork_camera" parent="${prefix}right_fork_sensor_link" prefix_topic="right_fork_camera"  use_nominal_extrinsics="true" >
+        <origin xyz="0 0 0" rpy="0 0 0"/>
+  </xacro:sensor_intel_d435>
+  <xacro:sensor_imu_hector prefix="${prefix}imu" parent="${prefix}base_link">
+    <origin xyz="${imu_offset_x} -${imu_offset_y} ${imu_offset_z}" rpy="0 0 0"/>
+  </xacro:sensor_imu_hector>
   <!-- REGISTERS -->
   <!-- Front -->
@@ -128,7 +137,4 @@
   <!-- Gazebo ros control pluggins -->
   <xacro:ros_control />
-  <xacro:sensor_imu_hector prefix="${prefix}imu" parent="${prefix}base_link">
-    <origin xyz="${imu_offset_x} -${imu_offset_y} ${imu_offset_z}" rpy="0 0 0"/>
-  </xacro:sensor_imu_hector>
   <gazebo>
     <plugin name="ground_truth_controller" filename="librobotnik_gazebo_ground_truth_odom.so">

File: pallet_truck_common/pallet_truck_description/urdf/elevator/fork.urdf.xacro (robot description, xacro)
@@ -58,4 +58,11 @@
        <material>Gazebo/Black</material>
      </gazebo>
+    <joint name="${prefix}fork_sensor_joint" type="fixed">
+       <!-- xyz is estimated, not from cad -->
+       <origin xyz="-1.05 0.00000 0.012941" rpy="0 0 3.14159" />
+       <parent link="${prefix}fork_link"/>
+       <child link="${prefix}fork_sensor_link" />
+     </joint>
+    <link name="${prefix}fork_sensor_link" />
   </xacro:macro>
 </robot>

Commit message: simulation works with several spawned robot
however:
- odometry does not work properly (both robots move)
- imu is not subscribed

File: pallet_truck_common/pallet_truck_description/robots/pallet_truck_std.urdf.xacro (robot description, xacro)
@@ -71,5 +71,7 @@
   <!-- *************** -->
   <!-- Here we create the robot elements using the xacro:macros imported at the beggining of this file -->
-  <xacro:arg name="prefix" default="pallet_truck_"/>
+  <xacro:arg name="id_robot" default="pallet_truck"/>
+  <xacro:arg name="prefix" default="$(arg prefix)_"/>
+  <xacro:property name="id_robot" value="$(arg id_robot)" />
   <xacro:property name="prefix" value="$(arg prefix)" />
   <xacro:pallet_truck prefix="${prefix}" publish_bf="true"/> <!-- BASE -->
@@ -101,8 +103,8 @@
       <origin xyz="${front_laser_x} ${front_laser_y} ${front_laser_z}" rpy="${PI} 0 0"/>
   </xacro:sensor_sick_s300>
-  <xacro:sensor_intel_d435 prefix="${prefix}left_fork_camera" parent="${prefix}left_fork_sensor_link" prefix_topic="left_fork_camera" use_nominal_extrinsics="true" >
+  <xacro:sensor_intel_d435 prefix="${prefix}left_fork_camera" parent="${prefix}left_fork_sensor_link" prefix_topic="${id_robot}/left_fork_camera" use_nominal_extrinsics="true" >
         <origin xyz="0 0 0" rpy="0 0 0"/>
   </xacro:sensor_intel_d435>
-  <xacro:sensor_intel_d435 prefix="${prefix}right_fork_camera" parent="${prefix}right_fork_sensor_link" prefix_topic="right_fork_camera"  use_nominal_extrinsics="true" >
+  <xacro:sensor_intel_d435 prefix="${prefix}right_fork_camera" parent="${prefix}right_fork_sensor_link" prefix_topic="${id_robot}/right_fork_camera" use_nominal_extrinsics="true" >
         <origin xyz="0 0 0" rpy="0 0 0"/>
   </xacro:sensor_intel_d435>

Commit message: solved inconsistency of xx_robot and robot_xx

File: pallet_truck_common/pallet_truck_description/robots/pallet_truck_std.urdf.xacro (robot description, xacro)
@@ -72,7 +72,7 @@
   <!-- *************** -->
   <!-- Here we create the robot elements using the xacro:macros imported at the beggining of this file -->
-  <xacro:arg name="id_robot" default="pallet_truck"/>
+  <xacro:arg name="robot_id" default="pallet_truck"/>
   <xacro:arg name="prefix" default="$(arg prefix)_"/>
-  <xacro:property name="id_robot" value="$(arg id_robot)" />
+  <xacro:property name="robot_id" value="$(arg robot_id)" />
   <xacro:property name="prefix" value="$(arg prefix)" />
   <xacro:pallet_truck prefix="${prefix}" publish_bf="true"/> <!-- BASE -->
@@ -104,8 +104,8 @@
       <origin xyz="${front_laser_x} ${front_laser_y} ${front_laser_z}" rpy="${PI} 0 0"/>
   </xacro:sensor_sick_s300>
-  <xacro:sensor_intel_d435 prefix="${prefix}left_fork_camera" parent="${prefix}left_fork_sensor_link" prefix_topic="${id_robot}/left_fork_camera" use_nominal_extrinsics="true" >
+  <xacro:sensor_intel_d435 prefix="${prefix}left_fork_camera" parent="${prefix}left_fork_sensor_link" prefix_topic="${robot_id}/left_fork_camera" use_nominal_extrinsics="true" >
         <origin xyz="0 0 0" rpy="0 0 0"/>
   </xacro:sensor_intel_d435>
-  <xacro:sensor_intel_d435 prefix="${prefix}right_fork_camera" parent="${prefix}right_fork_sensor_link" prefix_topic="${id_robot}/right_fork_camera" use_nominal_extrinsics="true" >
+  <xacro:sensor_intel_d435 prefix="${prefix}right_fork_camera" parent="${prefix}right_fork_sensor_link" prefix_topic="${robot_id}/right_fork_camera" use_nominal_extrinsics="true" >
         <origin xyz="0 0 0" rpy="0 0 0"/>
   </xacro:sensor_intel_d435>

Commit message: select if simulation uses gpu or not (and documented!)

File: pallet_truck_common/pallet_truck_description/robots/pallet_truck_std.urdf.xacro (robot description, xacro)
@@ -72,8 +72,9 @@
   <!-- *************** -->
   <!-- Here we create the robot elements using the xacro:macros imported at the beggining of this file -->
-  <xacro:arg name="robot_id" default="pallet_truck"/>
+  <xacro:arg name="robot_id" default="$(arg robot_id)"/>
   <xacro:arg name="prefix" default="$(arg prefix)_"/>
   <xacro:property name="robot_id" value="$(arg robot_id)" />
   <xacro:property name="prefix" value="$(arg prefix)" />
+  <xacro:property name="gpu" value="$(arg use_gpu_for_simulation)" />
   <xacro:pallet_truck prefix="${prefix}" publish_bf="true"/> <!-- BASE -->
   <xacro:motor_wheel prefix="${prefix}" parent="${prefix}front_case_link">
@@ -98,8 +99,8 @@
       <origin xyz="${front_support_wheel_offset_x} -${front_support_wheel_offset_x} ${front_support_wheel_offset_z}" rpy="0 0 0"/>
   </xacro:support_wheel>
-  <xacro:sensor_rslidar_16 prefix="${prefix}top_lidar" parent="${prefix}front_case_link" prefix_topic="top_lidar" gpu="false">
+  <xacro:sensor_rslidar_16 prefix="${prefix}top_lidar" parent="${prefix}front_case_link" prefix_topic="top_lidar" gpu="${gpu}">
       <origin xyz="${top_lidar_offset_x} ${top_lidar_offset_y} ${top_lidar_offset_z}" rpy="0 0 0"/>
   </xacro:sensor_rslidar_16>
-  <xacro:sensor_sick_s300 prefix="${prefix}front_laser" parent="${prefix}front_case_link" prefix_topic="front_laser" min_angle="-2.35" max_angle="2.35" >
+  <xacro:sensor_sick_s300 prefix="${prefix}front_laser" parent="${prefix}front_case_link" prefix_topic="front_laser" min_angle="-2.35" max_angle="2.35" gpu="${gpu}" >
       <origin xyz="${front_laser_x} ${front_laser_y} ${front_laser_z}" rpy="${PI} 0 0"/>
   </xacro:sensor_sick_s300>

Commit message: updated camera positions

File: pallet_truck_common/pallet_truck_description/robots/pallet_truck_std.urdf.xacro (robot description, xacro)
@@ -61,4 +61,7 @@
   <xacro:property name="front_register_offset_y" value="0.0" />
   <xacro:property name="front_register_offset_z" value="-0.228" />
+  <xacro:property name="rear_register_offset_x" value="-0.452" />
+  <xacro:property name="rear_register_offset_y" value="0.0" />
+  <xacro:property name="rear_register_offset_z" value="-0.228" />
   <xacro:property name="side_register_offset_x" value="0.1855" />
   <xacro:property name="side_register_offset_y" value="0.276" />
@@ -106,8 +109,11 @@
   </xacro:sensor_sick_s300>
   <xacro:sensor_intel_d435 prefix="${prefix}left_fork_camera" parent="${prefix}left_fork_sensor_link" prefix_topic="${robot_id}/left_fork_camera" use_nominal_extrinsics="true" >
-        <origin xyz="0 0 0" rpy="0 0 0"/>
+        <origin xyz="0 0 0" rpy="0 -${5.0*PI/180.0} 0"/>
   </xacro:sensor_intel_d435>
   <xacro:sensor_intel_d435 prefix="${prefix}right_fork_camera" parent="${prefix}right_fork_sensor_link" prefix_topic="${robot_id}/right_fork_camera" use_nominal_extrinsics="true" >
-        <origin xyz="0 0 0" rpy="0 0 0"/>
+        <origin xyz="0 0 0" rpy="0 -${5.0*PI/180.0} 0"/>
+  </xacro:sensor_intel_d435>
+  <xacro:sensor_intel_d435 prefix="${prefix}rear_camera" parent="${prefix}rear_register_link" prefix_topic="${robot_id}/rear_camera" use_nominal_extrinsics="true" >
+        <origin xyz="0 0 0" rpy="0 ${5.0*PI/180.0} 0"/>
   </xacro:sensor_intel_d435>
   <xacro:sensor_imu_hector prefix="${prefix}imu" parent="${prefix}base_link">
@@ -122,4 +128,12 @@
   </joint>
   <link name="${prefix}front_register_link">
+  </link>
+  <!-- Rear -->
+  <joint name="${prefix}rear_register_joint" type="fixed">
+    <origin xyz="${rear_register_offset_x} ${rear_register_offset_y} ${rear_register_offset_z}" rpy="0 0 -${PI}"/>
+    <parent link="${prefix}front_case_link"/>
+    <child link="${prefix}rear_register_link" />
+  </joint>
+  <link name="${prefix}rear_register_link">
   </link>
   <!-- Right side -->

Commit message: Corrected castor wheels position (wrong y_offset)

File: pallet_truck_common/pallet_truck_description/robots/pallet_truck_std.urdf.xacro (robot description, xacro)
@@ -98,8 +98,8 @@
   </xacro:front_case>
   <xacro:support_wheel prefix="${prefix}front_left_" parent="${prefix}front_case_link">
-      <origin xyz="${front_support_wheel_offset_x} ${front_support_wheel_offset_x} ${front_support_wheel_offset_z}" rpy="0 0 0"/>
+      <origin xyz="${front_support_wheel_offset_x} ${front_support_wheel_offset_y} ${front_support_wheel_offset_z}" rpy="0 0 0"/>
   </xacro:support_wheel>
   <xacro:support_wheel prefix="${prefix}front_right_" parent="${prefix}front_case_link">
-      <origin xyz="${front_support_wheel_offset_x} -${front_support_wheel_offset_x} ${front_support_wheel_offset_z}" rpy="0 0 0"/>
+      <origin xyz="${front_support_wheel_offset_x} -${front_support_wheel_offset_y} ${front_support_wheel_offset_z}" rpy="0 0 0"/>
   </xacro:support_wheel>
   <xacro:sensor_rslidar_16 prefix="${prefix}top_lidar" parent="${prefix}front_case_link" prefix_topic="top_lidar" gpu="${gpu}">
